File: MIPI.sch (KiCad schematic (older format))
At the start: 47 parts

Commit message: update
Parts:
- removed RPi_CAMERA?: 1.0mm-pitch_ZIF_SMT-15P, OLIMEX_Connectors-FP:TE_1-1734248-5, symbol S3-OLinuXino_Rev_A:RPi_LCD-MiPi(1-1734248-5)
Connections:
- net labels added: MIPI-MSCK
- net labels removed: MCSI_CK+, MCSI_CK-, MCSI_DATA0+, MCSI_DATA0-, MCSI_DATA1+, MCSI_DATA1-
- wire segments 164 -> 140
- no-connect marks 17 -> 2
Other:
- note removed: "RPi-MiPi_Camera"
Changed lines of the file:
@@
 $EndComp
-Wire Notes Line
-	11300 800  7400 800
 Wire Notes Line
 	11300 800  11300 2900
-Text Notes 7900 1100 0    150  Italic 30
-RPi-MiPi_Camera
 $Comp
 L S3-OLinuXino_Rev_A:GND #PWR?
@@
 	1    0    0    -1
 $EndComp
-Wire Wire Line
-	10100 2200 9400 2200
-Wire Wire Line
-	10100 2300 9400 2300
-Text Label 9200 1900 0    60   Italic 12
-MCSI_CK-
-Text Label 9200 1600 0    60   Italic 12
-MCSI_DATA1-
-Text Label 9200 1700 0    60   Italic 12
-MCSI_DATA1+
-Text Label 9200 2000 0    60   Italic 12
-MCSI_CK+
-Text Label 9200 1300 0    60   Italic 12
-MCSI_DATA0-
-Text Label 9200 1400 0    60   Italic 12
-MCSI_DATA0+
-Wire Wire Line
-	10100 1500 9100 1500
-Wire Wire Line
-	10100 2100 9100 2100
-Wire Wire Line
-	10100 2400 9400 2400
-Wire Wire Line
-	10100 2500 9400 2500
-Wire Wire Line
-	10100 2600 9100 2600
-Wire Wire Line
-	10100 1800 9100 1800
-Wire Wire Line
-	10100 1200 9100 1200
-$Comp
-L S3-OLinuXino_Rev_A:RPi_LCD-MiPi(1-1734248-5) RPi_CAMERA?
-U 1 1 621FACD3
-P 10400 1900
-AR Path="/5D8A1FAC/621FACD3" Ref="RPi_CAMERA?"  Part="1"
-AR Path="/621FACD3" Ref="RPi_CAMERA?"  Part="1"
-AR Path="/620E795B/621FACD3" Ref="RPi_CAMERA?"  Part="1"
-F 0 "RPi_CAMERA?" H 10350 2750 50  0000 C CNN
-F 1 "1.0mm-pitch_ZIF_SMT-15P" H 10350 1050 50  0000 C CNN
-F 2 "OLIMEX_Connectors-FP:TE_1-1734248-5" H 10400 900 40  0001 C CNN
-F 3 "" H 10400 1700 60  0000 C CNN
-	1    10400 1900
-	1    0    0    -1
-$EndComp
-Wire Wire Line
-	10600 2600 11000 2600
-Wire Wire Line
-	10600 2500 11000 2500
-Wire Wire Line
-	10600 2400 11000 2400
-Wire Wire Line
-	10600 2000 11000 2000
-Wire Wire Line
-	10600 1900 11000 1900
-Wire Wire Line
-	10600 1700 11000 1700
-Wire Wire Line
-	10600 2200 11000 2200
-Wire Wire Line
-	10600 2100 11000 2100
-Wire Wire Line
-	10600 1200 11000 1200
-Wire Wire Line
-	10600 1300 11000 1300
-Wire Wire Line
-	10600 2300 11000 2300
-Wire Wire Line
-	10600 1800 11000 1800
-Wire Wire Line
-	10600 1500 11000 1500
-Wire Wire Line
-	10600 1400 11000 1400
-Wire Wire Line
-	10600 1600 11000 1600
-NoConn ~ 11000 1600
-NoConn ~ 11000 1400
-NoConn ~ 11000 1500
-NoConn ~ 11000 1800
-NoConn ~ 11000 2300
-NoConn ~ 11000 1300
-NoConn ~ 11000 1200
-NoConn ~ 11000 2100
-NoConn ~ 11000 2200
-NoConn ~ 11000 1700
-NoConn ~ 11000 1900
-NoConn ~ 11000 2000
-NoConn ~ 11000 2400
-NoConn ~ 11000 2500
-NoConn ~ 11000 2600
 $Comp
 L S3-OLinuXino_Rev_A:+3.3V #PWR?
@@
 Wire Wire Line
 	4100 3400 5300 3400
+Text GLabel 8100 2700 2    50   Input ~ 0
+MIPI-MSCK
 $EndSCHEMATC

Commit message: update
Parts:
- gave numbers to parts that had none: 46

Commit message: update
Parts:
- added J9: MIPI, otter:FH35C-25S, symbol Connector_Generic_MountingPin:Conn_01x25_MountingPin
- added R94: 51, otter:C_0402, symbol Device:R_Small
- U1: footprint OLIMEX_IC-FP:FBGA-234(Pitch-0.65mm_Pad-0.3mm_11x11x1.08mm) -> otter:FBGA-234(Pitch-0.65mm_Pad-0.3mm_11x11x1.08mm)
- Y2, Y3: footprint (none) -> otter:Oscillator_3225
Connections:
- net +3V3: now also J9.2 (Pin_2), J9.3 (Pin_3)
- net GND: now also J9.1 (Pin_1), J9.10 (Pin_10), J9.13 (Pin_13), J9.16 (Pin_16), J9.19 (Pin_19), J9.22 (Pin_22), J9.25 (Pin_25), J9.4 (Pin_4), J9.8 (Pin_8), J9.MP (MountPin)
- net MIPI-CK_N: now also J9.12 (Pin_12)
- net MIPI-CK_P: now also J9.11 (Pin_11)
- net MIPI-D0_N: now also J9.15 (Pin_15)
- net MIPI-D0_P: now also J9.14 (Pin_14)
- net MIPI-D1_N: now also J9.18 (Pin_18)
- net MIPI-D1_P: now also J9.17 (Pin_17)
- net MIPI-D2_N: now also J9.21 (Pin_21)
- net MIPI-D2_P: now also J9.20 (Pin_20)
- net MIPI-D3_N: now also J9.24 (Pin_24)
- net MIPI-D3_P: now also J9.23 (Pin_23)
- net MIPI-MSCK: now also R94.2
- net MIPI-RESET: now also J9.7 (Pin_7)
- net MIPI-SCK: now also J9.5 (Pin_5)
- net MIPI-SDA: now also J9.6 (Pin_6)
- new net: J9.9 (Pin_9), R94.1
Other:
- moved on the sheet: C100, C101, C102, C103, C104, J8, R90, R91, R92, R93

Commit message: update
Parts:
- Y2: footprint otter:Oscillator_3225 -> Crystal:Crystal_SMD_3215-2Pin_3.2x1.5mm
Changed lines of the file:
@@
 F 0 "Y2" H 5000 4750 50  0000 C CNN
 F 1 "32.768kHz" H 5000 4650 50  0000 C CNN
-F 2 "otter:Oscillator_3225" H 4650 4700 50  0001 C CNN
+F 2 "Crystal:Crystal_SMD_3215-2Pin_3.2x1.5mm" H 4650 4700 50  0001 C CNN
 F 3 "~" H 4650 4700 50  0001 C CNN
 	1    4650 4700

Commit message: update
Parts:
- Y2: footprint Crystal:Crystal_SMD_3215-2Pin_3.2x1.5mm -> otter:Crystal_SMD_3215-2Pin_3.2x1.5mm
Changed lines of the file:
@@
 F 0 "Y2" H 5000 4750 50  0000 C CNN
 F 1 "32.768kHz" H 5000 4650 50  0000 C CNN
-F 2 "Crystal:Crystal_SMD_3215-2Pin_3.2x1.5mm" H 4650 4700 50  0001 C CNN
+F 2 "otter:Crystal_SMD_3215-2Pin_3.2x1.5mm" H 4650 4700 50  0001 C CNN
 F 3 "~" H 4650 4700 50  0001 C CNN
 	1    4650 4700

Commit message: update
Parts:
- removed R85: 0, otter:C_0402, symbol Device:R_Small
Connections:
- net at U1.P4 (X24MOUT): now also C94.1, Y3.3
Changed lines of the file:
@@
 	4100 4900 4400 4900
-Wire Wire Line
-	4200 5300 4100 5300
 Wire Wire Line
 	4100 4400 4550 4400
@@
 	2550 5600 2500 5600
 $Comp
-L Device:R_Small R?
-U 1 1 687D2D86
-P 4300 5300
-AR Path="/687D2D86" Ref="R?"  Part="1"
-AR Path="/620E795B/687D2D86" Ref="R85"  Part="1"
-F 0 "R85" V 4404 5300 50  0000 C CNN
-F 1 "0" V 4495 5300 50  0000 C CNN
-F 2 "otter:C_0402" H 4300 5300 50  0001 C CNN
-F 3 "~" H 4300 5300 50  0001 C CNN
-	1    4300 5300
-	0    1    1    0
-$EndComp
-$Comp
 L Device:Crystal_GND24_Small Y3
 U 1 1 687E2CB7
@@
 Wire Wire Line
 	10300 4200 10550 4200
+Wire Wire Line
+	4100 5300 4400 5300
 $EndSCHEMATC

Commit message: update
Parts:
- removed C80: 4.7u, otter:C_0603, symbol Device:C_Small
- removed C81, C87: 10u, otter:C_0603, symbol Device:C_Small
- removed C86: DNP, otter:C_0603, symbol Device:C_Small
- added C?: 100n, otter:C_0402, symbol Device:C_Small
Connections:
- net GND: now also C?.2
- net at R78.1, U1.N10 (VRA2): now also C?.1
- net HPOUTFB: no longer names the net of U1.N11 (HPCOMFB)
- net HPOUTFB: no longer U1.N12 (HPCOM)
- net HPOUTL: no longer names the net of U1.P13 (HPOUTL)
- net HPOUTR: no longer names the net of U1.N13 (HPOUTR)
- net LINEINL: no longer names the net of U1.R12 (LINEINL)
- net LINEINR: no longer names the net of U1.T12 (LINEINR)
- net LINEOUTL: no longer names the net of U1.R6 (LINEOUTL)
- net LINEOUTR: no longer names the net of U1.T6 (LINEOUTR)
- net MBIAS: no longer names the net of U1.P10 (MBIAS)
- net MICIN1_N: no longer names the net of U1.R10 (MICIN1N)
- net MICIN1_P: no longer names the net of U1.T10 (MICIN1P)
- net MICIN3_N: no longer names the net of U1.R9 (MICIN3N)
- net MICIN3_P: no longer names the net of U1.P9 (MICIN3P)
- no-connect marks 2 -> 8
Other:
- moved on the sheet: C85
Changed lines of the file:
@@
 L S3-OLinuXino_Rev_A:GND #PWR?
 U 1 1 621FAA25
-P 2000 3900
+P 2350 3900
 AR Path="/5D8A1FAC/621FAA25" Ref="#PWR?"  Part="1"
 AR Path="/621FAA25" Ref="#PWR?"  Part="1"
 AR Path="/620E795B/621FAA25" Ref="#PWR0245"  Part="1"
-F 0 "#PWR0245" H 2000 3650 50  0001 C CNN
-F 1 "GND" V 2000 3700 50  0000 C CNN
-F 2 "" H 2000 3900 60  0000 C CNN
-F 3 "" H 2000 3900 60  0000 C CNN
-	1    2000 3900
+F 0 "#PWR0245" H 2350 3650 50  0001 C CNN
+F 1 "GND" V 2350 3700 50  0000 C CNN
+F 2 "" H 2350 3900 60  0000 C CNN
+F 3 "" H 2350 3900 60  0000 C CNN
+	1    2350 3900
 	0    1    -1   0
 $EndComp
@@
 L S3-OLinuXino_Rev_A:+3.0VA #PWR?
 U 1 1 621FAA2B
-P 2000 3700
+P 2350 3700
 AR Path="/5D8A1FAC/621FAA2B" Ref="#PWR?"  Part="1"
 AR Path="/621FAA2B" Ref="#PWR?"  Part="1"
 AR Path="/620E795B/621FAA2B" Ref="#PWR0246"  Part="1"
-F 0 "#PWR0246" H 2000 3550 50  0001 C CNN
-F 1 "+3.0VA" V 2000 3800 50  0000 L CNN
-F 2 "" H 2000 3700 60  0000 C CNN
-F 3 "" H 2000 3700 60  0000 C CNN
-	1    2000 3700
+F 0 "#PWR0246" H 2350 3550 50  0001 C CNN
+F 1 "+3.0VA" V 2350 3800 50  0000 L CNN
+F 2 "" H 2350 3700 60  0000 C CNN
+F 3 "" H 2350 3700 60  0000 C CNN
+	1    2350 3700
 	0    -1   -1   0
 $EndComp
@@
 $Comp
 L S3-OLinuXino_Rev_A:GND #PWR?
-U 1 1 621FAA55
-P 2000 3100
-AR Path="/5D8A1FAC/621FAA55" Ref="#PWR?"  Part="1"
-AR Path="/621FAA55" Ref="#PWR?"  Part="1"
-AR Path="/620E795B/621FAA55" Ref="#PWR0248"  Part="1"
-F 0 "#PWR0248" H 2000 2850 50  0001 C CNN
-F 1 "GND" H 2005 2927 50  0000 C CNN
-F 2 "" H 2000 3100 60  0000 C CNN
-F 3 "" H 2000 3100 60  0000 C CNN
-	1    2000 3100
-	-1   0    0    -1
-$EndComp
-$Comp
-L S3-OLinuXino_Rev_A:GND #PWR?
 U 1 1 621FAA8A
 P 1200 4350
@@
 Text GLabel 2700 2500 0    50   Input ~ 0
 USB-D_P
-Text GLabel 2700 2700 0    50   Input ~ 0
-MBIAS
-Text GLabel 2700 2900 0    50   Input ~ 0
-MICIN3_P
-Text GLabel 2700 3000 0    50   Input ~ 0
-MICIN3_N
-Text GLabel 2700 3300 0    50   Input ~ 0
-MICIN1_P
-Text GLabel 2700 3400 0    50   Input ~ 0
-MICIN1_N
-Wire Wire Line
-	2700 4300 2700 4400
-Text GLabel 2700 4400 0    50   Input ~ 0
-HPOUTFB
-Text GLabel 2700 4500 0    50   Input ~ 0
-HPOUTL
-Text GLabel 2700 4600 0    50   Input ~ 0
-HPOUTR
-Text GLabel 2700 4800 0    50   Input ~ 0
-LINEOUTL
-Text GLabel 2700 4900 0    50   Input ~ 0
-LINEINL
-Text GLabel 2700 5000 0    50   Input ~ 0
-LINEINR
-Wire Wire Line
-	1600 4250 1600 4200
-Wire Wire Line
-	1600 4200 1950 4200
-Wire Wire Line
-	1950 4250 1950 4200
-Connection ~ 1950 4200
-Wire Wire Line
-	1950 4200 2700 4200
-Wire Wire Line
-	1950 4500 1600 4500
-Wire Wire Line
-	1600 4500 1600 4450
-Wire Wire Line
-	1950 4500 1950 4450
-Wire Wire Line
-	1550 4500 1600 4500
-Connection ~ 1600 4500
 Wire Wire Line
 	1200 4350 1250 4350
@@
 $EndComp
 Wire Wire Line
-	2050 3700 2400 3700
-Wire Wire Line
-	2050 3900 2400 3900
-Connection ~ 2400 3700
-Wire Wire Line
 	2400 3700 2700 3700
-Connection ~ 2400 3900
 Wire Wire Line
 	2400 3900 2700 3900
-Wire Wire Line
-	2000 3700 2050 3700
-Connection ~ 2050 3700
-Wire Wire Line
-	2000 3900 2050 3900
-Connection ~ 2050 3900
-$Comp
-L Device:C_Small C?
-U 1 1 681C1C81
-P 1300 3650
-AR Path="/681C1C81" Ref="C?"  Part="1"
-AR Path="/602ACDF9/681C1C81" Ref="C?"  Part="1"
-AR Path="/620E795B/681C1C81" Ref="C80"  Part="1"
-F 0 "C80" H 1392 3696 50  0000 L CNN
-F 1 "4.7u" H 1392 3605 50  0000 L CNN
-F 2 "otter:C_0603" H 1300 3650 50  0001 C CNN
-F 3 "~" H 1300 3650 50  0001 C CNN
-	1    1300 3650
-	1    0    0    -1
-$EndComp
 Wire Wire Line
 	1300 3500 1300 3550
@@
 	1100 3800 1150 3800
 Connection ~ 1150 3800
-$Comp
-L Device:C_Small C?
-U 1 1 68254F7D
-P 2000 2950
-AR Path="/68254F7D" Ref="C?"  Part="1"
-AR Path="/602ACDF9/68254F7D" Ref="C?"  Part="1"
-AR Path="/620E795B/68254F7D" Ref="C86"  Part="1"
-F 0 "C86" H 2092 2996 50  0000 L CNN
-F 1 "DNP" H 2092 2905 50  0000 L CNN
-F 2 "otter:C_0603" H 2000 2950 50  0001 C CNN
-F 3 "~" H 2000 2950 50  0001 C CNN
-	1    2000 2950
-	1    0    0    -1
-$EndComp
-Wire Wire Line
-	2000 2850 2000 2800
-Wire Wire Line
-	2000 2800 2700 2800
-Wire Wire Line
-	2000 3100 2000 3050
 $Comp
 L Device:C_Small C?
@@
 	5950 4350 5950 4400
 Connection ~ 5950 4400
-Text GLabel 2700 4700 0    50   Input ~ 0
-LINEOUTR
 $Comp
 L Connector:RJ45_Abracon_ARJP11A-MASA-B-A-EMU2 J8
@@
 $Comp
 L Device:C_Small C?
-U 1 1 68143627
-P 2050 3800
-AR Path="/68143627" Ref="C?"  Part="1"
-AR Path="/602ACDF9/68143627" Ref="C?"  Part="1"
-AR Path="/620E795B/68143627" Ref="C87"  Part="1"
-F 0 "C87" H 2142 3846 50  0000 L CNN
-F 1 "10u" H 2142 3755 50  0000 L CNN
-F 2 "otter:C_0603" H 2050 3800 50  0001 C CNN
-F 3 "~" H 2050 3800 50  0001 C CNN
-	1    2050 3800
-	1    0    0    -1
-$EndComp
-$Comp
-L Device:C_Small C?
 U 1 1 685A8C38
 P 2150 5300
@@
 $Comp
 L Device:C_Small C?
-U 1 1 68092C34
+U 1 1 68092C2E
 P 1600 4350
-AR Path="/68092C34" Ref="C?"  Part="1"
-AR Path="/602ACDF9/68092C34" Ref="C?"  Part="1"
-AR Path="/620E795B/68092C34" Ref="C81"  Part="1"
-F 0 "C81" H 1692 4396 50  0000 L CNN
-F 1 "10u" H 1692 4305 50  0000 L CNN
-F 2 "otter:C_0603" H 1600 4350 50  0001 C CNN
+AR Path="/68092C2E" Ref="C?"  Part="1"
+AR Path="/620E795B/68092C2E" Ref="C85"  Part="1"
+F 0 "C85" H 1692 4396 50  0000 L CNN
+F 1 "100n" H 1692 4305 50  0000 L CNN
+F 2 "otter:C_0402" H 1600 4350 50  0001 C CNN
 F 3 "~" H 1600 4350 50  0001 C CNN
 	1    1600 4350
-	1    0    0    -1
-$EndComp
-$Comp
-L Device:C_Small C?
-U 1 1 68092C2E
-P 1950 4350
-AR Path="/68092C2E" Ref="C?"  Part="1"
-AR Path="/620E795B/68092C2E" Ref="C85"  Part="1"
-F 0 "C85" H 2042 4396 50  0000 L CNN
-F 1 "100n" H 2042 4305 50  0000 L CNN
-F 2 "otter:C_0402" H 1950 4350 50  0001 C CNN
-F 3 "~" H 1950 4350 50  0001 C CNN
-	1    1950 4350
 	1    0    0    -1
 $EndComp
@@
 Wire Wire Line
 	4100 5300 4400 5300
+NoConn ~ 2700 2800
+NoConn ~ 2700 3000
+NoConn ~ 2700 2900
+NoConn ~ 2700 3400
+NoConn ~ 2700 3300
+NoConn ~ 2700 2700
+Wire Wire Line
+	1550 4500 1600 4500
+Wire Wire Line
+	1600 4500 1600 4450
+Wire Wire Line
+	1600 4250 1600 4200
+Wire Wire Line
+	1600 4200 2700 4200
+Wire Wire Line
+	2350 3700 2400 3700
+Connection ~ 2400 3700
+Wire Wire Line
+	2350 3900 2400 3900
+Connection ~ 2400 3900
+$Comp
+L Device:C_Small C?
+U 1 1 5FFEE453
+P 1300 3650
+AR Path="/5FFEE453" Ref="C?"  Part="1"
+AR Path="/620E795B/5FFEE453" Ref="C?"  Part="1"
+F 0 "C?" H 1392 3696 50  0000 L CNN
+F 1 "100n" H 1392 3605 50  0000 L CNN
+F 2 "otter:C_0402" H 1300 3650 50  0001 C CNN
+F 3 "~" H 1300 3650 50  0001 C CNN
+	1    1300 3650
+	1    0    0    -1
+$EndComp
 $EndSCHEMATC

Commit message: update
Parts:
- removed C84, C91: 100n, otter:C_0402, symbol Device:C_Small
- gave numbers to parts that had none: 1
Connections:
- no-connect marks 8 -> 16
Changed lines of the file:
@@
-$EndComp
-$Comp
-L S3-OLinuXino_Rev_A:GND #PWR?
-U 1 1 621FABB9
-P 1900 2550
-AR Path="/5D8A1FAC/621FABB9" Ref="#PWR?"  Part="1"
-AR Path="/621FABB9" Ref="#PWR?"  Part="1"
-AR Path="/620E795B/621FABB9" Ref="#PWR0259"  Part="1"
-F 0 "#PWR0259" H 1900 2300 50  0001 C CNN
-F 1 "GND" V 1900 2350 50  0000 C CNN
-F 2 "" H 1900 2550 60  0000 C CNN
-F 3 "" H 1900 2550 60  0000 C CNN
-	1    1900 2550
-	0    1    -1   0
 $EndComp
 $Comp
@@
 	0    1    1    0
 $EndComp
-Wire Wire Line
-	4100 2200 4750 2200
 $Comp
 L S3-OLinuXino_Rev_A:+3.3V_RTC #PWR?
@@
 L S3-OLinuXino_Rev_A:+3.3V #PWR?
 U 1 1 621FACF7
-P 4750 2150
+P 4100 2200
 AR Path="/5D8A1FAC/621FACF7" Ref="#PWR?"  Part="1"
 AR Path="/621FACF7" Ref="#PWR?"  Part="1"
 AR Path="/620E795B/621FACF7" Ref="#PWR0266"  Part="1"
-F 0 "#PWR0266" H 4750 2000 50  0001 C CNN
-F 1 "+3.3V" H 4765 2323 50  0000 C CNN
-F 2 "" H 4750 2150 60  0000 C CNN
-F 3 "" H 4750 2150 60  0000 C CNN
-	1    4750 2150
-	-1   0    0    -1
-$EndComp
-$Comp
-L S3-OLinuXino_Rev_A:GND #PWR?
-U 1 1 621FACFE
-P 4750 2450
-AR Path="/5D8A1FAC/621FACFE" Ref="#PWR?"  Part="1"
-AR Path="/621FACFE" Ref="#PWR?"  Part="1"
-AR Path="/620E795B/621FACFE" Ref="#PWR0267"  Part="1"
-F 0 "#PWR0267" H 4750 2200 50  0001 C CNN
-F 1 "GND" V 4750 2250 50  0000 C CNN
-F 2 "" H 4750 2450 60  0000 C CNN
-F 3 "" H 4750 2450 60  0000 C CNN
-	1    4750 2450
-	-1   0    0    -1
+F 0 "#PWR0266" H 4100 2050 50  0001 C CNN
+F 1 "+3.3V" V 4115 2328 50  0000 L CNN
+F 2 "" H 4100 2200 60  0000 C CNN
+F 3 "" H 4100 2200 60  0000 C CNN
+	1    4100 2200
+	0    1    -1   0
 $EndComp
 Text GLabel 10550 3900 0    50   Input ~ 0
@@
 	1100 3800 1150 3800
 Connection ~ 1150 3800
-$Comp
-L Device:C_Small C?
-U 1 1 682DD643
-P 1950 2450
-AR Path="/682DD643" Ref="C?"  Part="1"
-AR Path="/620E795B/682DD643" Ref="C84"  Part="1"
-F 0 "C84" H 2042 2496 50  0000 L CNN
-F 1 "100n" H 2042 2405 50  0000 L CNN
-F 2 "otter:C_0402" H 1950 2450 50  0001 C CNN
-F 3 "~" H 1950 2450 50  0001 C CNN
-	1    1950 2450
-	1    0    0    -1
-$EndComp
-Wire Wire Line
-	1950 2350 1950 2300
-Wire Wire Line
-	1950 2300 2700 2300
-Wire Wire Line
-	1900 2550 1950 2550
-Wire Wire Line
-	1900 2300 1950 2300
-Connection ~ 1950 2300
 Wire Wire Line
 	2000 1900 2100 1900
@@
 Text GLabel 4100 2300 2    50   Input ~ 0
 MIPI-D3_N
-$Comp
-L Device:C_Small C?
-U 1 1 6839075B
-P 4750 2350
-AR Path="/6839075B" Ref="C?"  Part="1"
-AR Path="/620E795B/6839075B" Ref="C91"  Part="1"
-F 0 "C91" H 4842 2396 50  0000 L CNN
-F 1 "100n" H 4842 2305 50  0000 L CNN
-F 2 "otter:C_0402" H 4750 2350 50  0001 C CNN
-F 3 "~" H 4750 2350 50  0001 C CNN
-	1    4750 2350
-	1    0    0    -1
-$EndComp
-Wire Wire Line
-	4750 2250 4750 2200
-Connection ~ 4750 2200
-Wire Wire Line
-	4750 2150 4750 2200
 Text GLabel 10550 4400 0    50   Input ~ 0
 MIPI-CK_P
@@
 P 1300 3650
 AR Path="/5FFEE453" Ref="C?"  Part="1"
-AR Path="/620E795B/5FFEE453" Ref="C?"  Part="1"
-F 0 "C?" H 1392 3696 50  0000 L CNN
+AR Path="/620E795B/5FFEE453" Ref="C3"  Part="1"
+F 0 "C3" H 1392 3696 50  0000 L CNN
 F 1 "100n" H 1392 3605 50  0000 L CNN
 F 2 "otter:C_0402" H 1300 3650 50  0001 C CNN
@@
 	1    0    0    -1
 $EndComp
+NoConn ~ 2700 4300
+NoConn ~ 2700 4400
+NoConn ~ 2700 4500
+NoConn ~ 2700 4600
+NoConn ~ 2700 4700
+NoConn ~ 2700 4800
+NoConn ~ 2700 4900
+NoConn ~ 2700 5000
+Wire Wire Line
+	1900 2300 2700 2300
 $EndSCHEMATC
