File: MIPI.sch (KiCad schematic (older format))
At the start: 40 parts, among them J8 49F-1201GYD2NL, U1 AllWinner-S3(FBGA-234), Y2 32.768kHz, Y3 24MHz

Commit message: fixed ETH, added AGND plane to prevent Line-In Noise, optimized power
Connections:
- net +3V3: now also J8.11, J8.9; no longer J8.10, J8.12
- net at R87.2: now also J8.12; no longer J8.11
- net at R88.2: now also J8.10; no longer J8.9
Other:
- moved on the sheet: R87, R88
Changed lines of the file:
@@
 L Device:R_Small R?
 U 1 1 6851960A
-P 7750 1450
+P 7650 1450
 AR Path="/6851960A" Ref="R?"  Part="1"
 AR Path="/620E795B/6851960A" Ref="R87"  Part="1"
-F 0 "R87" V 7700 1300 50  0000 C CNN
-F 1 "2k2" V 7700 1650 50  0000 C CNN
-F 2 "otter:R_0402" H 7750 1450 50  0001 C CNN
-F 3 "~" H 7750 1450 50  0001 C CNN
-	1    7750 1450
+F 0 "R87" V 7600 1300 50  0000 C CNN
+F 1 "2k2" V 7600 1650 50  0000 C CNN
+F 2 "otter:R_0402" H 7650 1450 50  0001 C CNN
+F 3 "~" H 7650 1450 50  0001 C CNN
+	1    7650 1450
 	1    0    0    -1
 $EndComp
@@
 L Device:R_Small R?
 U 1 1 685269CF
-P 7450 1450
+P 7350 1450
 AR Path="/685269CF" Ref="R?"  Part="1"
 AR Path="/620E795B/685269CF" Ref="R88"  Part="1"
-F 0 "R88" V 7400 1300 50  0000 C CNN
-F 1 "2k2" V 7400 1650 50  0000 C CNN
-F 2 "otter:R_0402" H 7450 1450 50  0001 C CNN
-F 3 "~" H 7450 1450 50  0001 C CNN
-	1    7450 1450
+F 0 "R88" V 7300 1300 50  0000 C CNN
+F 1 "2k2" V 7300 1650 50  0000 C CNN
+F 2 "otter:R_0402" H 7350 1450 50  0001 C CNN
+F 3 "~" H 7350 1450 50  0001 C CNN
+	1    7350 1450
 	1    0    0    -1
 $EndComp
@@
 Text GLabel 9000 2650 2    50   Input ~ 0
 EPHY_RX_N
-Text GLabel 7750 1200 1    50   Input ~ 0
+Text GLabel 7650 1200 1    50   Input ~ 0
 EPHY_LINK_LED
-Text GLabel 7450 1200 1    50   Input ~ 0
+Text GLabel 7350 1200 1    50   Input ~ 0
 EPHY_SPD_LED
 $Comp
 L S3-OLinuXino_Rev_A:+3.3V #PWR?
 U 1 1 68ABBB53
-P 7650 1650
+P 7750 1650
 AR Path="/5D8A1FAC/68ABBB53" Ref="#PWR?"  Part="1"
 AR Path="/68ABBB53" Ref="#PWR?"  Part="1"
 AR Path="/620E795B/68ABBB53" Ref="#PWR0279"  Part="1"
-F 0 "#PWR0279" H 7650 1500 50  0001 C CNN
-F 1 "+3.3V" V 7650 1875 50  0000 C CNN
-F 2 "" H 7650 1650 60  0000 C CNN
-F 3 "" H 7650 1650 60  0000 C CNN
-	1    7650 1650
+F 0 "#PWR0279" H 7750 1500 50  0001 C CNN
+F 1 "+3.3V" V 7750 1875 50  0000 C CNN
+F 2 "" H 7750 1650 60  0000 C CNN
+F 3 "" H 7750 1650 60  0000 C CNN
+	1    7750 1650
 	-1   0    0    -1
 $EndComp
@@
 L S3-OLinuXino_Rev_A:+3.3V #PWR?
 U 1 1 68AC8602
-P 7350 1650
+P 7450 1650
 AR Path="/5D8A1FAC/68AC8602" Ref="#PWR?"  Part="1"
 AR Path="/68AC8602" Ref="#PWR?"  Part="1"
 AR Path="/620E795B/68AC8602" Ref="#PWR0280"  Part="1"
-F 0 "#PWR0280" H 7350 1500 50  0001 C CNN
-F 1 "+3.3V" V 7350 1875 50  0000 C CNN
-F 2 "" H 7350 1650 60  0000 C CNN
-F 3 "" H 7350 1650 60  0000 C CNN
-	1    7350 1650
+F 0 "#PWR0280" H 7450 1500 50  0001 C CNN
+F 1 "+3.3V" V 7450 1875 50  0000 C CNN
+F 2 "" H 7450 1650 60  0000 C CNN
+F 3 "" H 7450 1650 60  0000 C CNN
+	1    7450 1650
 	-1   0    0    -1
 $EndComp
@@
 	4100 4000 4900 4000
 Wire Wire Line
-	7750 1200 7750 1350
-Wire Wire Line
-	7750 1550 7750 1650
+	7650 1200 7650 1350
+Wire Wire Line
+	7650 1550 7650 1650
 Wire Wire Line
 	4100 4100 4900 4100
 Wire Wire Line
-	7450 1550 7450 1650
-Wire Wire Line
-	7450 1350 7450 1200
+	7350 1550 7350 1650
+Wire Wire Line
+	7350 1350 7350 1200
 $EndSCHEMATC

Commit message: fixed ETH cur ref
Connections:
- net +3.3V_RTC: no longer R89.1
- net GND: now also R89.1
Changed lines of the file:
@@
 Wire Wire Line
 	4550 4400 5950 4400
-$Comp
-L S3-OLinuXino_Rev_A:+3.3V_RTC #PWR?
-U 1 1 68A599A9
-P 5100 4200
-AR Path="/5D8A1FAC/68A599A9" Ref="#PWR?"  Part="1"
-AR Path="/68A599A9" Ref="#PWR?"  Part="1"
-AR Path="/620E795B/68A599A9" Ref="#PWR0278"  Part="1"
-F 0 "#PWR0278" H 5100 3900 60  0001 C CNN
-F 1 "+3.3V_RTC" V 5115 4328 50  0000 L CNN
-F 2 "" H 5100 4200 60  0001 C CNN
-F 3 "" H 5100 4200 60  0001 C CNN
-	1    5100 4200
-	0    1    1    0
-$EndComp
 Wire Wire Line
 	5950 4350 5950 4400
@@
 Wire Wire Line
 	7350 1350 7350 1200
+$Comp
+L S3-OLinuXino_Rev_A:GND #PWR?
+U 1 1 60388407
+P 5100 4200
+AR Path="/5D8A1FAC/60388407" Ref="#PWR?"  Part="1"
+AR Path="/60388407" Ref="#PWR?"  Part="1"
+AR Path="/620E795B/60388407" Ref="#PWR?"  Part="1"
+F 0 "#PWR?" H 5100 3950 50  0001 C CNN
+F 1 "GND" V 5105 4072 50  0000 R CNN
+F 2 "" H 5100 4200 60  0000 C CNN
+F 3 "" H 5100 4200 60  0000 C CNN
+	1    5100 4200
+	0    -1   1    0
+$EndComp
 $EndSCHEMATC

Commit message: beautify kicad project
Connections:
- net +1.1V renamed +1V1
- net AP-CK32KO renamed AP_CK32KO
- net MIPI-CK_N renamed MIPI_CK_N
- net MIPI-CK_P renamed MIPI_CK_P
- net MIPI-D0_N renamed MIPI_D0_N
- net MIPI-D0_P renamed MIPI_D0_P
- net MIPI-D1_N renamed MIPI_D1_N
- net MIPI-D1_P renamed MIPI_D1_P
- net MIPI-D2_N renamed MIPI_D2_N
- net MIPI-D2_P renamed MIPI_D2_P
- net MIPI-D3_N renamed MIPI_D3_N
- net MIPI-D3_P renamed MIPI_D3_P
- net USB-D_N renamed USB_D_N
- net USB-D_P renamed USB_D_P
Other:
- moved on the sheet: C100, C101, C102, C103, C104, C82, C83, C88, J8, R79, R80, R87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
