File: Power.sch (KiCad schematic (older format))
At the start: 90 parts

Commit message: update
Parts:
- removed C?: 10uF/6.3V/20%/X5R/C0603, OLIMEX_RLC-FP:C_0603_5MIL_DWS, symbol S3-OLinuXino_Rev_A:C
- removed C?: 47uF/6.3V/20%/X5R/C0805, OLIMEX_RLC-FP:C_0805_5MIL_DWS, symbol S3-OLinuXino_Rev_A:C
- removed D? (x2): 1N5822/SS34/SMA, OLIMEX_Diodes-FP:SMA-KA, symbol S3-OLinuXino_Rev_A:D_Schottky
- removed FET?: IRLML6402(SOT-23), OLIMEX_Transistors-FP:SOT23, symbol S3-OLinuXino_Rev_A:P-MOS+DIOD
- removed L?: 2.2uH/4.5A/28mR/20%/CD75/7.8x7.0x5.0mm(YS75-2R2M), OLIMEX_RLC-FP:YS75_7X8MM, symbol S3-OLinuXino_Rev_A:L
- removed PWRLED?: LED\\Red\\0603, OLIMEX_LEDs-FP:LED_0603_KA, symbol S3-OLinuXino_Rev_A:LED
- removed R?: 2.2k/R0402, OLIMEX_RLC-FP:R_0402_5MIL_DWS, symbol S3-OLinuXino_Rev_A:R
- removed R?: 1.1k/1%/R0402, OLIMEX_RLC-FP:R_0402_5MIL_DWS, symbol S3-OLinuXino_Rev_A:R
- removed R?: 8.25k/1%/R0402, OLIMEX_RLC-FP:R_0402_5MIL_DWS, symbol S3-OLinuXino_Rev_A:R
- removed R?: 10k/R0402, OLIMEX_RLC-FP:R_0402_5MIL_DWS, symbol S3-OLinuXino_Rev_A:R
- removed U?: MT3608(SOT23-6), OLIMEX_IC-FP:SOT23-6, symbol S3-OLinuXino_Rev_A:MT3608(SOT23-6)
- added D?: LED, symbol Device:LED
- added R?: 5k1, otter:C_0402, symbol Device:R_Small
- added R? (x2): DNP, otter:C_0402, symbol Device:R_Small
- J?: value USB_C_Receptacle_USB2.0 -> USB
Connections:
- net labels removed: +5V_EXT
- wire segments 362 -> 326
- no-connect marks 6 -> 8
Other:
- note removed: "DELETE?\nMacht 5V ext aus batt"
- note removed: "Ra"
- note removed: "Rb"
- note removed: "Vout=0.6*(1+Ra\Rb)"
- moved on the sheet: C?, J?, L?, R?, U?

Commit message: update
Parts:
- gave numbers to parts that had none: 82
Other:
- note added: "USB Power in"
- moved on the sheet: C30, C31, C32, C33, C34, C35, C36, C37, C38, C39, C40, C41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

Commit message: update
Parts:
- D3: renamed from D4; footprint (none) -> otter:LED_0603_1608Metric
- D4: renamed from D3; footprint (none) -> Diode_SMD:D_SMB
- J3: footprint (none) -> otter:USB-C 16Pin
- J4: footprint (none) -> Connector_PinHeader_2.00mm:PinHeader_1x04_P2.00mm_Vertical
- L1, L2, L3, L4: footprint (none) -> Inductor_SMD:L_Taiyo-Yuden_MD-3030
- Q1: footprint (none) -> Package_TO_SOT_SMD:SOT-23
- SW1, SW2: footprint (none) -> Button_Switch_SMD:SW_SPST_PTS810
- U1: footprint OLIMEX_IC-FP:FBGA-234(Pitch-0.65mm_Pad-0.3mm_11x11x1.08mm) -> otter:FBGA-234(Pitch-0.65mm_Pad-0.3mm_11x11x1.08mm)
- U3: footprint OLIMEX_IC-FP:QFN48-6x6mm-OLIMEX_V2 -> otter:QFN-48-1EP_6x6mm_P0.4mm_EP4.05x4.05mm
- U4: footprint OLIMEX_Regulators-FP:SOT-23-5 -> Package_TO_SOT_SMD:SOT-23-5
- U5: footprint (none) -> Package_TO_SOT_SMD:SOT-23-5
Changed lines of the file:
@@
 F 0 "U4" H 7550 8350 50  0000 C CNN
 F 1 "SY8089AAAC" H 7550 7850 39  0000 C CNN
-F 2 "OLIMEX_Regulators-FP:SOT-23-5" H 7580 8250 20  0001 C CNN
+F 2 "Package_TO_SOT_SMD:SOT-23-5" H 7580 8250 20  0001 C CNN
 F 3 "" H 7550 8100 60  0000 C CNN
 F 4 "Value 1" H 7550 8100 60  0001 C CNN "Fieldname 1"
@@
 F 0 "L3" V 4735 3150 50  0000 C CNN
 F 1 "2.2uH" V 4644 3150 50  0000 C CNN
-F 2 "" H 4550 3150 50  0001 C CNN
+F 2 "Inductor_SMD:L_Taiyo-Yuden_MD-3030" H 4550 3150 50  0001 C CNN
 F 3 "~" H 4550 3150 50  0001 C CNN
 	1    4550 3150
@@
 F 0 "L2" V 4735 2550 50  0000 C CNN
 F 1 "2.2uH" V 4644 2550 50  0000 C CNN
-F 2 "" H 4550 2550 50  0001 C CNN
+F 2 "Inductor_SMD:L_Taiyo-Yuden_MD-3030" H 4550 2550 50  0001 C CNN
 F 3 "~" H 4550 2550 50  0001 C CNN
 	1    4550 2550
@@
 F 0 "L1" V 4650 1950 50  0000 C CNN
 F 1 "2.2uH" V 4500 1950 50  0000 C CNN
-F 2 "" H 4550 1950 50  0001 C CNN
+F 2 "Inductor_SMD:L_Taiyo-Yuden_MD-3030" H 4550 1950 50  0001 C CNN
 F 3 "~" H 4550 1950 50  0001 C CNN
 	1    4550 1950
@@
 F 0 "Q1" H 2750 5200 50  0000 L CNN
 F 1 "DTA114YKA" H 2550 5400 50  0000 L CNN
-F 2 "" H 3100 5300 50  0001 C CNN
+F 2 "Package_TO_SOT_SMD:SOT-23" H 3100 5300 50  0001 C CNN
 F 3 "~" H 3100 5300 50  0001 C CNN
 	1    3100 5300
@@
 F 0 "SW2" H 1850 5350 50  0000 C CNN
 F 1 "RST" H 2250 5350 50  0000 C CNN
-F 2 "" H 2050 5500 50  0001 C CNN
+F 2 "Button_Switch_SMD:SW_SPST_PTS810" H 2050 5500 50  0001 C CNN
 F 3 "~" H 2050 5500 50  0001 C CNN
 	1    2050 5300
@@
 	1800 2350 1850 2350
 $Comp
-L Device:D_TVS D3
+L Device:D_TVS D4
 U 1 1 66BA7290
 P 1850 2100
-F 0 "D3" V 1804 2179 50  0000 L CNN
+F 0 "D4" V 1804 2179 50  0000 L CNN
 F 1 "P6SMB6.8CA" V 1895 2179 50  0000 L CNN
-F 2 "" H 1850 2100 50  0001 C CNN
+F 2 "Diode_SMD:D_SMB" H 1850 2100 50  0001 C CNN
 F 3 "~" H 1850 2100 50  0001 C CNN
 	1    1850 2100
@@
 F 0 "SW1" H 1850 5000 50  0000 C CNN
 F 1 "PWRON" H 2300 5000 50  0000 C CNN
-F 2 "" H 2050 5150 50  0001 C CNN
+F 2 "Button_Switch_SMD:SW_SPST_PTS810" H 2050 5150 50  0001 C CNN
 F 3 "~" H 2050 5150 50  0001 C CNN
 	1    2050 4950
@@
 F 0 "L4" V 8100 8000 50  0000 C CNN
 F 1 "2.2uH" V 7950 8000 50  0000 C CNN
-F 2 "" H 8000 8000 50  0001 C CNN
+F 2 "Inductor_SMD:L_Taiyo-Yuden_MD-3030" H 8000 8000 50  0001 C CNN
 F 3 "~" H 8000 8000 50  0001 C CNN
 	1    8000 8000
@@
 F 0 "U3" H 3850 6115 50  0000 C CNN
 F 1 "AXP209(QFN-48)" H 3850 6024 50  0000 C CNN
-F 2 "OLIMEX_IC-FP:QFN48-6x6mm-OLIMEX_V2" H 3850 850 50  0001 C CNN
+F 2 "otter:QFN-48-1EP_6x6mm_P0.4mm_EP4.05x4.05mm" H 3850 850 50  0001 C CNN
 F 3 "http://dl.linux-sunxi.org/AXP/AXP209_Datasheet_v1.0en.pdf" H 3850 750 50  0001 C CNN
 	1    3850 3550
@@
 F 0 "U1" H 12750 5581 50  0000 C CNN
 F 1 "AllWinner-S3(FBGA-234)" H 12750 5490 50  0000 C CNN
-F 2 "OLIMEX_IC-FP:FBGA-234(Pitch-0.65mm_Pad-0.3mm_11x11x1.08mm)" H 12750 1850 50  0001 C CNN
+F 2 "otter:FBGA-234(Pitch-0.65mm_Pad-0.3mm_11x11x1.08mm)" H 12750 1850 50  0001 C CNN
 F 3 "" H 12950 5600 50  0001 C CNN
 	4    12750 3900
@@
 F 0 "U5" H 11850 8475 50  0000 C CNN
 F 1 "SY6280AAC" H 11850 8384 50  0000 C CNN
-F 2 "" H 11850 8100 50  0001 C CNN
+F 2 "Package_TO_SOT_SMD:SOT-23-5" H 11850 8100 50  0001 C CNN
 F 3 "" H 11850 8100 50  0001 C CNN
 	1    11850 8100
@@
 F 0 "J4" H 14330 8042 50  0000 L CNN
 F 1 "OTG" H 14330 7951 50  0000 L CNN
-F 2 "" H 14250 8050 50  0001 C CNN
+F 2 "Connector_PinHeader_2.00mm:PinHeader_1x04_P2.00mm_Vertical" H 14250 8050 50  0001 C CNN
 F 3 "~" H 14250 8050 50  0001 C CNN
 	1    14250 8050
@@
 F 0 "J3" H 2907 9067 50  0000 C CNN
 F 1 "USB" H 2907 8976 50  0000 C CNN
-F 2 "" H 2950 8200 50  0001 C CNN
+F 2 "otter:USB-C 16Pin" H 2950 8200 50  0001 C CNN
 F 3 "https://www.usb.org/sites/default/files/documents/usb_type-c.zip" H 2950 8200 50  0001 C CNN
 	1    2800 8200
@@
 P 1850 8300
 AR Path="/5FC342C2" Ref="D?"  Part="1"
-AR Path="/602ACDF9/5FC342C2" Ref="D4"  Part="1"
-F 0 "D4" V 1889 8183 50  0000 R CNN
+AR Path="/602ACDF9/5FC342C2" Ref="D3"  Part="1"
+F 0 "D3" V 1889 8183 50  0000 R CNN
 F 1 "LED" V 1798 8183 50  0000 R CNN
-F 2 "" H 1850 8300 50  0001 C CNN
+F 2 "otter:LED_0603_1608Metric" H 1850 8300 50  0001 C CNN
 F 3 "~" H 1850 8300 50  0001 C CNN
 	1    1850 8300

Commit message: update
Parts:
- removed L4: 2.2uH, Inductor_SMD:L_Taiyo-Yuden_MD-3030, symbol Device:L_Small
- removed R27: R03, Resistor_SMD:R_1206_3216Metric, symbol Device:R_Small
- C15, C21: value 10u -> 100n; footprint otter:C_0603 -> otter:C_0402
- C18: value 2.2u -> 100n; footprint otter:C_0603 -> otter:C_0402
- D3: footprint otter:LED_0603_1608Metric -> LED_SMD:LED_0603_1608Metric_Castellated
- L1, L2, L3: LCSC (none) -> C167747
Connections:
- net VBAT is gone; now on an unnamed net: U3.38 (BAT)
- net +1.1V: now also C18.1
- net +3V3: now also C21.1, L1.2; no longer L3.2
- net GND: now also C12.2, C18.2; no longer C12.1
- net VCC-DDR: now also L3.2
- net at U4.3 (LX): now also L3.1
- net at U3.15 (LX3): now also L1.1; no longer L3.1
- net at U3.45 (LX1): no longer L1.1
- net at U3.39 (BAT), U3.42 (BATSENSE): now also C15.1; no longer C18.2, C21.1
- net AXP_PWRON: no longer names the net of SW1.2, U3.47 (PWRON)
- net AXP_PWRON: now also C12.1; no longer C12.2
- net AXP_RST: no longer names the net of Q1.1 (B), SW2.2
- now unconnected: U3.43 (CHSENSE)
- no-connect marks 8 -> 10
Other:
- moved on the sheet: C12

Commit message: update
Connections:
- net +5V_USBOTG: now also J4.4 (Pin_4); no longer J4.1 (Pin_1)
- net GND: now also J4.1 (Pin_1); no longer J4.4 (Pin_4)
Changed lines of the file:
@@
 L Connector_Generic:Conn_01x04 J?
 U 1 1 67E47B05
-P 14250 8050
+P 14250 8150
 AR Path="/67E47B05" Ref="J?"  Part="1"
 AR Path="/602ACDF9/67E47B05" Ref="J4"  Part="1"
-F 0 "J4" H 14330 8042 50  0000 L CNN
-F 1 "OTG" H 14330 7951 50  0000 L CNN
-F 2 "Connector_PinHeader_2.00mm:PinHeader_1x04_P2.00mm_Vertical" H 14250 8050 50  0001 C CNN
-F 3 "~" H 14250 8050 50  0001 C CNN
-	1    14250 8050
-	1    0    0    -1
+F 0 "J4" H 14330 8142 50  0000 L CNN
+F 1 "OTG" H 14330 8051 50  0000 L CNN
+F 2 "Connector_PinHeader_2.00mm:PinHeader_1x04_P2.00mm_Vertical" H 14250 8150 50  0001 C CNN
+F 3 "~" H 14250 8150 50  0001 C CNN
+	1    14250 8150
+	1    0    0    1
 $EndComp
 $Comp
@@
 	-1   0    0    1
 $EndComp
+Text GLabel 14050 8150 0    50   Input ~ 0
+USB-D_N
 Text GLabel 14050 8050 0    50   Input ~ 0
-USB-D_N
-Text GLabel 14050 8150 0    50   Input ~ 0
 USB-D_P
 $Comp

Commit message: update
Parts:
- added D6: ESD5302F, Package_TO_SOT_SMD:SOT-23, symbol Power_Protection:SP0502BAHT
- J4: footprint Connector_PinHeader_2.00mm:PinHeader_1x04_P2.00mm_Vertical -> otter:PinHeader_1x04_P2.00mm_Vertical_nosilk_center
Connections:
- net +5V_USBOTG: now also D6.3 (A)
- net USB-D_N: now also J4.3 (Pin_3), D6.2 (K); no longer J4.2 (Pin_2)
- net USB-D_P: now also J4.2 (Pin_2), D6.1 (K); no longer J4.3 (Pin_3)
Changed lines of the file:
@@
 F 0 "J4" H 14330 8142 50  0000 L CNN
 F 1 "OTG" H 14330 8051 50  0000 L CNN
-F 2 "Connector_PinHeader_2.00mm:PinHeader_1x04_P2.00mm_Vertical" H 14250 8150 50  0001 C CNN
+F 2 "otter:PinHeader_1x04_P2.00mm_Vertical_nosilk_center" H 14250 8150 50  0001 C CNN
 F 3 "~" H 14250 8150 50  0001 C CNN
 	1    14250 8150
@@
 	-1   0    0    1
 $EndComp
+Text GLabel 14050 8050 0    50   Input ~ 0
+USB-D_N
 Text GLabel 14050 8150 0    50   Input ~ 0
-USB-D_N
-Text GLabel 14050 8050 0    50   Input ~ 0
 USB-D_P
 $Comp
@@
 Wire Wire Line
 	3500 8300 3400 8300
-Connection ~ 3400 8300
 Wire Wire Line
 	3400 8200 3500 8200
-Connection ~ 3400 8200
 Text Notes 2550 7250 0    50   ~ 0
 USB Power in
@@
 	5350 2550 5650 2550
 Connection ~ 5650 2750
+Text GLabel 10450 9900 0    50   Input ~ 0
+USB-D_N
+Text GLabel 10450 10100 0    50   Input ~ 0
+USB-D_P
+$Comp
+L Power_Protection:SP0502BAHT D6
+U 1 1 5FC7EF96
+P 10650 10000
+F 0 "D6" V 10992 10000 50  0000 C CNN
+F 1 "ESD5302F" V 10901 10000 50  0000 C CNN
+F 2 "Package_TO_SOT_SMD:SOT-23" H 10875 9950 50  0001 L CNN
+F 3 "http://www.littelfuse.com/~/media/files/littelfuse/technical%20resources/documents/data%20sheets/sp05xxba.pdf" H 10775 10125 50  0001 C CNN
+F 4 "C239643" V 10650 10000 50  0001 C CNN "LCSC"
+	1    10650 10000
+	0    -1   -1   0
+$EndComp
+$Comp
+L S3-OLinuXino_Rev_A:+5V_USBOTG #PWR?
+U 1 1 5FC176D0
+P 10850 10000
+AR Path="/5D8A1FAC/5FC176D0" Ref="#PWR?"  Part="1"
+AR Path="/5FC176D0" Ref="#PWR?"  Part="1"
+AR Path="/602ACDF9/5FC176D0" Ref="#PWR0110"  Part="1"
+F 0 "#PWR0110" H 10850 9850 50  0001 C CNN
+F 1 "+5V_USBOTG" V 10850 10150 50  0000 L CNN
+F 2 "" H 10850 10000 60  0000 C CNN
+F 3 "" H 10850 10000 60  0000 C CNN
+	1    10850 10000
+	0    1    1    0
+$EndComp
+Connection ~ 3400 8300
+Connection ~ 3400 8200
 $EndSCHEMATC

Commit message: update
Parts:
- removed R33: DNP, otter:C_0402, symbol Device:R_Small
Other:
- moved on the sheet: R34
Changed lines of the file:
@@
 	0    -1   -1   0
 $EndComp
-Connection ~ 11050 4800
-$Comp
-L S3-OLinuXino_Rev_A:+2.5V #PWR?
-U 1 1 612C27EA
-P 10600 4800
-AR Path="/5D8A1FAC/612C27EA" Ref="#PWR?"  Part="1"
-AR Path="/612C27EA" Ref="#PWR?"  Part="1"
-AR Path="/602ACDF9/612C27EA" Ref="#PWR0134"  Part="1"
-F 0 "#PWR0134" H 10600 4650 50  0001 C CNN
-F 1 "+2.5V" V 10600 4900 50  0000 L CNN
-F 2 "" H 10600 4800 60  0000 C CNN
-F 3 "" H 10600 4800 60  0000 C CNN
-	1    10600 4800
-	0    -1   -1   0
-$EndComp
-Wire Wire Line
-	11050 4800 10850 4800
 Wire Wire Line
 	11250 4500 11250 4400
@@
 Wire Wire Line
 	11250 4600 11250 4500
-Wire Wire Line
-	11050 4800 11450 4800
 $Comp
 L S3-OLinuXino_Rev_A:GND #PWR?
 U 1 1 612C281A
-P 10600 4950
+P 10550 4800
 AR Path="/5D8A1FAC/612C281A" Ref="#PWR?"  Part="1"
 AR Path="/612C281A" Ref="#PWR?"  Part="1"
 AR Path="/602ACDF9/612C281A" Ref="#PWR0135"  Part="1"
-F 0 "#PWR0135" H 10600 4700 50  0001 C CNN
-F 1 "GND" V 10605 4822 50  0000 R CNN
-F 2 "" H 10600 4950 60  0000 C CNN
-F 3 "" H 10600 4950 60  0000 C CNN
-	1    10600 4950
+F 0 "#PWR0135" H 10550 4550 50  0001 C CNN
+F 1 "GND" V 10555 4672 50  0000 R CNN
+F 2 "" H 10550 4800 60  0000 C CNN
+F 3 "" H 10550 4800 60  0000 C CNN
+	1    10550 4800
 	0    1    -1   0
 $EndComp
@@
 $Comp
 L Device:R_Small R?
-U 1 1 6467BD71
+U 1 1 646A8F8C
 P 10750 4800
-AR Path="/6467BD71" Ref="R?"  Part="1"
-AR Path="/602ACDF9/6467BD71" Ref="R33"  Part="1"
-F 0 "R33" V 10700 4650 50  0000 C CNN
-F 1 "DNP" V 10700 4950 50  0000 C CNN
+AR Path="/646A8F8C" Ref="R?"  Part="1"
+AR Path="/602ACDF9/646A8F8C" Ref="R34"  Part="1"
+F 0 "R34" V 10700 4650 50  0000 C CNN
+F 1 "22" V 10700 4950 50  0000 C CNN
 F 2 "otter:C_0402" H 10750 4800 50  0001 C CNN
 F 3 "~" H 10750 4800 50  0001 C CNN
@@
 	0    1    1    0
 $EndComp
-$Comp
-L Device:R_Small R?
-U 1 1 646A8F8C
-P 10750 4950
-AR Path="/646A8F8C" Ref="R?"  Part="1"
-AR Path="/602ACDF9/646A8F8C" Ref="R34"  Part="1"
-F 0 "R34" V 10700 4800 50  0000 C CNN
-F 1 "22" V 10700 5100 50  0000 C CNN
-F 2 "otter:C_0402" H 10750 4950 50  0001 C CNN
-F 3 "~" H 10750 4950 50  0001 C CNN
-	1    10750 4950
-	0    1    1    0
-$EndComp
-Wire Wire Line
-	11050 4800 11050 4950
-Wire Wire Line
-	10850 4950 11050 4950
-Wire Wire Line
-	10600 4800 10650 4800
-Wire Wire Line
-	10600 4950 10650 4950
 $Comp
 L S3-OLinuXino_Rev_A:IPS #PWR?
@@
 Connection ~ 3400 8300
 Connection ~ 3400 8200
+Wire Wire Line
+	10550 4800 10650 4800
+Wire Wire Line
+	10850 4800 11450 4800
 $EndSCHEMATC

Commit message: update
Parts:
- added SW3: RST, otter:SW_SPST_PTS810, symbol Switch:SW_Push
- SW1: value PWRON -> DNP; footprint Button_Switch_SMD:SW_SPST_PTS810 -> otter:SW_SPST_PTS810
- SW2: value RST -> DNP; footprint Button_Switch_SMD:SW_SPST_PTS810 -> otter:SW_SPST_PTS810
Connections:
- net GND: now also SW3.1
- net at Q1.1 (B), SW2.2: now also SW3.2
Other:
- moved on the sheet: SW2
Changed lines of the file:
@@
 L Switch:SW_Push SW2
 U 1 1 6637168B
-P 2050 5300
-F 0 "SW2" H 1850 5350 50  0000 C CNN
-F 1 "RST" H 2250 5350 50  0000 C CNN
-F 2 "Button_Switch_SMD:SW_SPST_PTS810" H 2050 5500 50  0001 C CNN
-F 3 "~" H 2050 5500 50  0001 C CNN
-	1    2050 5300
+P 1450 5250
+F 0 "SW2" H 1250 5300 50  0000 C CNN
+F 1 "DNP" H 1650 5300 50  0000 C CNN
+F 2 "otter:SW_SPST_PTS810" H 1450 5450 50  0001 C CNN
+F 3 "~" H 1450 5450 50  0001 C CNN
+	1    1450 5250
 	1    0    0    -1
 $EndComp
@@
 L S3-OLinuXino_Rev_A:GND #PWR?
 U 1 1 663B8CCA
-P 1800 5300
+P 1200 5250
 AR Path="/5D8A1FAC/663B8CCA" Ref="#PWR?"  Part="1"
 AR Path="/663B8CCA" Ref="#PWR?"  Part="1"
 AR Path="/602ACDF9/663B8CCA" Ref="#PWR0165"  Part="1"
-F 0 "#PWR0165" H 1800 5050 50  0001 C CNN
-F 1 "GND" V 1805 5172 50  0000 R CNN
-F 2 "" H 1800 5300 60  0000 C CNN
-F 3 "" H 1800 5300 60  0000 C CNN
-	1    1800 5300
+F 0 "#PWR0165" H 1200 5000 50  0001 C CNN
+F 1 "GND" V 1205 5122 50  0000 R CNN
+F 2 "" H 1200 5250 60  0000 C CNN
+F 3 "" H 1200 5250 60  0000 C CNN
+	1    1200 5250
 	0    1    -1   0
 $EndComp
 Wire Wire Line
-	1850 5300 1800 5300
+	1250 5250 1200 5250
 $Comp
 L Device:C_Small C?
@@
 P 2050 4950
 F 0 "SW1" H 1850 5000 50  0000 C CNN
-F 1 "PWRON" H 2300 5000 50  0000 C CNN
-F 2 "Button_Switch_SMD:SW_SPST_PTS810" H 2050 5150 50  0001 C CNN
+F 1 "DNP" H 2300 5000 50  0000 C CNN
+F 2 "otter:SW_SPST_PTS810" H 2050 5150 50  0001 C CNN
 F 3 "~" H 2050 5150 50  0001 C CNN
 	1    2050 4950
@@
 $EndComp
 Wire Wire Line
-	2250 5300 2750 5300
-Wire Wire Line
 	2150 5100 2350 5100
 Wire Wire Line
@@
 Wire Wire Line
 	10850 4800 11450 4800
+$Comp
+L Switch:SW_Push SW3
+U 1 1 601100C1
+P 1450 5400
+F 0 "SW3" H 1250 5450 50  0000 C CNN
+F 1 "RST" H 1650 5450 50  0000 C CNN
+F 2 "otter:SW_SPST_PTS810" H 1450 5600 50  0001 C CNN
+F 3 "~" H 1450 5600 50  0001 C CNN
+	1    1450 5400
+	1    0    0    -1
+$EndComp
+$Comp
+L S3-OLinuXino_Rev_A:GND #PWR?
+U 1 1 60166E26
+P 1200 5400
+AR Path="/5D8A1FAC/60166E26" Ref="#PWR?"  Part="1"
+AR Path="/60166E26" Ref="#PWR?"  Part="1"
+AR Path="/602ACDF9/60166E26" Ref="#PWR0134"  Part="1"
+F 0 "#PWR0134" H 1200 5150 50  0001 C CNN
+F 1 "GND" V 1205 5272 50  0000 R CNN
+F 2 "" H 1200 5400 60  0000 C CNN
+F 3 "" H 1200 5400 60  0000 C CNN
+	1    1200 5400
+	0    1    -1   0
+$EndComp
+Wire Wire Line
+	1200 5400 1250 5400
+Wire Wire Line
+	1800 5300 1800 5250
+Wire Wire Line
+	1800 5250 1650 5250
+Wire Wire Line
+	1800 5300 2750 5300
+Wire Wire Line
+	1650 5400 1800 5400
+Wire Wire Line
+	1800 5400 1800 5300
+Connection ~ 1800 5300
 $EndSCHEMATC
