File: Power.sch (KiCad schematic (older format))
At the start: 78 parts, among them J3 USB, J4 OTG, Q1 DTA114YKA, SW3 RST, U1 AllWinner-S3(FBGA-234), U3 AXP209(QFN-48), U4 SY8089AAAC, U5 SY6280AAC

Commit message: finalized v2.1, ordered boards
Parts:
- R17, R28: value 2.2k -> 2k2
- R30: value 5.1k -> 5k1
- R31: value 3.3k -> 3k3
Changed lines of the file:
@@
 AR Path="/602ACDF9/65DF1730" Ref="R28"  Part="1"
 F 0 "R28" V 5350 5600 50  0000 C CNN
-F 1 "2.2k" V 5350 5950 50  0000 C CNN
+F 1 "2k2" V 5350 5950 50  0000 C CNN
 F 2 "otter:R_0402" H 5400 5750 50  0001 C CNN
 F 3 "~" H 5400 5750 50  0001 C CNN
@@
 AR Path="/602ACDF9/67669AFD" Ref="R30"  Part="1"
 F 0 "R30" H 8209 8196 50  0000 L CNN
-F 1 "5.1k" H 8209 8105 50  0000 L CNN
+F 1 "5k1" H 8209 8105 50  0000 L CNN
 F 2 "otter:R_0402" H 8150 8150 50  0001 C CNN
 F 3 "~" H 8150 8150 50  0001 C CNN
@@
 AR Path="/602ACDF9/6768CD43" Ref="R31"  Part="1"
 F 0 "R31" H 8209 8496 50  0000 L CNN
-F 1 "3.3k" H 8209 8405 50  0000 L CNN
+F 1 "3k3" H 8209 8405 50  0000 L CNN
 F 2 "otter:R_0402" H 8150 8450 50  0001 C CNN
 F 3 "~" H 8150 8450 50  0001 C CNN
@@
 AR Path="/602ACDF9/6629AA02" Ref="R17"  Part="1"
 F 0 "R17" V 2000 5400 50  0000 C CNN
-F 1 "2.2k" V 2000 5750 50  0000 C CNN
+F 1 "2k2" V 2000 5750 50  0000 C CNN
 F 2 "otter:R_0402" H 2050 5550 50  0001 C CNN
 F 3 "~" H 2050 5550 50  0001 C CNN

Commit message: broken links
Parts:
- U4: symbol S3-OLinuXino_Rev_A:SY8009AAAC(SOT23-5) -> OtterCastAudioV2-rescue:SY8009AAAC(SOT23-5)-S3-OLinuXino_Rev_A

Commit message: beautify kicad project
Parts:
- U4: symbol OtterCastAudioV2-rescue:SY8009AAAC(SOT23-5)-S3-OLinuXino_Rev_A -> otter:SY8009AAAC(SOT23-5)
Connections:
- net +1.1V renamed +1V1
- net +2.5V renamed +2V5
- net GPIO-RST renamed GPIO_RST
- net MIPI-SCK renamed MIPI_SCK
- net MIPI-SDA renamed MIPI_SDA
- net USB-DRV renamed USB_DRV
- net USB-D_N renamed USB_D_N
- net USB-D_P renamed USB_D_P
- net USB-ID renamed USB_ID
- net USB-VBUSDET renamed USB_VBUSDET
