File: OtterCastAudioV2.kicad_pcb (KiCad board)
At the start: 2 copper layers, 50 x 49.3 mm, 232 parts, among them J1 UART, J2 SD, J3 USB, J4 OTG, J5 PJ-3270, J6 PJ-3270, J7 PJ-3270, J8 ARJP11A-MASA-B-A-EMU2, J9 MIPI, Q1 DTA114YKA, SW1 PWRON, SW2 RST, U1 AllWinner-S3(FBGA-234), U2 AT24CS16-MAHM, U3 AXP209(QFN-48), U4 SY8089AAAC, U5 SY6280AAC, U6 SSM2603, U7 RTL8723BS, Y1 12.288Mhz, Y2 32.768kHz, Y3 24MHz

Commit message: update
Parts:
- C1, C3, J2: moved to B.Cu
- Y2: footprint otter:Oscillator_3225 -> Crystal:Crystal_SMD_3215-2Pin_3.2x1.5mm
- moved C101 158.2 mm to (45.4, 72.9)
- moved C80 158.2 mm to (51.4, 61.0)
- moved C83 158.2 mm to (42.9, 75.1)
- moved C91 158.2 mm to (43.6, 71.3)
- moved R78 158.2 mm to (58.7, 57.1)
- moved R80 158.2 mm to (46.0, 69.7)
- moved R81 158.2 mm to (43.6, 69.7)
- moved R86 158.2 mm to (61.2, 57.1)
- moved R89 158.2 mm to (46.0, 71.3)
- moved R92 158.2 mm to (42.9, 73.5)
- moved C100 158.2 mm to (40.5, 78.3)
- moved C102 158.2 mm to (59.0, 60.6)
- moved C103 158.2 mm to (51.6, 67.5)
- moved C104 158.2 mm to (45.7, 62.6)
- moved C79 158.2 mm to (43.9, 66.1)
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Connections:
- J4 pad 1: +5V_USBOTG -> GND
- J4 pad 4: GND -> +5V_USBOTG

Commit message: update
Parts:
- removed C3: 100n, otter:C_0402
- removed R53, R55, R56, R57: 22, otter:C_0402
- added D5: ESD5302F, Package_TO_SOT_SMD:SOT-23, F.Cu at (83.3, 87.7)
- added D6: ESD5302F, Package_TO_SOT_SMD:SOT-23, F.Cu at (100.0, 110.6)
- added NT1: NT, NetTie:NetTie-2_SMD_Pad0.5mm, F.Cu at (127.7, 87.0)
- AE1, C32, C33, C34, C35, C36, C37, C98, C99, U7: moved to B.Cu
- C1: value 100n -> 10u; footprint otter:C_0402 -> otter:C_0603
- J4: footprint Connector_PinHeader_2.00mm:PinHeader_1x04_P2.00mm_Vertical -> otter:PinHeader_1x04_P2.00mm_Vertical_nosilk_center
- Y2: footprint Crystal:Crystal_SMD_3215-2Pin_3.2x1.5mm -> otter:Crystal_SMD_3215-2Pin_3.2x1.5mm
- moved U7 200.7 mm to (88.5, 136.2)
- moved L3 192.9 mm to (92.7, 110.0)
- moved AE1 186.9 mm to (83.5, 113.8), turned to 40 degrees
- moved R48 152.7 mm to (107.5, 94.1), turned to 270 degrees
- moved R67 120.9 mm to (151.6, 81.0)
- moved R68 120.9 mm to (149.1, 81.0)
- moved C72 120.9 mm to (149.5, 76.3)
- moved C73 120.9 mm to (160.0, 77.8)
- moved C74 120.9 mm to (149.5, 79.1)
- moved C75 120.9 mm to (157.6, 77.8)
- moved C76 120.9 mm to (155.1, 77.8)
- moved C77 120.9 mm to (160.0, 76.2)
- moved C78 120.9 mm to (157.6, 76.2)
- moved L5 120.9 mm to (152.5, 76.4)
- moved R64 120.9 mm to (158.9, 81.0)
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Connections:
- J4 pad 2: USB-D_N -> USB-D_P
- J4 pad 3: USB-D_P -> USB-D_N
- U6 pad 10: Net-(R56-Pad1) -> BT-PCM-DIN
- U6 pad 15: GND -> GNDA
- U6 pad 19: GND -> GNDA
- U6 pad 7: Net-(R57-Pad1) -> BT-PCM-CLK
- U6 pad 8: Net-(R55-Pad1) -> BT-PCM-DOUT
- U6 pad 9: Net-(R53-Pad1) -> BT-PCM-SYNC

Commit message: update
Parts:
- removed C48, C49: 100n, otter:C_0402
- removed R85: 0, otter:C_0402
- C38, R94: moved to B.Cu
- U7: moved to F.Cu
- moved J9 72.4 mm to (95.4, 107.2)
- moved R60 70.6 mm to (99.4, 89.5)
- moved MK1 67.1 mm to (104.6, 93.0)
- moved R58 64.4 mm to (101.2, 89.5), turned to 180 degrees
- moved R42 63.6 mm to (103.0, 88.8), turned to 90 degrees
- moved C46 60.3 mm to (102.7, 90.7), turned to 270 degrees
- moved R63 54.5 mm to (113.2, 81.1), turned to 90 degrees
- moved C38 54.0 mm to (99.5, 103.9)
- moved C71 52.8 mm to (114.2, 81.1), turned to 90 degrees
- moved C69 52.7 mm to (108.8, 91.8), turned to 180 degrees
- moved R46 52.4 mm to (109.6, 93.2)
- moved C47 51.0 mm to (107.8, 93.2), turned to 180 degrees
- moved R39 50.0 mm to (103.2, 97.4), turned to 90 degrees
- moved FB3 47.6 mm to (114.1, 86.3), turned to 180 degrees
- moved C61 47.5 mm to (113.4, 89.3), turned to 180 degrees
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Connections:
- U1 pad P4: Net-(R85-Pad2) -> Net-(C94-Pad1)

Commit message: update
Parts:
- removed C86: DNP, otter:C_0603
- C85, C89: moved to B.Cu
- moved C81 70.3 mm to (103.8, 97.5)
- moved C95 68.8 mm to (98.3, 107.6), turned to 270 degrees
- moved C87 67.9 mm to (103.8, 100.0)
- moved C79 67.0 mm to (103.8, 96.2)
- moved C92 66.6 mm to (99.6, 107.6), turned to 270 degrees
- moved C89 65.0 mm to (100.1, 101.6)
- moved C80 64.6 mm to (103.8, 98.8)
- moved C85 62.2 mm to (100.0, 100.2), turned to 90 degrees
- moved R83 56.0 mm to (90.8, 104.7), turned to 270 degrees
- moved R78 56.0 mm to (99.8, 95.2)
- moved R82 55.8 mm to (90.9, 102.8), turned to 90 degrees
- moved C102 36.2 mm to (24.9, 72.8)
- moved R87 34.8 mm to (23.3, 61.1)
- moved R89 23.9 mm to (24.9, 82.5)
- moved R88 20.6 mm to (20.1, 79.2)
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Other:
- net class Default: clearance 0.2 -> 0.11; trace_width 0.25 -> 0.127; via_dia 0.8 -> 0.6; via_drill 0.4 -> 0.3
- rule pad_to_mask_clearance: 0.051 -> 0
- rule trace_clearance: 0.2 -> 0.11
- rule trace_min: 0.2 -> 0.127
- rule via_min_drill: 0.3 -> 0.2
- rule via_min_size: 0.4 -> 0.45
- board text added: "Here be Otters"

Commit message: update
Parts:
- removed C80: 4.7u, otter:C_0603
- removed C81, C87: 10u, otter:C_0603
- removed C84, C91: 100n, otter:C_0402
- removed R33: DNP, otter:C_0402
- added C3: 100n, otter:C_0402, F.Cu at (103.6, 99.6)
- moved R76 86.6 mm to (76.2, 96.7), turned to 90 degrees
- moved R81 52.6 mm to (103.5, 97.9)
- moved C88 50.8 mm to (97.1, 107.3), turned to 270 degrees
- moved R86 49.6 mm to (100.6, 107.0), turned to 270 degrees
- moved R79 49.3 mm to (95.1, 107.3), turned to 270 degrees
- moved C83 48.2 mm to (96.3, 107.3), turned to 270 degrees
- moved R80 47.8 mm to (95.5, 107.3), turned to 270 degrees
- moved C82 45.7 mm to (94.8, 107.3), turned to 270 degrees
- moved C103 28.2 mm to (34.6, 72.5)
- moved R78 5.22 mm to (103.6, 98.8)
- moved R34 1.14 mm to (97.0, 109.3), turned to 270 degrees
- moved R82 0.50 mm to (91.0, 102.3)
Connections:
- net HPOUTL renamed Net-(U1-PadP13)
- net HPOUTR renamed Net-(U1-PadN13)
- net LINEINL renamed Net-(U1-PadR12)
- net LINEINR renamed Net-(U1-PadT12)
- net LINEOUTL renamed Net-(U1-PadR6)
- net LINEOUTR renamed Net-(U1-PadT6)
- net MBIAS renamed Net-(U1-PadP10)
- net MICIN1_N renamed Net-(U1-PadR10)
- net MICIN1_P renamed Net-(U1-PadT10)
- net MICIN3_N renamed Net-(U1-PadR9)
- net MICIN3_P renamed Net-(U1-PadP9)
- U1 pad N11: HPOUTFB -> Net-(U1-PadN11)
- U1 pad N12: HPOUTFB -> Net-(U1-PadN12)

Commit message: update
Parts:
- added SW3: RST, otter:SW_SPST_PTS810, F.Cu at (121.4, 101.9)
- J1: footprint Connector_PinHeader_2.00mm:PinHeader_1x04_P2.00mm_Vertical -> otter:PinHeader_1x04_P2.00mm_Vertical_nosilk_center
- L5: footprint Inductor_SMD:L_0402_1005Metric -> otter:L_0402
- SW1: value PWRON -> DNP; footprint Button_Switch_SMD:SW_SPST_PTS810 -> otter:SW_SPST_PTS810
- SW2: value RST -> DNP; footprint Button_Switch_SMD:SW_SPST_PTS810 -> otter:SW_SPST_PTS810
- moved C76 99.7 mm to (57.4, 97.5)
- moved R64 99.7 mm to (61.2, 100.7)
- moved R65 99.7 mm to (58.8, 100.7)
- moved R66 99.7 mm to (56.3, 100.7)
- moved R72 99.7 mm to (59.4, 99.1)
- moved R73 99.7 mm to (57.0, 99.1)
- moved R74 99.7 mm to (54.5, 99.1)
- moved R69 99.7 mm to (64.3, 99.1)
- moved R70 99.7 mm to (61.9, 99.1)
- moved R75 99.7 mm to (66.1, 100.7)
- moved R77 99.7 mm to (66.7, 98.6)
- moved R67 99.7 mm to (53.9, 100.7)
- moved R68 99.7 mm to (51.4, 100.7)
- moved C77 77.2 mm to (88.9, 106.3)
- moved D2 76.4 mm to (85.3, 90.2)
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Connections:
- J1 pad 2: UART1_TX -> UART1_RX
- J1 pad 3: UART1_RX -> UART1_TX
Other:
- board text added: "Design by Jan Henrik 2020"
- board text added: "OtterCast Audio V2"
- board text added: "Power"
- board text added: "RST"
- board text added: "Status"
- board text removed: "Here be Otters"

Commit message: update
Parts:
- removed C2: 100n, otter:C_0402
- moved J8 37.6 mm to (25.1, 92.3)
- moved R5 35.0 mm to (91.4, 92.5), turned to 0 degrees
- moved U2 34.9 mm to (94.3, 93.9), turned to 180 degrees
- moved R74 33.3 mm to (87.0, 106.8)
- moved R6 32.2 mm to (91.9, 93.8), turned to 90 degrees
- moved R73 31.2 mm to (87.5, 92.3), turned to 270 degrees
- moved R65 29.0 mm to (86.5, 92.3), turned to 270 degrees
- moved R1 26.9 mm to (90.7, 108.4), turned to 90 degrees
- moved R72 26.2 mm to (84.8, 92.3), turned to 270 degrees
- moved R64 25.9 mm to (85.7, 92.3), turned to 270 degrees
- moved FB1 25.2 mm to (80.3, 107.1)
- moved R68 25.1 mm to (76.5, 98.9)
- moved R75 24.9 mm to (90.8, 97.9), turned to 270 degrees
- moved R2 24.5 mm to (90.8, 99.5), turned to 270 degrees
- moved C76 23.5 mm to (80.2, 91.7)
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Routing:
- net Net-(C13-Pad1): track 0.00 -> 24.2 mm, vias 0 -> 2
- net +5V: track 0.00 -> 21.9 mm
- added copper zone on F.Cu, net GND
Other:
- copper layers 2 -> 4

Commit message: update
Parts:
- J8: value ARJP11A-MASA-B-A-EMU2 -> HR961160C; footprint Connector_RJ:RJ45_Abracon_ARJP11A-MA_Horizontal -> otter:HR961160C; moved to B.Cu
- moved J8 80.0 mm to (100.0, 120.3)
- moved C15 0.20 mm to (116.8, 110.3)
- moved C18 0.14 mm to (110.9, 106.0)
Routing:
- net IPS: track 0.00 -> 17.1 mm
- net /Power/PB6\TWI0-SCK: track 0.00 -> 5.10 mm
- net /Power/PB7\TWI0-SDA: track 0.00 -> 4.77 mm
- net Net-(L2-Pad1): track 0.00 -> 4.65 mm
- net Net-(C15-Pad1): track 0.00 -> 4.52 mm
- net +1V2: track 0.00 -> 2.47 mm
- net Net-(R15-Pad1): track 0.00 -> 2.18 mm
- net /Power/NMI: track 0.00 -> 1.50 mm
- net +1.1V: track 0.00 -> 1.43 mm
- net GND: track 0.00 -> 1.35 mm
- net Net-(C12-Pad1): track 0.00 -> 1.26 mm
