File: OtterCastAudioV2.kicad_pcb (KiCad board)
At the start: 4 copper layers, 50 x 49.3 mm, 221 parts, among them J1 UART, J2 SD, J3 USB, J4 OTG, J5 PJ-3270, J6 PJ-3270, J7 PJ-3270, J8 49F-1201GYD2NL, J9 MIPI, Q1 DTA114YKA, SW1 DNP, SW2 DNP, SW3 RST, U1 AllWinner-S3(FBGA-234), U2 AT24CS16-MAHM, U3 AXP209(QFN-48), U4 SY8089AAAC, U5 SY6280AAC, U6 SSM2603, U7 RTL8723BS, Y1 12.288Mhz, Y2 32.768kHz, Y3 24MHz

Commit message: update
Parts:
- removed C40: 10u, otter:C_0603
- C33, C34, C35, C36: moved to F.Cu
- moved C99 36.2 mm to (76.8, 131.5)
- moved C32 35.0 mm to (60.9, 100.5)
- moved C92 28.8 mm to (75.6, 123.7)
- moved C34 6.49 mm to (93.8, 107.4)
- moved C35 6.41 mm to (98.6, 94.6), turned to 90 degrees
- moved C33 5.51 mm to (99.5, 94.6), turned to 90 degrees
- moved C36 4.98 mm to (97.8, 94.6), turned to 90 degrees
- moved R13 1.28 mm to (90.5, 92.5), turned to 180 degrees
- moved R5 0.83 mm to (92.2, 92.5)
- moved R1 0.81 mm to (90.6, 108.8), turned to 90 degrees
- moved C41 0.48 mm to (92.3, 107.8)
- moved R12 0.45 mm to (82.0, 106.8)
- moved R89 0.38 mm to (102.9, 100.8)
- moved C82 0.33 mm to (94.7, 107.4)
- moved R79 0.33 mm to (95.5, 107.4)
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Connections:
- J8 pad 12: +3V3 -> Net-(J8-Pad12)
- R87 pad 1: EPHY_LINK_LED -> +3V3
- R87 pad 2: Net-(R87-Pad2) -> Net-(J8-Pad12)
- U1 pad K5: Net-(R87-Pad2) -> EPHY_LINK_LED
Routing:
- net +3V3: track 64.5 -> 124.6 mm, vias 17 -> 24
- net USB-VBUSDET: track 1.82 -> 16.2 mm, vias 0 -> 2
- net BT-UART-CTS: track 0.00 -> 8.43 mm
- net Net-(C4-Pad1): track 0.00 -> 7.89 mm, vias 0 -> 2
- net +1.1V: track 45.2 -> 37.4 mm, vias 12 -> 13
- net BT-UART-TX: track 0.00 -> 7.63 mm, vias 0 -> 2
- net BT-UART-RX: track 0.00 -> 7.50 mm, vias 0 -> 2
- net Net-(R82-Pad1): track 0.30 -> 7.61 mm, vias 1 -> 0
- net SDC0-CLK: track 0.30 -> 7.41 mm, vias 1 -> 2
- net SDC0-D3: track 0.30 -> 6.55 mm, vias 1 -> 2
- net SDC0-CMD: track 0.00 -> 6.03 mm, vias 0 -> 1
- net SDC0-D0: track 0.20 -> 5.96 mm, vias 1 -> 2
- net SDC0-D1: track 0.49 -> 5.58 mm, vias 1 -> 2
- net SDC0-D2: track 0.00 -> 4.79 mm, vias 0 -> 1
- net Net-(R83-Pad1): track 0.00 -> 4.75 mm
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
Commit message: update
Parts:
- removed C79: 10u, otter:C_0603
- R88: moved to B.Cu
- moved R88 53.7 mm to (115.1, 90.8), turned to 180 degrees
- moved R87 52.6 mm to (104.6, 96.2), turned to 90 degrees
- moved R93 49.1 mm to (105.9, 98.3), turned to 180 degrees
- moved C102 48.4 mm to (109.7, 96.3)
- moved R90 47.3 mm to (108.3, 98.0), turned to 180 degrees
- moved R91 45.7 mm to (108.3, 98.8), turned to 180 degrees
- moved R92 43.6 mm to (105.9, 97.4), turned to 180 degrees
- moved C103 40.9 mm to (109.4, 97.2)
- moved C100 40.1 mm to (107.7, 96.6)
- moved C101 39.5 mm to (104.6, 97.8), turned to 270 degrees
- moved R51 3.65 mm to (105.4, 96.2), turned to 90 degrees
- moved R50 3.36 mm to (106.3, 95.7), turned to 90 degrees
- moved C85 2.34 mm to (107.1, 99.8), turned to 270 degrees
- moved R49 1.62 mm to (107.5, 95.1)
- moved C90 0.97 mm to (105.3, 99.7), turned to 0 degrees
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Connections:
- J8 pad 10: +3V3 -> Net-(J8-Pad10)
- R50 pad 1: /Audio/MIPI-SDA -> MIPI-SDA
- R51 pad 1: /Audio/MIPI-SCK -> MIPI-SCK
- R88 pad 1: EPHY_SPD_LED -> +3V3
- R88 pad 2: Net-(R88-Pad2) -> Net-(J8-Pad10)
- U1 pad L5: Net-(R88-Pad2) -> EPHY_SPD_LED
- U6 pad 27: /Audio/MIPI-SDA -> MIPI-SDA
- U6 pad 28: /Audio/MIPI-SCK -> MIPI-SCK
Routing:
- net EPHY_RX_N: track 0.00 -> 27.7 mm, vias 0 -> 2
- net EPHY_RX_P: track 0.00 -> 27.3 mm, vias 0 -> 3
- net EPHY_TX_N: track 0.00 -> 22.9 mm, vias 0 -> 2
- net EPHY_TX_P: track 0.00 -> 22.6 mm, vias 0 -> 3
- net MIPI-SDA: track 0.00 -> 19.5 mm, vias 0 -> 2
- net MIPI-SCK: track 0.00 -> 19.4 mm, vias 0 -> 2
- net BT-WAKE-AP: track 0.00 -> 16.1 mm, vias 0 -> 2
- net +3.3V_RTC: track 42.6 -> 36.8 mm, vias 6 -> 5
- net /Audio/MIPI-SDA: track 4.90 -> 0.00 mm
- net Net-(C103-Pad2): track 0.00 -> 4.56 mm, vias 0 -> 1
- net /Audio/MIPI-SCK: track 4.50 -> 0.00 mm
- net Net-(C102-Pad2): track 0.00 -> 4.03 mm, vias 0 -> 1
- net GND: track 210.5 -> 206.6 mm, vias 121 -> 116
- net +3.0VA: track 95.6 -> 91.8 mm, vias 16 -> 14
- net Net-(R2-Pad1): track 0.00 -> 2.88 mm
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
Commit message: update
Parts:
- moved C95 1.68 mm to (100.2, 107.7)
- moved R86 1.60 mm to (99.2, 107.4)
- moved R9 0.70 mm to (76.8, 93.7)
- moved D1 0.60 mm to (85.7, 88.3)
- moved C77 0.54 mm to (89.2, 106.8)
- moved R76 0.53 mm to (76.9, 95.8), turned to 270 degrees
- moved R12 0.47 mm to (81.5, 106.8), turned to 180 degrees
- moved D2 0.46 mm to (85.7, 89.9)
- moved L5 0.33 mm to (90.5, 106.2)
- moved C37 0.30 mm to (92.5, 106.8)
- moved R1 0.24 mm to (90.4, 109.0)
- moved C75 0.20 mm to (89.7, 107.6)
- moved J9 0.17 mm to (95.4, 108.2)
Routing:
- net AP-CK32KO: track 3.19 -> 40.2 mm, vias 0 -> 2
- net SDC0-DET#: track 2.38 -> 39.3 mm, vias 2 -> 3
- net +3V3: track 125.1 -> 157.3 mm, vias 24 -> 25
- net SDC0-CMD: track 7.41 -> 34.6 mm, vias 2 -> 3
- net SDC0-D3: track 6.55 -> 33.4 mm, vias 2 -> 3
- net SDC0-D2: track 5.22 -> 31.4 mm, vias 2 -> 3
- net SDC0-CLK: track 7.41 -> 31.9 mm, vias 2 -> 3
- net SDC0-D0: track 5.96 -> 28.5 mm, vias 2 -> 3
- net SDC0-D1: track 5.58 -> 27.2 mm
- net BT-DIS-N: track 0.00 -> 14.2 mm
- net UART1_TX: track 0.00 -> 10.5 mm
- net UART1_RX: track 0.00 -> 9.36 mm
- net WL-SDIO-D0: track 1.26 -> 9.86 mm
- net GND: track 206.6 -> 213.2 mm, vias 116 -> 119
- net AP-WAKE-BT: track 0.00 -> 6.07 mm
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
Commit message: update
Parts:
- moved C89 0.20 mm to (97.3, 107.4)
- moved C83 0.17 mm to (96.5, 107.4)
Routing:
- net BT-WAKE-AP: track 16.4 -> 11.1 mm
- net BT-PCM-DOUT: track 0.00 -> 4.91 mm, vias 0 -> 2
- net +1.1V: track 39.4 -> 37.3 mm
- net GND: track 213.2 -> 214.8 mm
- net BT-PCM-CLK: track 0.30 -> 1.71 mm, vias 1 -> 2
- net +3.0VA: track 91.0 -> 91.8 mm
- net BT-PCM-DIN: track 0.46 -> 1.16 mm, vias 1 -> 2
- net Net-(C82-Pad1): track 4.94 -> 5.60 mm
- net BT-PCM-SYNC: track 1.93 -> 2.06 mm, vias 1 -> 2
- added copper zone on In2.Cu, net +1.1V

Commit message: update
Routing:
- net +3.0VA: track 91.8 -> 121.2 mm, vias 14 -> 15
- net BT-PCM-CLK: track 1.71 -> 20.7 mm
- net BT-PCM-DOUT: track 4.91 -> 23.4 mm
- net BT-PCM-SYNC: track 2.06 -> 20.1 mm
- net BT-PCM-DIN: track 1.16 -> 18.9 mm
- net GND: track 214.8 -> 216.2 mm, vias 119 -> 118

Commit message: update
Routing:
- net BT-PCM-SYNC: track 20.1 -> 48.6 mm, vias 2 -> 4
- net BT-PCM-CLK: track 20.7 -> 48.8 mm, vias 2 -> 4
- net BT-PCM-DIN: track 18.9 -> 46.6 mm, vias 2 -> 4
- net BT-PCM-DOUT: track 23.4 -> 51.0 mm, vias 2 -> 4
- net WL-SDIO-CLK: track 1.17 -> 19.7 mm, vias 1 -> 2
- net WL-SDIO-D1: track 2.35 -> 20.8 mm, vias 1 -> 2
- net WL-SDIO-D3: track 1.80 -> 18.9 mm, vias 1 -> 2
- net WL-SDIO-D2: track 1.56 -> 18.6 mm, vias 1 -> 2
- net WL-SDIO-D0: track 9.86 -> 23.8 mm, vias 0 -> 2
- net WL-SDIO-CMD: track 5.68 -> 18.8 mm, vias 0 -> 2
- net UART1_RX: track 9.36 -> 10.2 mm
- net BT-WAKE-AP: track 11.2 -> 11.8 mm
- net UART1_TX: track 10.5 -> 11.0 mm

Commit message: update
Parts:
- added C79: 10u, otter:C_0603, F.Cu at (67.1, 113.1)
- R88: moved to F.Cu
- moved C38 62.3 mm to (64.0, 102.8)
- moved C99 29.7 mm to (60.8, 106.4)
- moved C92 19.4 mm to (62.5, 109.3)
- moved R88 11.1 mm to (108.3, 99.7), turned to 0 degrees
Connections:
- J8 pad 10: Net-(J8-Pad10) -> +3V3
- J8 pad 11: EPHY_LINK_LED -> Net-(J8-Pad11)
- J8 pad 12: Net-(J8-Pad12) -> +3V3
- J8 pad 9: EPHY_SPD_LED -> Net-(J8-Pad9)
- R87 pad 1: +3V3 -> EPHY_LINK_LED
- R87 pad 2: Net-(J8-Pad12) -> Net-(J8-Pad11)
- R88 pad 1: +3V3 -> EPHY_SPD_LED
- R88 pad 2: Net-(J8-Pad10) -> Net-(J8-Pad9)
Routing:
- net MIC-DET: track 1.01 -> 30.3 mm, vias 1 -> 2
- net Net-(J8-Pad9): track 0.00 -> 28.8 mm, vias 0 -> 2
- net +3V3: track 157.3 -> 182.7 mm, vias 25 -> 26
- net GPIO_LED2: track 0.29 -> 18.9 mm, vias 1 -> 2
- net GPIO_LED1: track 0.30 -> 18.0 mm, vias 1 -> 2
- net UART1_RX: track 10.2 -> 27.0 mm, vias 0 -> 2
- net UART1_TX: track 11.0 -> 27.5 mm, vias 0 -> 2
- net EPHY_LINK_LED: track 0.32 -> 13.8 mm, vias 1 -> 3
- net EPHY_SPD_LED: track 0.30 -> 13.7 mm, vias 1 -> 3
- net WL-WAKE-AP: track 0.29 -> 12.8 mm, vias 1 -> 2
- net WL-PMU-EN: track 1.63 -> 12.7 mm, vias 0 -> 2
- net PB9\TWI1-SDA: track 2.77 -> 12.8 mm, vias 1 -> 2
- net PB8\TWI1-SCK: track 2.15 -> 11.4 mm, vias 1 -> 2
- net GND: track 216.5 -> 224.7 mm, vias 118 -> 122
- net Net-(J8-Pad11): track 0.00 -> 7.27 mm, vias 0 -> 2
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
Commit message: no drc error
Parts:
- removed C79: 10u, otter:C_0603
- removed C99: 100n, otter:C_0402
- removed J9: MIPI, otter:FH35C-25S
- removed NT1: NT, NetTie:NetTie-2_SMD_Pad0.5mm
- removed R94: 51, otter:C_0402
- added R27: 0R, otter:R_0805, F.Cu at (122.9, 94.5)
- C92: moved to B.Cu
- R1, R10, R11, R12, R13, R14, R15, R16, R17, R18, R19, R2, R20, R21, R22, R23, R24, R25, R26, R28, R29, R3, R30, R31, R32, R34, R35, R36, R37, R38, R39, R4, R40, R41, R42, R43, R44, R45, R46, R47, R48, R49, R5, R50, R51, R52, R54, R58, R59, R6, R60, R61, R62, R63, R64, R65, R66, R67, R68, R69, R7, R70, R71, R72, R73, R74, R75, R76, R77, R78, R79, R8, R80, R81, R82, R83, R84, R86, R87, R88, R89, R9, R90, R91, R92, R93: footprint otter:C_0402 -> otter:R_0402
- moved C92 35.2 mm to (96.3, 99.6), turned to 180 degrees
- moved C32 35.2 mm to (96.0, 100.6), turned to 180 degrees
- moved C38 34.7 mm to (98.6, 99.5), turned to 225 degrees
Routing:
- net +3.3V_RTC: track 35.5 -> 43.6 mm, vias 4 -> 5
- net Net-(C82-Pad1): track 5.60 -> 13.5 mm, vias 1 -> 2
- net GND: track 224.7 -> 231.7 mm, vias 122 -> 190
- net +1.1V: track 37.3 -> 40.3 mm
- net VCC-DDR: track 16.2 -> 18.8 mm
- net MIPI-SDA: track 19.6 -> 17.0 mm
- net +3V3: track 182.7 -> 183.7 mm
