File: OtterCastAudioV2.kicad_pcb (KiCad board)
At the start: 4 copper layers, 50 x 49.3 mm, 221 parts, among them J1 UART, J2 SD, J3 USB, J4 OTG, J5 PJ-3270, J6 PJ-3270, J7 PJ-3270, J8 49F-1201GYD2NL, Q1 DTA114YKA, SW1 DNP, SW2 DNP, SW3 RST, U1 AllWinner-S3(FBGA-234), U2 AT24CS16-MAHM, U3 AXP209(QFN-48), U4 SY8089AAAC, U5 SY6280AAC, U6 SSM2603, U7 AP6236, X1 26Mhz TCXO, Y1 12.288Mhz, Y2 32.768kHz, Y3 24MHz

Commit message: working on silkscreen
Parts:
- added G***: LOGO, otter:OtterCastAudioV2_silk_headphones, B.Cu at (96.7, 107.0)
- added G***: LOGO, otter:OtterCastAudioV2_silk_status, F.Cu at (81.8, 88.7)
- added G***: LOGO, otter:OtterCastAudioV2_silk_power, F.Cu at (81.8, 87.2)
- added G***: LOGO, otter:OtterCastAudioV2_silk_designby, F.Cu at (85.5, 116.2)
- added G***: LOGO, otter:OtterCastAudioV2_silk_3, F.Cu at (87.6, 112.5)
- added G***: LOGO, otter:OtterCastAudioV2_silk_2, F.Cu at (82.8, 112.3)
- added G***: LOGO, otter:OtterCastAudioV2_silk_1, F.Cu at (83.1, 109.5)
Routing:
- net Net-(J8-Pad9): track 28.8 -> 12.3 mm, vias 2 -> 1
- net GND: track 228.4 -> 235.4 mm, vias 198 -> 209
- net Net-(J8-Pad11): track 7.27 -> 5.49 mm
- net MIC-DET: track 35.7 -> 34.8 mm
- net WL-WAKE-AP: track 12.8 -> 13.5 mm
Other:
- board text removed: "Design by Jan Henrik 2020"
- board text removed: "OtterCast Audio V2"
- board text removed: "Power"
- board text removed: "Status"

Commit message: regenerated gerber
Routing:
- net GNDA: track 109.4 -> 110.7 mm

Commit message: fixed axp bug, fixed schematics, fixed eeprom
Parts:
- removed R5, R6: 2.2k, otter:R_0402
- removed U2: AT24CS16-MAHM, Package_DFN_QFN:DFN-8-1EP_3x2mm_P0.5mm_EP1.3x1.5mm
- added C79: 10u, otter:C_0603, F.Cu at (110.9, 150.8)
- added C99: 100n, otter:C_0402, F.Cu at (113.7, 150.7)
Connections:
- U1 pad M13: BT-PCM-DOUT -> BT-PCM-DIN
- U1 pad T15: BT-PCM-DIN -> BT-PCM-DOUT
- U3 pad 29: Net-(U3-Pad29) -> +3.3V_RTC
- X1 pad 1: GND -> Net-(X1-Pad1)
Routing:
- net PB9\TWI1-SDA: track 12.9 -> 0.00 mm, vias 2 -> 0
- net PB8\TWI1-SCK: track 11.4 -> 0.00 mm, vias 2 -> 0
- net +3V3: track 193.0 -> 189.3 mm
- net MIC-DET: track 35.3 -> 32.6 mm
- net GPIO_LED2: track 23.2 -> 20.6 mm
- net GPIO_LED1: track 20.2 -> 17.6 mm
- net UART1_TX: track 25.2 -> 23.8 mm
- net WL-PMU-EN: track 15.4 -> 14.2 mm
- net GND: track 235.4 -> 234.7 mm
- net +3.3V_RTC: track 43.6 -> 44.2 mm

Commit message: fixed ETH, added AGND plane to prevent Line-In Noise, optimized power
Parts:
- removed C79: 10u, otter:C_0603
- removed C99: 100n, otter:C_0402
- moved R54 0.75 mm to (119.8, 94.2)
Connections:
- J8 pad 10: +3V3 -> Net-(J8-Pad10)
- J8 pad 11: Net-(J8-Pad11) -> +3V3
- J8 pad 12: +3V3 -> Net-(J8-Pad12)
- J8 pad 9: Net-(J8-Pad9) -> +3V3
- R87 pad 2: Net-(J8-Pad11) -> Net-(J8-Pad12)
- R88 pad 2: Net-(J8-Pad9) -> Net-(J8-Pad10)
Routing:
- net GNDA: track 110.7 -> 45.2 mm, vias 5 -> 16
- net Net-(J8-Pad9): track 12.3 -> 0.00 mm, vias 1 -> 0
- net Net-(J8-Pad10): track 0.00 -> 10.4 mm, vias 0 -> 1
- net BT-PCM-DIN: track 47.1 -> 53.1 mm, vias 4 -> 5
- net Net-(J8-Pad11): track 5.49 -> 0.00 mm, vias 2 -> 0
- net Net-(J8-Pad12): track 0.00 -> 3.72 mm, vias 0 -> 1
- net BT-PCM-SYNC: track 48.7 -> 50.8 mm
- net BT-PCM-CLK: track 49.0 -> 47.5 mm
- net BT-PCM-DOUT: track 51.2 -> 49.8 mm
- net Net-(C55-Pad1): track 7.19 -> 8.09 mm
- net +3V3: track 189.3 -> 188.6 mm
- net Net-(R54-Pad1): track 1.79 -> 2.40 mm
- added copper zone on In1.Cu, net GNDA

Commit message: fixed ETH cur ref
Connections:
- R89 pad 1: +3.3V_RTC -> GND
Routing:
- net GND: track 234.5 -> 235.8 mm, vias 209 -> 210
Changed lines of the file:
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@@
     (thickness 1.6)
     (drawings 70)
-    (tracks 3255)
+    (tracks 3256)
     (zones 0)
     (modules 225)
@@
   )
   (setup
-    (last_trace_width 0.2)
+    (last_trace_width 0.127)
     (user_trace_width 0.127)
     (user_trace_width 0.2)
@@
       (net 154 "Net-(R89-Pad2)"))
     (pad 1 smd rect (at -0.47 0 270) (size 0.5 0.6) (layers F.Cu F.Paste F.Mask)
-      (net 14 +3.3V_RTC))
+      (net 1 GND))
     (model ${KISYS3DMOD}/Resistor_SMD.3dshapes/R_0402_1005Metric.step
       (at (xyz 0 0 0))
@@
   (gr_line (start 112.5 78.35) (end 105.5 78.35) (layer Edge.Cuts) (width 0.05))
   (gr_line (start 87.500001 78.35) (end 94.5 78.35) (layer Edge.Cuts) (width 0.05))
+  (via (at 102.88 100.61449) (size 0.45) (drill 0.2) (layers F.Cu B.Cu) (net 1))
   (via (at 108.4 117.05) (size 0.6) (drill 0.3) (layers F.Cu B.Cu) (net 1))
   (via (at 107.2 117.05) (size 0.6) (drill 0.3) (layers F.Cu B.Cu) (net 1))
@@
   (segment (start 116.9 111.2) (end 116.9 107.6) (width 0.127) (layer In1.Cu) (net 14))
   (segment (start 115 113.1) (end 116.9 111.2) (width 0.127) (layer In1.Cu) (net 14))
-  (segment (start 102.88 100.335) (end 102.88 99.55) (width 0.127) (layer F.Cu) (net 14))
-  (segment (start 102.9 100.355) (end 102.88 100.335) (width 0.127) (layer F.Cu) (net 14))
-  (segment (start 102.048501 100.779499) (end 102.473 100.355) (width 0.127) (layer F.Cu) (net 14))
-  (segment (start 101.228782 102.25) (end 102.048501 101.430281) (width 0.127) (layer F.Cu) (net 14))
-  (segment (start 99.975 102.375) (end 100.1 102.25) (width 0.127) (layer F.Cu) (net 14))
-  (segment (start 102.048501 101.430281) (end 102.048501 100.779499) (width 0.127) (layer F.Cu) (net 14))
-  (segment (start 100.1 102.25) (end 101.228782 102.25) (width 0.127) (layer F.Cu) (net 14))
-  (segment (start 102.473 100.355) (end 102.9 100.355) (width 0.127) (layer F.Cu) (net 14))
+  (segment (start 102.9 100.355) (end 102.88 100.335) (width 0.127) (layer F.Cu) (net 1))
+  (segment (start 103.82 99.6) (end 103.065 100.355) (width 0.127) (layer F.Cu) (net 1))
+  (segment (start 103.065 100.355) (end 102.9 100.355) (width 0.127) (layer F.Cu) (net 1))
+  (segment (start 103.82 99.55) (end 103.82 99.6) (width 0.127) (layer F.Cu) (net 1))
   (via (at 99.975 102.375) (size 0.45) (drill 0.2) (layers F.Cu B.Cu) (net 14))
   (segment (start 101.25 110.475) (end 99.375 108.6) (width 0.127) (layer In1.Cu) (net 14))
@@
   (segment (start 111.298 112.65) (end 111.65 112.65) (width 0.127) (layer F.Cu) (net 14))
   (segment (start 111.65 112.65) (end 114.55 112.65) (width 0.127) (layer F.Cu) (net 14))
+  (segment (start 102.337011 99.715989) (end 102.503 99.55) (width 0.127) (layer F.Cu) (net 14))
+  (segment (start 102.337011 101.141771) (end 102.337011 99.715989) (width 0.127) (layer F.Cu) (net 14))
+  (segment (start 101.228782 102.25) (end 102.337011 101.141771) (width 0.127) (layer F.Cu) (net 14))
+  (segment (start 100.1 102.25) (end 101.228782 102.25) (width 0.127) (layer F.Cu) (net 14))
+  (segment (start 99.975 102.375) (end 100.1 102.25) (width 0.127) (layer F.Cu) (net 14))
+  (segment (start 102.503 99.55) (end 102.88 99.55) (width 0.127) (layer F.Cu) (net 14))
   (segment (start 113.95 86.85) (end 113.95 85.55) (width 0.5) (layer F.Cu) (net 15))
   (via (at 113.95 86.85) (size 0.6) (drill 0.3) (layers F.Cu B.Cu) (net 15))
@@
   (segment (start 106.07 114.75) (end 106.32 114.5) (width 0.2) (layer F.Cu) (net 117))
   (via (at 102.125 106.825) (size 0.45) (drill 0.2) (layers F.Cu B.Cu) (net 117))
-  (segment (start 101.399839 100.949999) (end 101.427826 100.922012) (width 0.127) (layer F.Cu) (net 117))
-  (segment (start 101.427826 100.922012) (end 101.652825 100.697013) (width 0.127) (layer F.Cu) (net 117))
-  (segment (start 100.921219 100.949999) (end 101.399839 100.949999) (width 0.127) (layer F.Cu) (net 117))
-  (segment (start 100.751499 101.119719) (end 100.921219 100.949999) (width 0.127) (layer F.Cu) (net 117))
-  (segment (start 100.751499 101.598501) (end 100.751499 101.119719) (width 0.127) (layer F.Cu) (net 117))
-  (via (at 101.652825 100.697013) (size 0.45) (drill 0.2) (layers F.Cu B.Cu) (net 117))
-  (segment (start 100.425 101.925) (end 100.751499 101.598501) (width 0.127) (layer F.Cu) (net 117))
   (segment (start 102.125 106.825) (end 102.166488 106.866488) (width 0.127) (layer F.Cu) (net 117))
   (segment (start 102.1 112.637698) (end 102.25 112.487698) (width 0.127) (layer F.Cu) (net 117))
@@
   (segment (start 102.25 112.487698) (end 102.25 106.95) (width 0.127) (layer F.Cu) (net 117))
   (segment (start 106.07 114.75) (end 105.568501 114.248501) (width 0.127) (layer F.Cu) (net 117))
-  (segment (start 101.652825 101.015211) (end 101.652825 100.697013) (width 0.127) (layer In1.Cu) (net 117))
-  (segment (start 102.613499 104.933719) (end 102.475 104.79522) (width 0.127) (layer In1.Cu) (net 117))
-  (segment (start 102.475 103.2) (end 101.652825 102.377825) (width 0.127) (layer In1.Cu) (net 117))
-  (segment (start 101.652825 102.377825) (end 101.652825 101.015211) (width 0.127) (layer In1.Cu) (net 117))
-  (segment (start 102.475 104.79522) (end 102.475 103.2) (width 0.127) (layer In1.Cu) (net 117))
+  (segment (start 101.649991 101.015211) (end 101.649991 100.697013) (width 0.127) (layer In1.Cu) (net 117))
+  (segment (start 101.397005 100.949999) (end 101.424992 100.922012) (width 0.127) (layer F.Cu) (net 117))
+  (segment (start 100.921219 100.949999) (end 101.397005 100.949999) (width 0.127) (layer F.Cu) (net 117))
+  (segment (start 101.649991 103.970211) (end 101.649991 101.015211) (width 0.127) (layer In1.Cu) (net 117))
   (segment (start 102.613499 105.366281) (end 102.613499 104.933719) (width 0.127) (layer In1.Cu) (net 117))
-  (segment (start 102.125 105.85478) (end 102.613499 105.366281) (width 0.127) (layer In1.Cu) (net 117))
   (segment (start 102.125 106.825) (end 102.125 105.85478) (width 0.127) (layer In1.Cu) (net 117))
+  (segment (start 102.125 105.85478) (end 102.613499 105.366281) (width 0.127) (layer In1.Cu) (net 117))
+  (segment (start 101.424992 100.922012) (end 101.649991 100.697013) (width 0.127) (layer F.Cu) (net 117))
+  (segment (start 100.751499 101.119719) (end 100.921219 100.949999) (width 0.127) (layer F.Cu) (net 117))
+  (via (at 101.649991 100.697013) (size 0.45) (drill 0.2) (layers F.Cu B.Cu) (net 117))
+  (segment (start 100.751499 101.598501) (end 100.751499 101.119719) (width 0.127) (layer F.Cu) (net 117))
+  (segment (start 102.613499 104.933719) (end 101.649991 103.970211) (width 0.127) (layer In1.Cu) (net 117))
+  (segment (start 100.425 101.925) (end 100.751499 101.598501) (width 0.127) (layer F.Cu) (net 117))
   (segment (start 107.92 115.05) (end 108.83 115.05) (width 0.2) (layer F.Cu) (net 118))
   (segment (start 108.841998 115.05) (end 108.83 115.05) (width 0.2) (layer F.Cu) (net 118))
@@
   (segment (start 101.964489 99.235511) (end 102.09 99.11) (width 0.127) (layer F.Cu) (net 245))
   (segment (start 99.775 99.975) (end 100.098501 99.651499) (width 0.127) (layer F.Cu) (net 245))
-  (segment (start 106.673 98.978) (end 107.05 99.355) (width 0.127) (layer F.Cu) (net 246))
-  (segment (start 102.589698 98.978) (end 106.673 98.978) (width 0.127) (layer F.Cu) (net 246))
+  (segment (start 102.1 99.467698) (end 102.589698 98.978) (width 0.127) (layer F.Cu) (net 246))
   (segment (start 107.05 99.355) (end 107.1 99.355) (width 0.127) (layer F.Cu) (net 246))
-  (segment (start 102.44 99.127698) (end 102.589698 98.978) (width 0.127) (layer F.Cu) (net 246))
-  (segment (start 102.44 99.835) (end 102.44 99.127698) (width 0.127) (layer F.Cu) (net 246))
-  (segment (start 101.976499 100.298501) (end 102.44 99.835) (width 0.127) (layer F.Cu) (net 246))
-  (segment (start 99.451499 100.298501) (end 101.976499 100.298501) (width 0.127) (layer F.Cu) (net 246))
+  (segment (start 101.976499 100.298501) (end 102.1 100.175) (width 0.127) (layer F.Cu) (net 246))
   (segment (start 99.125 100.625) (end 99.451499 100.298501) (width 0.127) (layer F.Cu) (net 246))
+  (segment (start 106.673 98.978) (end 107.05 99.355) (width 0.127) (layer F.Cu) (net 246))
+  (segment (start 99.451499 100.298501) (end 101.976499 100.298501) (width 0.127) (layer F.Cu) (net 246))
+  (segment (start 102.589698 98.978) (end 106.673 98.978) (width 0.127) (layer F.Cu) (net 246))
+  (segment (start 102.1 100.175) (end 102.1 99.467698) (width 0.127) (layer F.Cu) (net 246))
   (segment (start 99.125 102.575) (end 99.1 102.575) (width 0.127) (layer F.Cu) (net 247))
   (segment (start 97.555 109.525) (end 97.55 109.52) (width 0.127) (layer F.Cu) (net 247))

Commit message: fixed axp rst, gpio rst, din, dout, eth
Parts:
- removed the G*** at (96.7, 107.0)
- removed SW1, SW2: DNP, otter:SW_SPST_PTS810
- added C2: 470n, otter:C_0402, F.Cu at (102.8, 112.0)
- added R6: DNP, otter:R_0402, F.Cu at (119.1, 104.1)
Connections:
- SW3 pad 2: Net-(Q1-Pad1) -> GPIO-RST
- U1 pad A2: Net-(U1-PadA2) -> GPIO-RST
Routing:
- net GPIO-RST: track 0.00 -> 54.7 mm, vias 0 -> 2
- net Net-(Q1-Pad1): track 13.9 -> 1.16 mm
- net Net-(C12-Pad1): track 11.6 -> 1.34 mm
- net GND: track 235.8 -> 227.9 mm
- net MIC-DET: track 32.6 -> 33.2 mm
- net RESETn: track 25.4 -> 25.9 mm
Other:
- board text added: "Amp- Out"
- board text added: "Line- In"
- board text added: "Line- Out"
- board text added: "by @FauthNiklas @Toble_Miner @Manawyrm @JanHenrikH"

Commit message: added gitignore, finished v2.1, exported gerber, moved 2.0 data
Parts:
- removed the G*** at (85.5, 116.2)
- removed the G*** at (87.6, 112.5)
- added G***: LOGO, otter:OtterCastAudioV2_silk_amp_out, B.Cu at (109.0, 84.5)
- added G***: LOGO, otter:OtterCastAudioV2_silk_line_out, B.Cu at (100.0, 81.5)
- added G***: LOGO, otter:OtterCastAudioV2_silk_line_in, B.Cu at (91.0, 84.4)
- added G***: LOGO, otter:OtterCastAudioV2_silk_by, B.Cu at (96.4, 107.8)
- added G***: LOGO, otter:OtterCastAudioV2_silk_4, F.Cu at (84.8, 115.3)
Other:
- board text removed: "Amp- Out"
- board text removed: "Line- In"
- board text removed: "Line- Out"
- board text removed: "by @FauthNiklas @Toble_Miner @Manawyrm @JanHenrikH"

Commit message: added i2c to axp209, fixed tvs diodes
Parts:
- removed R19, R20: 2.2k, otter:R_0402
- R2: value DNP -> 22
Connections:
- D5 pad 3: +3V3 -> GND
- D6 pad 3: +5V_USBOTG -> GND
- U3 pad 1: /Power/PB7\TWI0-SDA -> MIPI-SDA
- U3 pad 2: /Power/PB6\TWI0-SCK -> MIPI-SCK
Routing:
- net MIPI-SDA: track 17.0 -> 38.3 mm, vias 2 -> 4
- net MIPI-SCK: track 19.4 -> 40.5 mm, vias 2 -> 4
- net +3V3: track 188.6 -> 171.6 mm, vias 27 -> 25
- net GPIO-RST: track 54.7 -> 45.9 mm
- net /Power/PB6\TWI0-SCK: track 5.07 -> 0.00 mm
- net /Power/PB7\TWI0-SDA: track 4.80 -> 0.00 mm
- net GND: track 227.9 -> 231.0 mm, vias 210 -> 211
- net +5V_USBOTG: track 29.3 -> 28.5 mm, vias 4 -> 3
- net Net-(J5-Pad2): track 3.94 -> 4.65 mm
