File: Audio.sch (KiCad schematic (older format))
At the start: 34 parts

Commit message: update
Parts:
- added C? (x2): 18p, otter:C_0402, symbol Device:C_Small
- added C? (x6): 10u, otter:CP_EIA-3216-10, symbol Device:CP_Small
- added C? (x6): 100n, otter:C_0402, symbol Device:C_Small
- added C? (x2): 100u, otter:CP_EIA-3528-12, symbol Device:CP_Small
- added C? (x2): 220p, otter:C_0402, symbol Device:C_Small
- added FB? (x2): FERRET, otter:R_0805, symbol Device:Ferrite_Bead_Small
- added J?: TRS, symbol Connector:AudioJack3_Ground_SwitchTR
- added R? (x4): 2.2k, otter:C_0402, symbol Device:R_Small
- added R? (x5): 22, otter:C_0402, symbol Device:R_Small
- added R? (x4): 47k, otter:C_0402, symbol Device:R_Small
- added R? (x2): 100, otter:C_0402, symbol Device:R_Small
- added U?: SSM2603, symbol otter:SSM2603
- added Y?: 12.288Mhz, symbol Device:Crystal_GND24_Small
Connections:
- net labels added: +3.3V, +3V3, BT-PCM-CLK, BT-PCM-DIN, BT-PCM-DOUT, BT-PCM-SYNC, GNDA, MIPI-SCK, MIPI-SDA
- wire segments 98 -> 208
- no-connect marks 2 -> 5
Other:
- note added: "0x1B"

Commit message: update
Parts:
- removed C? (x10): 100nF/10V/10%/X7R/C0402, OLIMEX_RLC-FP:C_0402_5MIL_DWS, symbol S3-OLinuXino_Rev_A:C
- removed C? (x4): 33pF/50V/5%/COG/C0402, OLIMEX_RLC-FP:C_0402_5MIL_DWS, symbol S3-OLinuXino_Rev_A:C
- removed C?: 10uF/6.3V/20%/X5R/C0603, OLIMEX_RLC-FP:C_0603_5MIL_DWS, symbol S3-OLinuXino_Rev_A:C
- removed HEADPHONES/LINEOUT?, MIC/LINEIN?: PJ-W47S-05D2-LF, OLIMEX_Connectors-FP:PJ-W47S-05D2-LF_5PIN_V2, symbol S3-OLinuXino_Rev_A:PJ-W47S-05D2-LF_V2
- removed HPHONEOUTL/LINEOUTL?, HPHONEOUTR/LINEOUTR?: Soldered(1-2);Opened(2-3), OLIMEX_Jumpers-FP:SJ_2_SMALL, symbol S3-OLinuXino_Rev_A:SJ2W_Closed(1-2)
- removed J?: TRS, symbol Connector:AudioJack3_Ground_SwitchTR
- removed L? (x3): FB0805\\600R\\2A, OLIMEX_RLC-FP:L_0805_5MIL_DWS, symbol S3-OLinuXino_Rev_A:L
- removed LINEINL/MICIN?, LINEINR/MICIN?: Opened(2-3);Soldered(1-2), OLIMEX_Jumpers-FP:SJ_2_SMALL, symbol S3-OLinuXino_Rev_A:SJ2W_Closed(1-2)
- removed R?: 200k/1%/R0402, OLIMEX_RLC-FP:R_0402_5MIL_DWS, symbol S3-OLinuXino_Rev_A:R
- removed R? (x3): 2.2k/R0402, OLIMEX_RLC-FP:R_0402_5MIL_DWS, symbol S3-OLinuXino_Rev_A:R
- removed R?: 470R/R0402, OLIMEX_RLC-FP:R_0402_5MIL_DWS, symbol S3-OLinuXino_Rev_A:R
- removed R? (x2): 22R/R0402, OLIMEX_RLC-FP:R_0402_5MIL_DWS, symbol S3-OLinuXino_Rev_A:R
- removed R?: 0R/R0402(Board_Mounted), OLIMEX_RLC-FP:R_0402_5MIL_0R(Board_Mounted), symbol S3-OLinuXino_Rev_A:R
- removed R? (x2): NA/R0402, OLIMEX_RLC-FP:R_0402_5MIL_DWS, symbol S3-OLinuXino_Rev_A:R
- added C46, C50, C53: 220p, otter:C_0402, symbol Device:C_Small
- added C47: 1n, otter:C_0402, symbol Device:C_Small
- added C56, C57, C69: 10u, otter:CP_EIA-3216-10, symbol Device:CP_Small
- added C61: 100n, otter:C_0402, symbol Device:C_Small
- added J5, J6, J7: PJ-3270, symbol otter:PJ-3270
- added MK1: Mic, symbol Device:Microphone
- added R40: 200k, otter:C_0402, symbol Device:R_Small
- added R41: 2k2, otter:C_0402, symbol Device:R_Small
- added R42: 47k, otter:C_0402, symbol Device:R_Small
- added R43: 680, otter:C_0402, symbol Device:R_Small
- added R44, R45, R46: 0, otter:C_0402, symbol Device:R_Small
- added R47, R52: DNP, otter:C_0402, symbol Device:R_Small
- gave numbers to parts that had none: 37
Connections:
- net labels added: MIC-DET
- net labels removed: HP(MIC)-DET, HPOUTFB, HPOUTL, HPOUTR, LINEINL, LINEINR, LINEOUTL, LINEOUTR, MBIAS, MICIN1_N, MICIN1_P, MICIN3_N, MICIN3_P
- wire segments 208 -> 159
- no-connect marks 5 -> 6
Other:
- note removed: "Audio"
- note removed: "Option for \nHandsfree\nUsage"
- moved on the sheet: C48, C49, C51, C52, C54, C55, C58, C59, C60, C62, C63, C64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

Commit message: update
Parts:
- J5, J6, J7: footprint (none) -> otter:PJ-3270
- MK1: footprint (none) -> otter:B4013AM422-42
- U6: footprint (none) -> otter:LFCSP-28-5x5mm-0.5mm-EP3.14x3.14mm
- Y1: footprint (none) -> otter:Oscillator_3225
Changed lines of the file:
@@
 F 0 "U6" H 6450 3900 50  0000 C CNN
 F 1 "SSM2603" H 6450 4000 50  0000 C CNN
-F 2 "" H 5750 4050 50  0001 C CNN
+F 2 "otter:LFCSP-28-5x5mm-0.5mm-EP3.14x3.14mm" H 5750 4050 50  0001 C CNN
 F 3 "" H 5750 4050 50  0001 C CNN
 	1    5750 4050
@@
 F 0 "Y1" V 4550 5250 50  0000 L CNN
 F 1 "12.288Mhz" V 4550 4750 50  0000 L CNN
-F 2 "" H 4750 5150 50  0001 C CNN
+F 2 "otter:Oscillator_3225" H 4750 5150 50  0001 C CNN
 F 3 "~" H 4750 5150 50  0001 C CNN
 	1    4750 5150
@@
 F 0 "MK1" H 2700 4350 50  0000 L CNN
 F 1 "Mic" H 2700 4050 50  0000 L CNN
-F 2 "" V 2650 4300 50  0001 C CNN
+F 2 "otter:B4013AM422-42" V 2650 4300 50  0001 C CNN
 F 3 "~" V 2650 4300 50  0001 C CNN
 	1    2650 4200
@@
 F 0 "J7" H 8712 2818 50  0000 R CNN
 F 1 "PJ-3270" H 8712 2727 50  0000 R CNN
-F 2 "" H 9050 2900 50  0001 C CNN
+F 2 "otter:PJ-3270" H 9050 2900 50  0001 C CNN
 F 3 "~" H 9050 2900 50  0001 C CNN
 	1    9050 2900
@@
 F 0 "J6" H 8112 3318 50  0000 R CNN
 F 1 "PJ-3270" H 8112 3227 50  0000 R CNN
-F 2 "" H 8450 3400 50  0001 C CNN
+F 2 "otter:PJ-3270" H 8450 3400 50  0001 C CNN
 F 3 "~" H 8450 3400 50  0001 C CNN
 	1    8450 3400
@@
 F 0 "J5" H 2862 3018 50  0000 R CNN
 F 1 "PJ-3270" H 2862 2927 50  0000 R CNN
-F 2 "" H 3200 3100 50  0001 C CNN
+F 2 "otter:PJ-3270" H 3200 3100 50  0001 C CNN
 F 3 "~" H 3200 3100 50  0001 C CNN
 	1    3200 3100

Commit message: update
Parts:
- removed R53, R55, R56, R57: 22, otter:C_0402, symbol Device:R_Small
- added NT1: NT, NetTie:NetTie-2_SMD_Pad0.5mm, symbol Device:Net-Tie_2
Connections:
- net BT-PCM-CLK: now also U6.7 (BCLK)
- net BT-PCM-DIN: now also U6.10 (RECDAT)
- net BT-PCM-DOUT: now also U6.8 (PBDAT)
- net BT-PCM-SYNC: now also U6.9 (PBLRC)
- net GND: now also NT1.2; no longer U6.15 (PGND), U6.19 (AGND)
- net GNDA: now also U6.15 (PGND), U6.19 (AGND), NT1.1
Changed lines of the file:
@@
-$EndComp
-$Comp
-L otter:GND #PWR0203
-U 1 1 5FF822B2
-P 5450 5800
-F 0 "#PWR0203" H 5450 5550 50  0001 C CNN
-F 1 "GND" H 5455 5627 50  0000 C CNN
-F 2 "" H 5450 5800 60  0000 C CNN
-F 3 "" H 5450 5800 60  0000 C CNN
-	1    5450 5800
-	1    0    0    -1
-$EndComp
-$Comp
-L otter:GND #PWR0204
-U 1 1 5FF859C3
-P 5650 5800
-F 0 "#PWR0204" H 5650 5550 50  0001 C CNN
-F 1 "GND" H 5655 5627 50  0000 C CNN
-F 2 "" H 5650 5800 60  0000 C CNN
-F 3 "" H 5650 5800 60  0000 C CNN
-	1    5650 5800
-	1    0    0    -1
 $EndComp
 $Comp
@@
 $Comp
 L Device:R_Small R?
-U 1 1 6004788C
-P 4900 3900
-AR Path="/6004788C" Ref="R?"  Part="1"
-AR Path="/602ACDF9/6004788C" Ref="R?"  Part="1"
-AR Path="/604A1CEE/6004788C" Ref="R53"  Part="1"
-F 0 "R53" V 4850 3750 50  0000 C CNN
-F 1 "22" V 4850 4100 50  0000 C CNN
-F 2 "otter:C_0402" H 4900 3900 50  0001 C CNN
-F 3 "~" H 4900 3900 50  0001 C CNN
-	1    4900 3900
-	0    1    1    0
-$EndComp
-$Comp
-L Device:R_Small R?
 U 1 1 60047892
 P 4900 4000
@@
 $EndComp
 Wire Wire Line
-	5200 3900 5000 3900
-Wire Wire Line
 	5200 4000 5000 4000
 Wire Wire Line
 	4800 4000 4700 4000
 Wire Wire Line
-	4700 3900 4800 3900
-Wire Wire Line
 	4650 4000 4700 4000
-$Comp
-L Device:R_Small R?
-U 1 1 60066F9A
-P 4900 4100
-AR Path="/60066F9A" Ref="R?"  Part="1"
-AR Path="/602ACDF9/60066F9A" Ref="R?"  Part="1"
-AR Path="/604A1CEE/60066F9A" Ref="R55"  Part="1"
-F 0 "R55" V 4850 3950 50  0000 C CNN
-F 1 "22" V 4850 4300 50  0000 C CNN
-F 2 "otter:C_0402" H 4900 4100 50  0001 C CNN
-F 3 "~" H 4900 4100 50  0001 C CNN
-	1    4900 4100
-	0    1    1    0
-$EndComp
-$Comp
-L Device:R_Small R?
-U 1 1 60066FA0
-P 4900 4200
-AR Path="/60066FA0" Ref="R?"  Part="1"
-AR Path="/602ACDF9/60066FA0" Ref="R?"  Part="1"
-AR Path="/604A1CEE/60066FA0" Ref="R56"  Part="1"
-F 0 "R56" V 4850 4050 50  0000 C CNN
-F 1 "22" V 4850 4400 50  0000 C CNN
-F 2 "otter:C_0402" H 4900 4200 50  0001 C CNN
-F 3 "~" H 4900 4200 50  0001 C CNN
-	1    4900 4200
-	0    1    1    0
-$EndComp
-$Comp
-L Device:R_Small R?
-U 1 1 6006C313
-P 4900 4300
-AR Path="/6006C313" Ref="R?"  Part="1"
-AR Path="/602ACDF9/6006C313" Ref="R?"  Part="1"
-AR Path="/604A1CEE/6006C313" Ref="R57"  Part="1"
-F 0 "R57" V 4850 4150 50  0000 C CNN
-F 1 "22" V 4850 4500 50  0000 C CNN
-F 2 "otter:C_0402" H 4900 4300 50  0001 C CNN
-F 3 "~" H 4900 4300 50  0001 C CNN
-	1    4900 4300
-	0    1    1    0
-$EndComp
-Wire Wire Line
-	4650 4100 4800 4100
-Wire Wire Line
-	4650 4200 4800 4200
-Wire Wire Line
-	4650 4300 4800 4300
-Wire Wire Line
-	5000 4300 5200 4300
-Wire Wire Line
-	5200 4200 5000 4200
-Wire Wire Line
-	5000 4100 5200 4100
 $Comp
 L Device:R_Small R?
@@
 	3900 1950 3950 1950
 $Comp
-L otter:GND #PWR0219
-U 1 1 60344556
-P 3900 2350
-F 0 "#PWR0219" H 3900 2100 50  0001 C CNN
-F 1 "GND" V 3905 2222 50  0000 R CNN
-F 2 "" H 3900 2350 60  0000 C CNN
-F 3 "" H 3900 2350 60  0000 C CNN
-	1    3900 2350
-	0    1    1    0
-$EndComp
-$Comp
 L S3-OLinuXino_Rev_A:+3.0VA #PWR?
 U 1 1 602F2215
@@
 AR Path="/602ACDF9/6077F988" Ref="R?"  Part="1"
 AR Path="/604A1CEE/6077F988" Ref="R47"  Part="1"
-F 0 "R47" H 3950 3300 50  0000 R CNN
+F 0 "R47" H 4000 3300 50  0000 R CNN
 F 1 "DNP" H 4000 3100 50  0000 R CNN
 F 2 "otter:C_0402" H 3800 3250 50  0001 C CNN
@@
 Wire Wire Line
 	2950 2450 2950 2400
+Wire Wire Line
+	4700 3900 5200 3900
+Wire Wire Line
+	4650 4100 5200 4100
+Wire Wire Line
+	4650 4200 5200 4200
+Wire Wire Line
+	4650 4300 5200 4300
+$Comp
+L power:GNDA #PWR0155
+U 1 1 5FE42585
+P 5650 5800
+F 0 "#PWR0155" H 5650 5550 50  0001 C CNN
+F 1 "GNDA" H 5655 5627 50  0000 C CNN
+F 2 "" H 5650 5800 50  0001 C CNN
+F 3 "" H 5650 5800 50  0001 C CNN
+	1    5650 5800
+	1    0    0    -1
+$EndComp
+$Comp
+L power:GNDA #PWR0203
+U 1 1 5FE49B0D
+P 5450 5800
+F 0 "#PWR0203" H 5450 5550 50  0001 C CNN
+F 1 "GNDA" H 5455 5627 50  0000 C CNN
+F 2 "" H 5450 5800 50  0001 C CNN
+F 3 "" H 5450 5800 50  0001 C CNN
+	1    5450 5800
+	1    0    0    -1
+$EndComp
+$Comp
+L otter:GND #PWR0219
+U 1 1 60344556
+P 3900 2350
+F 0 "#PWR0219" H 3900 2100 50  0001 C CNN
+F 1 "GND" V 3905 2222 50  0000 R CNN
+F 2 "" H 3900 2350 60  0000 C CNN
+F 3 "" H 3900 2350 60  0000 C CNN
+	1    3900 2350
+	0    1    1    0
+$EndComp
+$Comp
+L power:GNDA #PWR0204
+U 1 1 5FE53E3B
+P 5650 6600
+F 0 "#PWR0204" H 5650 6350 50  0001 C CNN
+F 1 "GNDA" V 5655 6473 50  0000 R CNN
+F 2 "" H 5650 6600 50  0001 C CNN
+F 3 "" H 5650 6600 50  0001 C CNN
+	1    5650 6600
+	0    1    1    0
+$EndComp
+$Comp
+L otter:GND #PWR0295
+U 1 1 5FE5C65A
+P 5850 6600
+F 0 "#PWR0295" H 5850 6350 50  0001 C CNN
+F 1 "GND" V 5855 6472 50  0000 R CNN
+F 2 "" H 5850 6600 60  0000 C CNN
+F 3 "" H 5850 6600 60  0000 C CNN
+	1    5850 6600
+	0    -1   -1   0
+$EndComp
+$Comp
+L Device:Net-Tie_2 NT1
+U 1 1 5FE66928
+P 5750 6600
+F 0 "NT1" H 5750 6781 50  0000 C CNN
+F 1 "NT" H 5750 6690 50  0000 C CNN
+F 2 "NetTie:NetTie-2_SMD_Pad0.5mm" H 5750 6600 50  0001 C CNN
+F 3 "~" H 5750 6600 50  0001 C CNN
+	1    5750 6600
+	1    0    0    -1
+$EndComp
 $EndSCHEMATC

Commit message: update
Parts:
- removed C48, C49: 100n, otter:C_0402, symbol Device:C_Small
Changed lines of the file:
@@
 L S3-OLinuXino_Rev_A:+3.0VA #PWR?
 U 1 1 6027AD71
-P 3900 1700
+P 4250 1700
 AR Path="/5D8A1FAC/6027AD71" Ref="#PWR?"  Part="1"
 AR Path="/6027AD71" Ref="#PWR?"  Part="1"
 AR Path="/602ACDF9/6027AD71" Ref="#PWR?"  Part="1"
 AR Path="/604A1CEE/6027AD71" Ref="#PWR0216"  Part="1"
-F 0 "#PWR0216" H 3900 1550 50  0001 C CNN
-F 1 "+3.0VA" V 3900 1825 50  0000 L CNN
-F 2 "" H 3900 1700 60  0000 C CNN
-F 3 "" H 3900 1700 60  0000 C CNN
-	1    3900 1700
-	0    -1   -1   0
-$EndComp
-$Comp
-L Device:C_Small C?
-U 1 1 602852B3
-P 3950 1850
-AR Path="/602852B3" Ref="C?"  Part="1"
-AR Path="/604A1CEE/602852B3" Ref="C48"  Part="1"
-F 0 "C48" H 4042 1896 50  0000 L CNN
-F 1 "100n" H 4042 1805 50  0000 L CNN
-F 2 "otter:C_0402" H 3950 1850 50  0001 C CNN
-F 3 "~" H 3950 1850 50  0001 C CNN
-	1    3950 1850
-	1    0    0    -1
-$EndComp
-$Comp
-L Device:C_Small C?
-U 1 1 6028FB2E
-P 3950 2250
-AR Path="/6028FB2E" Ref="C?"  Part="1"
-AR Path="/604A1CEE/6028FB2E" Ref="C49"  Part="1"
-F 0 "C49" H 4042 2296 50  0000 L CNN
-F 1 "100n" H 4042 2205 50  0000 L CNN
-F 2 "otter:C_0402" H 3950 2250 50  0001 C CNN
-F 3 "~" H 3950 2250 50  0001 C CNN
-	1    3950 2250
-	1    0    0    -1
+F 0 "#PWR0216" H 4250 1550 50  0001 C CNN
+F 1 "+3.0VA" V 4250 1825 50  0000 L CNN
+F 2 "" H 4250 1700 60  0000 C CNN
+F 3 "" H 4250 1700 60  0000 C CNN
+	1    4250 1700
+	0    -1   -1   0
 $EndComp
 $Comp
@@
 Wire Wire Line
 	4450 2100 4750 2100
-Wire Wire Line
-	4250 2100 3950 2100
-Wire Wire Line
-	3950 2100 3950 2150
-Wire Wire Line
-	4250 1700 3950 1700
-Wire Wire Line
-	3950 1700 3950 1750
 $Comp
 L power:GNDA #PWR0218
@@
 	0    1    1    0
 $EndComp
-Wire Wire Line
-	3900 2100 3950 2100
-Connection ~ 3950 2100
-Wire Wire Line
-	3900 1700 3950 1700
-Connection ~ 3950 1700
-Wire Wire Line
-	3900 2350 3950 2350
-Wire Wire Line
-	3900 1950 3950 1950
 $Comp
 L S3-OLinuXino_Rev_A:+3.0VA #PWR?
 U 1 1 602F2215
-P 3900 2100
+P 4250 2100
 AR Path="/5D8A1FAC/602F2215" Ref="#PWR?"  Part="1"
 AR Path="/602F2215" Ref="#PWR?"  Part="1"
 AR Path="/602ACDF9/602F2215" Ref="#PWR?"  Part="1"
 AR Path="/604A1CEE/602F2215" Ref="#PWR0220"  Part="1"
-F 0 "#PWR0220" H 3900 1950 50  0001 C CNN
-F 1 "+3.0VA" V 3900 2225 50  0000 L CNN
-F 2 "" H 3900 2100 60  0000 C CNN
-F 3 "" H 3900 2100 60  0000 C CNN
-	1    3900 2100
-	0    -1   -1   0
-$EndComp
-$Comp
-L otter:GND #PWR0221
-U 1 1 6035011E
-P 3900 1950
-F 0 "#PWR0221" H 3900 1700 50  0001 C CNN
-F 1 "GND" V 3905 1822 50  0000 R CNN
-F 2 "" H 3900 1950 60  0000 C CNN
-F 3 "" H 3900 1950 60  0000 C CNN
-	1    3900 1950
-	0    1    1    0
+F 0 "#PWR0220" H 4250 1950 50  0001 C CNN
+F 1 "+3.0VA" V 4250 2225 50  0000 L CNN
+F 2 "" H 4250 2100 60  0000 C CNN
+F 3 "" H 4250 2100 60  0000 C CNN
+	1    4250 2100
+	0    -1   -1   0
 $EndComp
 $Comp
@@
 $EndComp
 $Comp
-L otter:GND #PWR0219
-U 1 1 60344556
-P 3900 2350
-F 0 "#PWR0219" H 3900 2100 50  0001 C CNN
-F 1 "GND" V 3905 2222 50  0000 R CNN
-F 2 "" H 3900 2350 60  0000 C CNN
-F 3 "" H 3900 2350 60  0000 C CNN
-	1    3900 2350
-	0    1    1    0
-$EndComp
-$Comp

Commit message: update
Changed lines of the file:
@@
 Connection ~ 4150 4750
 Wire Wire Line
-	4450 4750 5200 4750
-Wire Wire Line
-	5200 4850 4450 4850
-Text Label 4750 4850 0    50   ~ 0
-MIPI-SCK
-Text Label 4750 4750 0    50   ~ 0
-MIPI-SDA
+	4450 4750 5100 4750
+Wire Wire Line
+	5200 4850 5100 4850
 $Comp
 L Device:R_Small R?
@@
 	1    0    0    -1
 $EndComp
+Text GLabel 5050 4700 0    50   Input ~ 0
+MIPI-SDA
+Text GLabel 5050 4800 0    50   Input ~ 0
+MIPI-SCK
+Wire Wire Line
+	5050 4800 5100 4800
+Wire Wire Line
+	5100 4800 5100 4850
+Connection ~ 5100 4850
+Wire Wire Line
+	5100 4850 4450 4850
+Wire Wire Line
+	5050 4700 5100 4700
+Wire Wire Line
+	5100 4700 5100 4750
+Connection ~ 5100 4750
+Wire Wire Line
+	5100 4750 5200 4750
 $EndSCHEMATC

Commit message: no drc error
Parts:
- removed NT1: NT, NetTie:NetTie-2_SMD_Pad0.5mm, symbol Device:Net-Tie_2
- added R?: 0R, otter:R_0805, symbol Device:R_Small
- R40, R41, R42, R43, R44, R45, R46, R47, R48, R49, R50, R51, R52, R54, R58, R59, R60, R61, R62, R63: footprint otter:C_0402 -> otter:R_0402
Connections:
- net GND: now also R?.1
- net GNDA: now also R?.2
Changed lines of the file:
@@
 F 0 "R50" V 4300 4600 50  0000 C CNN
 F 1 "2.2k" V 4300 4950 50  0000 C CNN
-F 2 "otter:C_0402" H 4350 4750 50  0001 C CNN
+F 2 "otter:R_0402" H 4350 4750 50  0001 C CNN
 F 3 "~" H 4350 4750 50  0001 C CNN
 	1    4350 4750
@@
 F 0 "R51" V 4300 4700 50  0000 C CNN
 F 1 "2.2k" V 4300 5050 50  0000 C CNN
-F 2 "otter:C_0402" H 4350 4850 50  0001 C CNN
+F 2 "otter:R_0402" H 4350 4850 50  0001 C CNN
 F 3 "~" H 4350 4850 50  0001 C CNN
 	1    4350 4850
@@
 F 0 "R54" V 4850 3850 50  0000 C CNN
 F 1 "22" V 4850 4200 50  0000 C CNN
-F 2 "otter:C_0402" H 4900 4000 50  0001 C CNN
+F 2 "otter:R_0402" H 4900 4000 50  0001 C CNN
 F 3 "~" H 4900 4000 50  0001 C CNN
 	1    4900 4000
@@
 F 0 "R49" V 4300 4500 50  0000 C CNN
 F 1 "2.2k" V 4300 4850 50  0000 C CNN
-F 2 "otter:C_0402" H 4350 4650 50  0001 C CNN
+F 2 "otter:R_0402" H 4350 4650 50  0001 C CNN
 F 3 "~" H 4350 4650 50  0001 C CNN
 	1    4350 4650
@@
 F 0 "R48" V 4300 4400 50  0000 C CNN
 F 1 "2.2k" V 4300 4750 50  0000 C CNN
-F 2 "otter:C_0402" H 4350 4550 50  0001 C CNN
+F 2 "otter:R_0402" H 4350 4550 50  0001 C CNN
 F 3 "~" H 4350 4550 50  0001 C CNN
 	1    4350 4550
@@
 F 0 "R58" H 7109 2796 50  0000 L CNN
 F 1 "47k" H 7109 2705 50  0000 L CNN
-F 2 "otter:C_0402" H 7050 2750 50  0001 C CNN
+F 2 "otter:R_0402" H 7050 2750 50  0001 C CNN
 F 3 "~" H 7050 2750 50  0001 C CNN
 	1    7050 2750
@@
 F 0 "R60" H 7409 2796 50  0000 L CNN
 F 1 "47k" H 7409 2705 50  0000 L CNN
-F 2 "otter:C_0402" H 7350 2750 50  0001 C CNN
+F 2 "otter:R_0402" H 7350 2750 50  0001 C CNN
 F 3 "~" H 7350 2750 50  0001 C CNN
 	1    7350 2750
@@
 F 0 "R61" V 7454 2900 50  0000 C CNN
 F 1 "100" V 7545 2900 50  0000 C CNN
-F 2 "otter:C_0402" H 7650 2900 50  0001 C CNN
+F 2 "otter:R_0402" H 7650 2900 50  0001 C CNN
 F 3 "~" H 7650 2900 50  0001 C CNN
 	1    7650 2900
@@
 F 0 "R62" V 7754 3100 50  0000 C CNN
 F 1 "100" V 7845 3100 50  0000 C CNN
-F 2 "otter:C_0402" H 7650 3100 50  0001 C CNN
+F 2 "otter:R_0402" H 7650 3100 50  0001 C CNN
 F 3 "~" H 7650 3100 50  0001 C CNN
 	1    7650 3100
@@
 F 0 "R59" H 7109 3796 50  0000 L CNN
 F 1 "47k" H 7109 3705 50  0000 L CNN
-F 2 "otter:C_0402" H 7050 3750 50  0001 C CNN
+F 2 "otter:R_0402" H 7050 3750 50  0001 C CNN
 F 3 "~" H 7050 3750 50  0001 C CNN
 	1    7050 3750
@@
 F 0 "R63" H 7709 3796 50  0000 L CNN
 F 1 "47k" H 7709 3705 50  0000 L CNN
-F 2 "otter:C_0402" H 7650 3750 50  0001 C CNN
+F 2 "otter:R_0402" H 7650 3750 50  0001 C CNN
 F 3 "~" H 7650 3750 50  0001 C CNN
 	1    7650 3750
@@
 F 0 "R47" H 4000 3300 50  0000 R CNN
 F 1 "DNP" H 4000 3100 50  0000 R CNN
-F 2 "otter:C_0402" H 3800 3250 50  0001 C CNN
+F 2 "otter:R_0402" H 3800 3250 50  0001 C CNN
 F 3 "~" H 3800 3250 50  0001 C CNN
 	1    3800 3250
@@
 F 0 "R52" H 4450 3300 50  0000 L CNN
 F 1 "DNP" H 4450 3100 50  0000 L CNN
-F 2 "otter:C_0402" H 4400 3250 50  0001 C CNN
+F 2 "otter:R_0402" H 4400 3250 50  0001 C CNN
 F 3 "~" H 4400 3250 50  0001 C CNN
 	1    4400 3250
@@
 F 0 "R44" V 3796 2900 50  0000 C CNN
 F 1 "0" V 3705 2900 50  0000 C CNN
-F 2 "otter:C_0402" H 3600 2900 50  0001 C CNN
+F 2 "otter:R_0402" H 3600 2900 50  0001 C CNN
 F 3 "~" H 3600 2900 50  0001 C CNN
 	1    3600 2900
@@
 F 0 "R45" V 3496 3100 50  0000 C CNN
 F 1 "0" V 3405 3100 50  0000 C CNN
-F 2 "otter:C_0402" H 3600 3100 50  0001 C CNN
+F 2 "otter:R_0402" H 3600 3100 50  0001 C CNN
 F 3 "~" H 3600 3100 50  0001 C CNN
 	1    3600 3100
@@
 F 0 "R43" V 3696 3900 50  0000 C CNN
 F 1 "680" V 3605 3900 50  0000 C CNN
-F 2 "otter:C_0402" H 3500 3900 50  0001 C CNN
+F 2 "otter:R_0402" H 3500 3900 50  0001 C CNN
 F 3 "~" H 3500 3900 50  0001 C CNN
 	1    3500 3900
@@
 F 0 "R46" V 3796 4250 50  0000 C CNN
 F 1 "0" V 3705 4250 50  0000 C CNN
-F 2 "otter:C_0402" H 3600 4250 50  0001 C CNN
+F 2 "otter:R_0402" H 3600 4250 50  0001 C CNN
 F 3 "~" H 3600 4250 50  0001 C CNN
 	1    3600 4250
@@
 F 0 "R42" H 3041 4246 50  0000 R CNN
 F 1 "47k" H 3041 4155 50  0000 R CNN
-F 2 "otter:C_0402" H 3100 4200 50  0001 C CNN
+F 2 "otter:R_0402" H 3100 4200 50  0001 C CNN
 F 3 "~" H 3100 4200 50  0001 C CNN
 	1    3100 4200
@@
 F 0 "R41" H 3009 2646 50  0000 L CNN
 F 1 "2k2" H 3009 2555 50  0000 L CNN
-F 2 "otter:C_0402" H 2950 2600 50  0001 C CNN
+F 2 "otter:R_0402" H 2950 2600 50  0001 C CNN
 F 3 "~" H 2950 2600 50  0001 C CNN
 	1    2950 2600
@@
 F 0 "R40" H 3009 2346 50  0000 L CNN
 F 1 "200k" H 3009 2255 50  0000 L CNN
-F 2 "otter:C_0402" H 2950 2300 50  0001 C CNN
+F 2 "otter:R_0402" H 2950 2300 50  0001 C CNN
 F 3 "~" H 2950 2300 50  0001 C CNN
 	1    2950 2300
@@
 	0    -1   -1   0
 $EndComp
-$Comp
-L Device:Net-Tie_2 NT1
-U 1 1 5FE66928
-P 5750 6600
-F 0 "NT1" H 5750 6781 50  0000 C CNN
-F 1 "NT" H 5750 6690 50  0000 C CNN
-F 2 "NetTie:NetTie-2_SMD_Pad0.5mm" H 5750 6600 50  0001 C CNN
-F 3 "~" H 5750 6600 50  0001 C CNN
-	1    5750 6600
-	1    0    0    -1
-$EndComp
 Text GLabel 5050 4700 0    50   Input ~ 0
 MIPI-SDA
@@
 Wire Wire Line
 	5100 4750 5200 4750
+$Comp
+L Device:R_Small R?
+U 1 1 5FCF40A4
+P 5750 6600
+AR Path="/5FCF40A4" Ref="R?"  Part="1"
+AR Path="/602ACDF9/5FCF40A4" Ref="R?"  Part="1"
+AR Path="/604A1CEE/5FCF40A4" Ref="R?"  Part="1"
+F 0 "R?" V 5554 6600 50  0000 C CNN
+F 1 "0R" V 5645 6600 50  0000 C CNN
+F 2 "otter:R_0805" H 5750 6600 50  0001 C CNN
+F 3 "~" H 5750 6600 50  0001 C CNN
+	1    5750 6600
+	0    1    1    0
+$EndComp
 $EndSCHEMATC

Commit message: no drc error
Parts:
- gave numbers to parts that had none: 1
Changed lines of the file:
@@
 AR Path="/5FCF40A4" Ref="R?"  Part="1"
 AR Path="/602ACDF9/5FCF40A4" Ref="R?"  Part="1"
-AR Path="/604A1CEE/5FCF40A4" Ref="R?"  Part="1"
-F 0 "R?" V 5554 6600 50  0000 C CNN
+AR Path="/604A1CEE/5FCF40A4" Ref="R27"  Part="1"
+F 0 "R27" V 5554 6600 50  0000 C CNN
 F 1 "0R" V 5645 6600 50  0000 C CNN
 F 2 "otter:R_0805" H 5750 6600 50  0001 C CNN
