File: OtterCastAudioV2.sch (KiCad schematic (older format))
At the start: 26 parts

Commit message: update
Parts:
- removed R? (x2): 5k1, otter:C_0402, symbol Device:R_Small
- added R? (x2): 2.2k, otter:C_0402, symbol Device:R_Small
Connections:
- net +3V3: now also R?.1, R?.1
- net PB8\TWI1-SCK: now also R?.2
- net PB9\TWI1-SDA: now also R?.2
- net MIPI-MSCK: now reaches U?.H15 (PE20/CSI_FIELD/CSI_MIPI_MCLK)
- no-connect marks 52 -> 51
Changed lines of the file:
@@
 Comment4 ""
 $EndDescr
-Text GLabel 4650 5200 2    60   Input ~ 0
-USB-ID
 $Comp
 L S3-OLinuXino_Rev_A:+3.3V #PWR032
@@
 	1    0    0    -1
 $EndComp
-NoConn ~ 4350 2950
 NoConn ~ 4350 3150
 NoConn ~ 4350 3250
@@
 	1    0    0    -1
 $EndComp
-$Comp
-L otter:AllWinner-S3(FBGA-234) U?
-U 3 1 67AFCAD8
-P 3050 3150
-F 0 "U?" H 3050 4015 50  0000 C CNN
-F 1 "AllWinner-S3(FBGA-234)" H 3050 3924 50  0000 C CNN
-F 2 "OLIMEX_IC-FP:FBGA-234(Pitch-0.65mm_Pad-0.3mm_11x11x1.08mm)" H 3050 1100 50  0001 C CNN
-F 3 "" H 3250 4850 50  0001 C CNN
-	3    3050 3150
-	1    0    0    -1
-$EndComp
 Text GLabel 1750 1300 0    50   Input ~ 0
 GPIO_LED2
@@
 Wire Wire Line
 	13950 7100 14150 7100
-$Comp
-L Device:R_Small R?
-U 1 1 67CD5CEB
-P 14650 7200
-F 0 "R?" H 14591 7154 50  0000 R CNN
-F 1 "5k1" H 14591 7245 50  0000 R CNN
-F 2 "otter:C_0402" H 14650 7200 50  0001 C CNN
-F 3 "~" H 14650 7200 50  0001 C CNN
-	1    14650 7200
-	-1   0    0    1
-$EndComp
-$Comp
-L Device:R_Small R?
-U 1 1 67CD9C01
-P 14900 7200
-F 0 "R?" H 14841 7154 50  0000 R CNN
-F 1 "5k1" H 14841 7245 50  0000 R CNN
-F 2 "otter:C_0402" H 14900 7200 50  0001 C CNN
-F 3 "~" H 14900 7200 50  0001 C CNN
-	1    14900 7200
-	-1   0    0    1
-$EndComp
 Wire Wire Line
 	15000 7350 14650 7350
@@
 	14650 7000 14650 7050
 Connection ~ 14650 7050
+Text GLabel 4650 5200 2    50   Input ~ 0
+USB-ID
+Text GLabel 4350 2950 2    50   Input ~ 0
+MIPI-MSCK
+$Comp
+L otter:AllWinner-S3(FBGA-234) U?
+U 3 1 67AFCAD8
+P 3050 3150
+F 0 "U?" H 3050 4015 50  0000 C CNN
+F 1 "AllWinner-S3(FBGA-234)" H 3050 3924 50  0000 C CNN
+F 2 "OLIMEX_IC-FP:FBGA-234(Pitch-0.65mm_Pad-0.3mm_11x11x1.08mm)" H 3050 1100 50  0001 C CNN
+F 3 "" H 3250 4850 50  0001 C CNN
+	3    3050 3150
+	1    0    0    -1
+$EndComp
+$Comp
+L Device:R_Small R?
+U 1 1 5FFC46C5
+P 14650 7200
+AR Path="/5FFC46C5" Ref="R?"  Part="1"
+AR Path="/602ACDF9/5FFC46C5" Ref="R?"  Part="1"
+F 0 "R?" H 14709 7246 50  0000 L CNN
+F 1 "2.2k" H 14709 7155 50  0000 L CNN
+F 2 "otter:C_0402" H 14650 7200 50  0001 C CNN
+F 3 "~" H 14650 7200 50  0001 C CNN
+	1    14650 7200
+	1    0    0    -1
+$EndComp
+$Comp
+L Device:R_Small R?
+U 1 1 5FFC572E
+P 14900 7200
+AR Path="/5FFC572E" Ref="R?"  Part="1"
+AR Path="/602ACDF9/5FFC572E" Ref="R?"  Part="1"
+F 0 "R?" H 14959 7246 50  0000 L CNN
+F 1 "2.2k" H 14959 7155 50  0000 L CNN
+F 2 "otter:C_0402" H 14900 7200 50  0001 C CNN
+F 3 "~" H 14900 7200 50  0001 C CNN
+	1    14900 7200
+	1    0    0    -1
+$EndComp
 $EndSCHEMATC

Commit message: update
Parts:
- gave numbers to parts that had none: 24
Connections:
- net labels added: MIC-DET
- net labels removed: HP(MIC)-DET
Other:
- moved on the sheet: C1, C2, C3, C4, D1, D2, FB1, J1, J2, R1, R10, R11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

Commit message: update
Parts:
- D1, D2: footprint (none) -> otter:LED_0603_1608Metric
- J1: footprint (none) -> Connector_PinHeader_2.00mm:PinHeader_1x04_P2.00mm_Vertical
- J2: footprint (none) -> Connector_Card:microSD_HC_Hirose_DM3D-SF
- U1: footprint OLIMEX_IC-FP:FBGA-234(Pitch-0.65mm_Pad-0.3mm_11x11x1.08mm) -> otter:FBGA-234(Pitch-0.65mm_Pad-0.3mm_11x11x1.08mm)
Other:
- moved on the sheet: U1B, U1C
Changed lines of the file:
@@
 F 0 "J2" H 13200 9117 50  0000 C CNN
 F 1 "SD" H 13200 9026 50  0000 C CNN
-F 2 "" H 15300 9000 50  0001 C CNN
+F 2 "Connector_Card:microSD_HC_Hirose_DM3D-SF" H 15300 9000 50  0001 C CNN
 F 3 "https://www.hirose.com/product/en/download_file/key_name/DM3/category/Catalog/doc_file_id/49662/?file_category_id=4&item_id=195&is_series=1" H 13250 8400 50  0001 C CNN
 	1    13250 8300
@@
 F 0 "J1" H 7480 10392 50  0000 L CNN
 F 1 "UART" H 7480 10301 50  0000 L CNN
-F 2 "" H 7400 10400 50  0001 C CNN
+F 2 "Connector_PinHeader_2.00mm:PinHeader_1x04_P2.00mm_Vertical" H 7400 10400 50  0001 C CNN
 F 3 "~" H 7400 10400 50  0001 C CNN
 	1    7400 10400
@@
 F 0 "D1" V 8139 10433 50  0000 R CNN
 F 1 "LED" V 8048 10433 50  0000 R CNN
-F 2 "" H 8100 10550 50  0001 C CNN
+F 2 "otter:LED_0603_1608Metric" H 8100 10550 50  0001 C CNN
 F 3 "~" H 8100 10550 50  0001 C CNN
 	1    8100 10550
@@
 Wire Wire Line
 	4100 6600 4150 6600
-Wire Wire Line
-	4150 6500 3800 6500
 NoConn ~ 4150 6100
 NoConn ~ 4150 6200
@@
 	1    0    0    -1
 $EndComp
-Wire Wire Line
-	4050 5800 3750 5800
 Connection ~ 4050 5800
 Connection ~ 3750 5800
@@
 F 0 "U1" H 5450 3765 50  0000 C CNN
 F 1 "AllWinner-S3(FBGA-234)" H 5450 3674 50  0000 C CNN
-F 2 "OLIMEX_IC-FP:FBGA-234(Pitch-0.65mm_Pad-0.3mm_11x11x1.08mm)" H 5450 850 50  0001 C CNN
+F 2 "otter:FBGA-234(Pitch-0.65mm_Pad-0.3mm_11x11x1.08mm)" H 5450 850 50  0001 C CNN
 F 3 "" H 5650 4600 50  0001 C CNN
 	1    5450 2900
@@
 L otter:AllWinner-S3(FBGA-234) U1
 U 3 1 67AF4AB4
-P 12350 4500
-F 0 "U1" H 12400 5965 50  0000 C CNN
-F 1 "AllWinner-S3(FBGA-234)" H 12400 5874 50  0000 C CNN
-F 2 "OLIMEX_IC-FP:FBGA-234(Pitch-0.65mm_Pad-0.3mm_11x11x1.08mm)" H 12350 2450 50  0001 C CNN
-F 3 "" H 12550 6200 50  0001 C CNN
-	3    12350 4500
+P 5450 6400
+F 0 "U1" H 5450 7250 50  0000 C CNN
+F 1 "AllWinner-S3(FBGA-234)" H 5450 7150 50  0000 C CNN
+F 2 "otter:FBGA-234(Pitch-0.65mm_Pad-0.3mm_11x11x1.08mm)" H 5450 4350 50  0001 C CNN
+F 3 "" H 5650 8100 50  0001 C CNN
+	3    5450 6400
 	1    0    0    -1
 $EndComp
@@
 F 0 "D2" V 8489 10433 50  0000 R CNN
 F 1 "LED" V 8398 10433 50  0000 R CNN
-F 2 "" H 8450 10550 50  0001 C CNN
+F 2 "otter:LED_0603_1608Metric" H 8450 10550 50  0001 C CNN
 F 3 "~" H 8450 10550 50  0001 C CNN
 	1    8450 10550
@@
 L otter:AllWinner-S3(FBGA-234) U1
 U 2 1 67AFCAD8
-P 5450 6400
-F 0 "U1" H 5450 7265 50  0000 C CNN
-F 1 "AllWinner-S3(FBGA-234)" H 5450 7174 50  0000 C CNN
-F 2 "OLIMEX_IC-FP:FBGA-234(Pitch-0.65mm_Pad-0.3mm_11x11x1.08mm)" H 5450 4350 50  0001 C CNN
-F 3 "" H 5650 8100 50  0001 C CNN
-	2    5450 6400
+P 12350 4500
+F 0 "U1" H 12350 5850 50  0000 C CNN
+F 1 "AllWinner-S3(FBGA-234)" H 12350 5950 50  0000 C CNN
+F 2 "otter:FBGA-234(Pitch-0.65mm_Pad-0.3mm_11x11x1.08mm)" H 12350 2450 50  0001 C CNN
+F 3 "" H 12550 6200 50  0001 C CNN
+	2    12350 4500
 	1    0    0    -1
 $EndComp
@@
 	1    0    0    -1
 $EndComp
+Wire Wire Line
+	3800 6500 4150 6500
+Wire Wire Line
+	3750 5800 4050 5800
 $EndSCHEMATC

Commit message: update
Parts:
- removed C3: 100n, otter:C_0402, symbol Device:C_Small
- added D5: ESD5302F, Package_TO_SOT_SMD:SOT-23, symbol Power_Protection:SP0502BAHT
- C1: value 100n -> 10u; footprint otter:C_0402 -> otter:C_0603
Connections:
- net +3V3: now also D5.3 (A)
- net UART1_RX: now also D5.1 (K)
- net UART1_TX: now also D5.2 (K)
Changed lines of the file:
@@
 	0    1    1    0
-$EndComp
-$Comp
-L Device:C_Small C3
-U 1 1 63233A4C
-P 10450 3450
-F 0 "C3" H 10358 3496 50  0000 R CNN
-F 1 "100n" H 10358 3405 50  0000 R CNN
-F 2 "otter:C_0402" H 10450 3450 50  0001 C CNN
-F 3 "~" H 10450 3450 50  0001 C CNN
-	1    10450 3450
-	1    0    0    -1
 $EndComp
 Wire Wire Line
@@
 L S3-OLinuXino_Rev_A:+3.3V #PWR0109
 U 1 1 63B28C18
-P 3750 5750
-F 0 "#PWR0109" H 3750 5600 50  0001 C CNN
-F 1 "+3.3V" H 3750 5890 50  0000 C CNN
-F 2 "" H 3750 5750 60  0000 C CNN
-F 3 "" H 3750 5750 60  0000 C CNN
-	1    3750 5750
+P 4050 5750
+F 0 "#PWR0109" H 4050 5600 50  0001 C CNN
+F 1 "+3.3V" H 4050 5890 50  0000 C CNN
+F 2 "" H 4050 5750 60  0000 C CNN
+F 3 "" H 4050 5750 60  0000 C CNN
+	1    4050 5750
 	-1   0    0    -1
 $EndComp
 Wire Wire Line
-	3750 5750 3750 5800
+	4050 5750 4050 5800
 Wire Wire Line
 	4050 5800 4150 5800
@@
 Wire Wire Line
 	4050 5900 4150 5900
-$Comp
-L Device:C_Small C1
-U 1 1 63B28C22
-P 3750 5950
-F 0 "C1" H 3658 5996 50  0000 R CNN
-F 1 "100n" H 3658 5905 50  0000 R CNN
-F 2 "otter:C_0402" H 3750 5950 50  0001 C CNN
-F 3 "~" H 3750 5950 50  0001 C CNN
-	1    3750 5950
-	1    0    0    -1
-$EndComp
 Connection ~ 4050 5800
-Connection ~ 3750 5800
-Wire Wire Line
-	3750 5800 3750 5850
-$Comp
-L otter:GND #PWR0110
-U 1 1 63B28C2C
-P 3750 6050
-F 0 "#PWR0110" H 3750 5800 50  0001 C CNN
-F 1 "GND" H 3755 5877 50  0000 C CNN
-F 2 "" H 3750 6050 60  0000 C CNN
-F 3 "" H 3750 6050 60  0000 C CNN
-	1    3750 6050
-	1    0    0    -1
-$EndComp
 NoConn ~ 6750 6400
 NoConn ~ 6750 6500
@@
 Wire Wire Line
 	3800 6500 4150 6500
-Wire Wire Line
-	3750 5800 4050 5800
+$Comp
+L Device:C_Small C1
+U 1 1 5FBB02B1
+P 10450 3450
+F 0 "C1" H 10358 3496 50  0000 R CNN
+F 1 "10u" H 10358 3405 50  0000 R CNN
+F 2 "otter:C_0603" H 10450 3450 50  0001 C CNN
+F 3 "~" H 10450 3450 50  0001 C CNN
+	1    10450 3450
+	1    0    0    -1
+$EndComp
+$Comp
+L Power_Protection:SP0502BAHT D5
+U 1 1 5FCE3FA8
+P 7350 9950
+F 0 "D5" V 7692 9950 50  0000 C CNN
+F 1 "ESD5302F" V 7601 9950 50  0000 C CNN
+F 2 "Package_TO_SOT_SMD:SOT-23" H 7575 9900 50  0001 L CNN
+F 3 "http://www.littelfuse.com/~/media/files/littelfuse/technical%20resources/documents/data%20sheets/sp05xxba.pdf" H 7475 10075 50  0001 C CNN
+F 4 "C239643" V 7350 9950 50  0001 C CNN "LCSC"
+	1    7350 9950
+	0    -1   -1   0
+$EndComp
+Text GLabel 7150 9850 0    50   Input ~ 0
+UART1_TX
+Text GLabel 7150 10050 0    50   Input ~ 0
+UART1_RX
+$Comp
+L S3-OLinuXino_Rev_A:+3.3V #PWR0154
+U 1 1 5FCE77D5
+P 7550 9950
+F 0 "#PWR0154" H 7550 9800 50  0001 C CNN
+F 1 "+3.3V" V 7565 10078 50  0000 L CNN
+F 2 "" H 7550 9950 60  0000 C CNN
+F 3 "" H 7550 9950 60  0000 C CNN
+	1    7550 9950
+	0    1    -1   0
+$EndComp
 $EndSCHEMATC

Commit message: update
Parts:
- J1: footprint Connector_PinHeader_2.00mm:PinHeader_1x04_P2.00mm_Vertical -> otter:PinHeader_1x04_P2.00mm_Vertical_nosilk_center
Connections:
- net UART1_RX: now also J1.2 (Pin_2); no longer J1.3 (Pin_3)
- net UART1_TX: now also J1.3 (Pin_3); no longer J1.2 (Pin_2)
Changed lines of the file:
@@
 F 0 "J1" H 7480 10392 50  0000 L CNN
 F 1 "UART" H 7480 10301 50  0000 L CNN
-F 2 "Connector_PinHeader_2.00mm:PinHeader_1x04_P2.00mm_Vertical" H 7400 10400 50  0001 C CNN
+F 2 "otter:PinHeader_1x04_P2.00mm_Vertical_nosilk_center" H 7400 10400 50  0001 C CNN
 F 3 "~" H 7400 10400 50  0001 C CNN
 	1    7400 10400
@@
 	0    1    1    0
 $EndComp
+Text GLabel 7200 10500 0    50   Input ~ 0
+UART1_TX
 Text GLabel 7200 10400 0    50   Input ~ 0
-UART1_TX
-Text GLabel 7200 10500 0    50   Input ~ 0
 UART1_RX
 $Comp

Commit message: update
Parts:
- removed C2: 100n, otter:C_0402, symbol Device:C_Small
Changed lines of the file:
@@
 	1    0    0    -1
 $EndComp
-Wire Wire Line
-	10050 10050 10050 10100
 $Comp
 L S3-OLinuXino_Rev_A:GND #PWR0112
@@
 	-1   0    0    -1
 $EndComp
-$Comp
-L Device:C_Small C2
-U 1 1 67C9846E
-P 9750 10100
-F 0 "C2" V 9979 10100 50  0000 C CNN
-F 1 "100n" V 9888 10100 50  0000 C CNN
-F 2 "otter:C_0402" H 9750 10100 50  0001 C CNN
-F 3 "~" H 9750 10100 50  0001 C CNN
-	1    9750 10100
-	0    -1   -1   0
-$EndComp
-$Comp
-L S3-OLinuXino_Rev_A:GND #PWR0113
-U 1 1 67C9D93C
-P 9550 10150
-F 0 "#PWR0113" H 9550 9900 50  0001 C CNN
-F 1 "GND" H 9550 10000 50  0000 C CNN
-F 2 "" H 9550 10150 60  0000 C CNN
-F 3 "" H 9550 10150 60  0000 C CNN
-	1    9550 10150
-	-1   0    0    -1
-$EndComp
-Wire Wire Line
-	9650 10100 9550 10100
-Wire Wire Line
-	9550 10100 9550 10150
-Connection ~ 10050 10100
-Wire Wire Line
-	10050 10100 10050 10150
 Text GLabel 10900 10450 2    50   Input ~ 0
 PB8\TWI1-SCK
@@
 Wire Wire Line
 	10500 10550 10500 10600
-Wire Wire Line
-	9850 10100 10050 10100
 Wire Wire Line
 	10900 10350 10550 10350
@@
 	0    1    -1   0
 $EndComp
+Wire Wire Line
+	10050 10050 10050 10150
 $EndSCHEMATC

Commit message: no drc error
Parts:
- R1, R10, R11, R12, R13, R2, R3, R4, R5, R6, R7, R8, R9: footprint otter:C_0402 -> otter:R_0402
Changed lines of the file:
@@
 F 0 "R7" V 11400 7750 50  0000 C CNN
 F 1 "47k" V 11400 8100 50  0000 C CNN
-F 2 "otter:C_0402" H 11450 7900 50  0001 C CNN
+F 2 "otter:R_0402" H 11450 7900 50  0001 C CNN
 F 3 "~" H 11450 7900 50  0001 C CNN
 	1    11450 7900
@@
 F 0 "R8" V 11400 7850 50  0000 C CNN
 F 1 "47k" V 11400 8200 50  0000 C CNN
-F 2 "otter:C_0402" H 11450 8000 50  0001 C CNN
+F 2 "otter:R_0402" H 11450 8000 50  0001 C CNN
 F 3 "~" H 11450 8000 50  0001 C CNN
 	1    11450 8000
@@
 F 0 "R9" V 11400 7950 50  0000 C CNN
 F 1 "47k" V 11400 8300 50  0000 C CNN
-F 2 "otter:C_0402" H 11450 8100 50  0001 C CNN
+F 2 "otter:R_0402" H 11450 8100 50  0001 C CNN
 F 3 "~" H 11450 8100 50  0001 C CNN
 	1    11450 8100
@@
 F 0 "R10" V 11400 8150 50  0000 C CNN
 F 1 "47k" V 11400 8500 50  0000 C CNN
-F 2 "otter:C_0402" H 11450 8300 50  0001 C CNN
+F 2 "otter:R_0402" H 11450 8300 50  0001 C CNN
 F 3 "~" H 11450 8300 50  0001 C CNN
 	1    11450 8300
@@
 F 0 "R11" V 11400 8350 50  0000 C CNN
 F 1 "47k" V 11400 8700 50  0000 C CNN
-F 2 "otter:C_0402" H 11450 8500 50  0001 C CNN
+F 2 "otter:R_0402" H 11450 8500 50  0001 C CNN
 F 3 "~" H 11450 8500 50  0001 C CNN
 	1    11450 8500
@@
 F 0 "R12" V 11400 8450 50  0000 C CNN
 F 1 "47k" V 11400 8800 50  0000 C CNN
-F 2 "otter:C_0402" H 11450 8600 50  0001 C CNN
+F 2 "otter:R_0402" H 11450 8600 50  0001 C CNN
 F 3 "~" H 11450 8600 50  0001 C CNN
 	1    11450 8600
@@
 F 0 "R13" V 11400 8550 50  0000 C CNN
 F 1 "47k" V 11400 8900 50  0000 C CNN
-F 2 "otter:C_0402" H 11450 8700 50  0001 C CNN
+F 2 "otter:R_0402" H 11450 8700 50  0001 C CNN
 F 3 "~" H 11450 8700 50  0001 C CNN
 	1    11450 8700
@@
 F 0 "R3" H 8041 10346 50  0000 R CNN
 F 1 "5k1" H 8041 10255 50  0000 R CNN
-F 2 "otter:C_0402" H 8100 10300 50  0001 C CNN
+F 2 "otter:R_0402" H 8100 10300 50  0001 C CNN
 F 3 "~" H 8100 10300 50  0001 C CNN
 	1    8100 10300
@@
 F 0 "R2" V 3950 6450 50  0000 C CNN
 F 1 "DNP" V 4000 6600 50  0000 C CNN
-F 2 "otter:C_0402" H 4000 6600 50  0001 C CNN
+F 2 "otter:R_0402" H 4000 6600 50  0001 C CNN
 F 3 "~" H 4000 6600 50  0001 C CNN
 	1    4000 6600
@@
 F 0 "R4" H 8391 10346 50  0000 R CNN
 F 1 "5k1" H 8391 10255 50  0000 R CNN
-F 2 "otter:C_0402" H 8450 10300 50  0001 C CNN
+F 2 "otter:R_0402" H 8450 10300 50  0001 C CNN
 F 3 "~" H 8450 10300 50  0001 C CNN
 	1    8450 10300
@@
 F 0 "R1" V 3646 2600 50  0000 C CNN
 F 1 "5k1" V 3555 2600 50  0000 C CNN
-F 2 "otter:C_0402" H 3450 2600 50  0001 C CNN
+F 2 "otter:R_0402" H 3450 2600 50  0001 C CNN
 F 3 "~" H 3450 2600 50  0001 C CNN
 	1    3450 2600
@@
 F 0 "R5" H 10609 10246 50  0000 L CNN
 F 1 "2.2k" H 10609 10155 50  0000 L CNN
-F 2 "otter:C_0402" H 10550 10200 50  0001 C CNN
+F 2 "otter:R_0402" H 10550 10200 50  0001 C CNN
 F 3 "~" H 10550 10200 50  0001 C CNN
 	1    10550 10200
@@
 F 0 "R6" H 10859 10246 50  0000 L CNN
 F 1 "2.2k" H 10859 10155 50  0000 L CNN
-F 2 "otter:C_0402" H 10800 10200 50  0001 C CNN
+F 2 "otter:R_0402" H 10800 10200 50  0001 C CNN
 F 3 "~" H 10800 10200 50  0001 C CNN
 	1    10800 10200

Commit message: no drc error
Parts:
- added R33: 100, otter:R_0402, symbol Device:R_Small
- R1: value 5k1 -> 100
Connections:
- net GND: no longer R1.1
- net UART1_RX: now also R1.2; no longer D5.1 (K), J1.2 (Pin_2)
- net UART1_TX: now also R33.2; no longer D5.2 (K), J1.3 (Pin_3)
- net BT-UART-RTS: now reaches U1.C4 (PB3/UART2_CTS/PB_EINT3)
- net BT-UART-RTS: no longer R1.2
- new net: D5.1 (K), J1.3 (Pin_3), R33.1
- new net: D5.2 (K), J1.2 (Pin_2), R1.1
Other:
- moved on the sheet: D5, J1
Changed lines of the file:
@@
-$EndComp
-$Comp
-L S3-OLinuXino_Rev_A:GND #PWR03
-U 1 1 5D904B73
-P 3300 2600
-F 0 "#PWR03" H 3300 2350 50  0001 C CNN
-F 1 "GND" V 3300 2425 50  0000 C CNN
-F 2 "" H 3300 2600 60  0000 C CNN
-F 3 "" H 3300 2600 60  0000 C CNN
-	1    3300 2600
-	0    1    1    0
 $EndComp
 $Comp
@@
 L Connector_Generic:Conn_01x04 J1
 U 1 1 635CE136
-P 7400 10400
-F 0 "J1" H 7480 10392 50  0000 L CNN
-F 1 "UART" H 7480 10301 50  0000 L CNN
-F 2 "otter:PinHeader_1x04_P2.00mm_Vertical_nosilk_center" H 7400 10400 50  0001 C CNN
-F 3 "~" H 7400 10400 50  0001 C CNN
-	1    7400 10400
+P 7000 9200
+F 0 "J1" H 7080 9192 50  0000 L CNN
+F 1 "UART" H 7080 9101 50  0000 L CNN
+F 2 "otter:PinHeader_1x04_P2.00mm_Vertical_nosilk_center" H 7000 9200 50  0001 C CNN
+F 3 "~" H 7000 9200 50  0001 C CNN
+	1    7000 9200
 	1    0    0    -1
 $EndComp
@@
 L otter:GND #PWR0107
 U 1 1 635CE777
-P 7200 10300
-F 0 "#PWR0107" H 7200 10050 50  0001 C CNN
-F 1 "GND" V 7205 10172 50  0000 R CNN
-F 2 "" H 7200 10300 60  0000 C CNN
-F 3 "" H 7200 10300 60  0000 C CNN
-	1    7200 10300
-	0    1    1    0
-$EndComp
-Text GLabel 7200 10500 0    50   Input ~ 0
+P 6800 9100
+F 0 "#PWR0107" H 6800 8850 50  0001 C CNN
+F 1 "GND" V 6805 8972 50  0000 R CNN
+F 2 "" H 6800 9100 60  0000 C CNN
+F 3 "" H 6800 9100 60  0000 C CNN
+	1    6800 9100
+	0    1    1    0
+$EndComp
+Text GLabel 6050 9300 0    50   Input ~ 0
 UART1_TX
-Text GLabel 7200 10400 0    50   Input ~ 0
+Text GLabel 6050 9200 0    50   Input ~ 0
 UART1_RX
 $Comp
 L S3-OLinuXino_Rev_A:+3.3V #PWR0108
 U 1 1 63623CC5
-P 7200 10600
-F 0 "#PWR0108" H 7200 10450 50  0001 C CNN
-F 1 "+3.3V" V 7215 10728 50  0000 L CNN
-F 2 "" H 7200 10600 60  0000 C CNN
-F 3 "" H 7200 10600 60  0000 C CNN
-	1    7200 10600
+P 6800 9400
+F 0 "#PWR0108" H 6800 9250 50  0001 C CNN
+F 1 "+3.3V" V 6815 9528 50  0000 L CNN
+F 2 "" H 6800 9400 60  0000 C CNN
+F 3 "" H 6800 9400 60  0000 C CNN
+	1    6800 9400
 	0    -1   1    0
 $EndComp
@@
 Text GLabel 4150 2500 0    50   Input ~ 0
 BT-UART-CTS
-$Comp
-L Device:R_Small R1
-U 1 1 67C10E27
-P 3450 2600
-F 0 "R1" V 3646 2600 50  0000 C CNN
-F 1 "5k1" V 3555 2600 50  0000 C CNN
-F 2 "otter:R_0402" H 3450 2600 50  0001 C CNN
-F 3 "~" H 3450 2600 50  0001 C CNN
-	1    3450 2600
-	0    -1   -1   0
-$EndComp
-Wire Wire Line
-	3300 2600 3350 2600
-Wire Wire Line
-	3550 2600 4150 2600
 Text GLabel 4150 2900 0    50   Input ~ 0
 PB6\TWI0-SCK
@@
 L Power_Protection:SP0502BAHT D5
 U 1 1 5FCE3FA8
-P 7350 9950
-F 0 "D5" V 7692 9950 50  0000 C CNN
-F 1 "ESD5302F" V 7601 9950 50  0000 C CNN
-F 2 "Package_TO_SOT_SMD:SOT-23" H 7575 9900 50  0001 L CNN
-F 3 "http://www.littelfuse.com/~/media/files/littelfuse/technical%20resources/documents/data%20sheets/sp05xxba.pdf" H 7475 10075 50  0001 C CNN
-F 4 "C239643" V 7350 9950 50  0001 C CNN "LCSC"
-	1    7350 9950
+P 7500 9250
+F 0 "D5" V 7842 9250 50  0000 C CNN
+F 1 "ESD5302F" V 7751 9250 50  0000 C CNN
+F 2 "Package_TO_SOT_SMD:SOT-23" H 7725 9200 50  0001 L CNN
+F 3 "http://www.littelfuse.com/~/media/files/littelfuse/technical%20resources/documents/data%20sheets/sp05xxba.pdf" H 7625 9375 50  0001 C CNN
+F 4 "C239643" V 7500 9250 50  0001 C CNN "LCSC"
+	1    7500 9250
 	0    -1   -1   0
 $EndComp
-Text GLabel 7150 9850 0    50   Input ~ 0
-UART1_TX
-Text GLabel 7150 10050 0    50   Input ~ 0
-UART1_RX
 $Comp
 L S3-OLinuXino_Rev_A:+3.3V #PWR0154
 U 1 1 5FCE77D5
-P 7550 9950
-F 0 "#PWR0154" H 7550 9800 50  0001 C CNN
-F 1 "+3.3V" V 7565 10078 50  0000 L CNN
-F 2 "" H 7550 9950 60  0000 C CNN
-F 3 "" H 7550 9950 60  0000 C CNN
-	1    7550 9950
+P 7700 9250
+F 0 "#PWR0154" H 7700 9100 50  0001 C CNN
+F 1 "+3.3V" V 7715 9378 50  0000 L CNN
+F 2 "" H 7700 9250 60  0000 C CNN
+F 3 "" H 7700 9250 60  0000 C CNN
+	1    7700 9250
 	0    1    -1   0
 $EndComp
 Wire Wire Line
 	10050 10050 10050 10150
+Text GLabel 4150 2600 0    50   Input ~ 0
+BT-UART-RTS
+$Comp
+L Device:R_Small R1
+U 1 1 5FE69B36
+P 6250 9200
+F 0 "R1" V 6200 9050 50  0000 C CNN
+F 1 "100" V 6250 9200 50  0000 C CNN
+F 2 "otter:R_0402" H 6250 9200 50  0001 C CNN
+F 3 "~" H 6250 9200 50  0001 C CNN
+	1    6250 9200
+	0    1    1    0
+$EndComp
+$Comp
+L Device:R_Small R33
+U 1 1 5FE69B3C
+P 6250 9300
+F 0 "R33" V 6200 9150 50  0000 C CNN
+F 1 "100" V 6250 9300 50  0000 C CNN
+F 2 "otter:R_0402" H 6250 9300 50  0001 C CNN
+F 3 "~" H 6250 9300 50  0001 C CNN
+	1    6250 9300
+	0    1    1    0
+$EndComp
+Wire Wire Line
+	6050 9200 6150 9200
+Wire Wire Line
+	6050 9300 6150 9300
+Wire Wire Line
+	6350 9200 6400 9200
+Wire Wire Line
+	6350 9300 6400 9300
+Wire Wire Line
+	6400 9300 6400 9500
+Wire Wire Line
+	6400 9500 7300 9500
+Wire Wire Line
+	7300 9500 7300 9350
+Connection ~ 6400 9300
+Wire Wire Line
+	6400 9300 6800 9300
+Wire Wire Line
+	6400 9200 6400 9000
+Wire Wire Line
+	6400 9000 7300 9000
+Wire Wire Line
+	7300 9000 7300 9150
+Connection ~ 6400 9200
+Wire Wire Line
+	6400 9200 6800 9200
 $EndSCHEMATC
