File: WifiBT.sch (KiCad schematic (older format))
At the start: 20 parts

Commit message: update
Parts:
- added R? (x4): DNP, otter:C_0402, symbol Device:R_Small
Connections:
- wire segments 67 -> 75
Other:
- moved on the sheet: C?, L?, R?

Commit message: update
Parts:
- gave numbers to parts that had none: 24

Commit message: update
Parts:
- removed AE1: ANT, symbol Device:Antenna_Shield
- added AE1: KH-5220-A56_U.FL, otter:KH-5220-A56, symbol otter:KH-5220-A56_U.FL
- U7: footprint (none) -> otter:STL8723BS
Connections:
- no-connect marks 0 -> 1
Changed lines of the file:
@@
 F 0 "U7" H 5350 5447 60  0000 C CNN
 F 1 "RTL8723BS" H 5350 5341 60  0000 C CNN
-F 2 "" H 5350 3950 60  0001 C CNN
+F 2 "otter:STL8723BS" H 5350 3950 60  0001 C CNN
 F 3 "" H 5350 3950 60  0000 C CNN
 	1    5350 4150
@@
 AR Path="/602ACDF9/67FCAAB7" Ref="L?"  Part="1"
 AR Path="/6191F40B/67FCAAB7" Ref="L5"  Part="1"
-F 0 "L5" V 4535 4400 50  0000 C CNN
-F 1 "2.2uH" V 4444 4400 50  0000 C CNN
+F 0 "L5" V 4500 4400 50  0000 C CNN
+F 1 "2.2uH" V 4400 4400 50  0000 C CNN
 F 2 "Inductor_SMD:L_0402_1005Metric" H 4350 4400 50  0001 C CNN
 F 3 "~" H 4350 4400 50  0001 C CNN
@@
 	1    4150 4550
 	-1   0    0    1
-$EndComp
-$Comp
-L Device:Antenna_Shield AE1
-U 1 1 67FD0CA7
-P 4150 4050
-F 0 "AE1" H 4070 4089 50  0000 R CNN
-F 1 "ANT" H 4070 3998 50  0000 R CNN
-F 2 "" H 4150 4150 50  0001 C CNN
-F 3 "~" H 4150 4150 50  0001 C CNN
-	1    4150 4050
-	-1   0    0    -1
 $EndComp
 Wire Wire Line
@@
 Wire Wire Line
 	6150 3950 5950 3950
+$Comp
+L otter:KH-5220-A56_U.FL AE1
+U 1 1 60E512A9
+P 4150 4050
+F 0 "AE1" H 4150 4417 50  0000 C CNN
+F 1 "KH-5220-A56_U.FL" H 4150 4326 50  0000 C CNN
+F 2 "otter:KH-5220-A56" H 4150 4150 50  0001 C CNN
+F 3 "~" H 4150 4150 50  0001 C CNN
+	1    4150 4050
+	-1   0    0    -1
+$EndComp
+NoConn ~ 4250 4250
 $EndSCHEMATC

Commit message: update
Parts:
- L5: footprint Inductor_SMD:L_0402_1005Metric -> otter:L_0402
Changed lines of the file:
@@
 F 0 "L5" V 4500 4400 50  0000 C CNN
 F 1 "2.2uH" V 4400 4400 50  0000 C CNN
-F 2 "Inductor_SMD:L_0402_1005Metric" H 4350 4400 50  0001 C CNN
+F 2 "otter:L_0402" H 4350 4400 50  0001 C CNN
 F 3 "~" H 4350 4400 50  0001 C CNN
 	1    4350 4400

Commit message: no drc error
Parts:
- R64, R65, R66, R67, R68, R69, R70, R71, R72, R73, R74, R75, R76, R77: footprint otter:C_0402 -> otter:R_0402
Changed lines of the file:
@@
 F 0 "R73" V 6600 2650 50  0000 C CNN
 F 1 "47k" V 6600 2950 50  0000 C CNN
-F 2 "otter:C_0402" H 6650 2800 50  0001 C CNN
+F 2 "otter:R_0402" H 6650 2800 50  0001 C CNN
 F 3 "~" H 6650 2800 50  0001 C CNN
 	1    6650 2800
@@
 F 0 "R72" V 6500 2650 50  0000 C CNN
 F 1 "47k" V 6500 2950 50  0000 C CNN
-F 2 "otter:C_0402" H 6550 2800 50  0001 C CNN
+F 2 "otter:R_0402" H 6550 2800 50  0001 C CNN
 F 3 "~" H 6550 2800 50  0001 C CNN
 	1    6550 2800
@@
 F 0 "R71" V 6400 2650 50  0000 C CNN
 F 1 "47k" V 6400 2950 50  0000 C CNN
-F 2 "otter:C_0402" H 6450 2800 50  0001 C CNN
+F 2 "otter:R_0402" H 6450 2800 50  0001 C CNN
 F 3 "~" H 6450 2800 50  0001 C CNN
 	1    6450 2800
@@
 F 0 "R70" V 6300 2650 50  0000 C CNN
 F 1 "47k" V 6300 2950 50  0000 C CNN
-F 2 "otter:C_0402" H 6350 2800 50  0001 C CNN
+F 2 "otter:R_0402" H 6350 2800 50  0001 C CNN
 F 3 "~" H 6350 2800 50  0001 C CNN
 	1    6350 2800
@@
 F 0 "R65" V 6200 2650 50  0000 C CNN
 F 1 "47k" V 6200 2950 50  0000 C CNN
-F 2 "otter:C_0402" H 6250 2800 50  0001 C CNN
+F 2 "otter:R_0402" H 6250 2800 50  0001 C CNN
 F 3 "~" H 6250 2800 50  0001 C CNN
 	1    6250 2800
@@
 F 0 "R64" V 6100 2650 50  0000 C CNN
 F 1 "47k" V 6100 2950 50  0000 C CNN
-F 2 "otter:C_0402" H 6150 2800 50  0001 C CNN
+F 2 "otter:R_0402" H 6150 2800 50  0001 C CNN
 F 3 "~" H 6150 2800 50  0001 C CNN
 	1    6150 2800
@@
 F 0 "R77" V 6900 3150 50  0000 C CNN
 F 1 "22" V 6900 3450 50  0000 C CNN
-F 2 "otter:C_0402" H 6950 3300 50  0001 C CNN
+F 2 "otter:R_0402" H 6950 3300 50  0001 C CNN
 F 3 "~" H 6950 3300 50  0001 C CNN
 	1    6950 3300
@@
 F 0 "R76" V 6700 4900 50  0000 C CNN
 F 1 "22" V 6700 5200 50  0000 C CNN
-F 2 "otter:C_0402" H 6750 5050 50  0001 C CNN
+F 2 "otter:R_0402" H 6750 5050 50  0001 C CNN
 F 3 "~" H 6750 5050 50  0001 C CNN
 	1    6750 5050
@@
 F 0 "R75" V 6700 4600 50  0000 C CNN
 F 1 "47k" V 6700 4900 50  0000 C CNN
-F 2 "otter:C_0402" H 6750 4750 50  0001 C CNN
+F 2 "otter:R_0402" H 6750 4750 50  0001 C CNN
 F 3 "~" H 6750 4750 50  0001 C CNN
 	1    6750 4750
@@
 F 0 "R74" V 6700 4250 50  0000 C CNN
 F 1 "47k" V 6700 4550 50  0000 C CNN
-F 2 "otter:C_0402" H 6750 4400 50  0001 C CNN
+F 2 "otter:R_0402" H 6750 4400 50  0001 C CNN
 F 3 "~" H 6750 4400 50  0001 C CNN
 	1    6750 4400
@@
 F 0 "R69" V 6200 4100 50  0000 C CNN
 F 1 "DNP" V 6200 4400 50  0000 C CNN
-F 2 "otter:C_0402" H 6250 4250 50  0001 C CNN
+F 2 "otter:R_0402" H 6250 4250 50  0001 C CNN
 F 3 "~" H 6250 4250 50  0001 C CNN
 	1    6250 4250
@@
 F 0 "R68" V 6200 4000 50  0000 C CNN
 F 1 "DNP" V 6200 4300 50  0000 C CNN
-F 2 "otter:C_0402" H 6250 4150 50  0001 C CNN
+F 2 "otter:R_0402" H 6250 4150 50  0001 C CNN
 F 3 "~" H 6250 4150 50  0001 C CNN
 	1    6250 4150
@@
 F 0 "R67" V 6200 3900 50  0000 C CNN
 F 1 "DNP" V 6200 4200 50  0000 C CNN
-F 2 "otter:C_0402" H 6250 4050 50  0001 C CNN
+F 2 "otter:R_0402" H 6250 4050 50  0001 C CNN
 F 3 "~" H 6250 4050 50  0001 C CNN
 	1    6250 4050
@@
 F 0 "R66" V 6200 3800 50  0000 C CNN
 F 1 "DNP" V 6200 4100 50  0000 C CNN
-F 2 "otter:C_0402" H 6250 3950 50  0001 C CNN
+F 2 "otter:R_0402" H 6250 3950 50  0001 C CNN
 F 3 "~" H 6250 3950 50  0001 C CNN
 	1    6250 3950

Commit message: no drc error
Parts:
- removed U7: RTL8723BS, otter:STL8723BS, symbol otter:RTL8723BS
- added C48: 10u, otter:C_0603, symbol Device:C_Small
- added C49: DNP, otter:C_0402, symbol Device:C_Small
- added L4: 2.2uH, Inductor_SMD:L_Taiyo-Yuden_MD-3030, symbol Device:L_Small
- added U7: AP6236, otter:LGA_44_12x12mm_0.9mm, symbol otter:AP6236
- added X1: 26Mhz TCXO, otter:2016_SMD_CRYSTAL, symbol Oscillator:TXC-7C
Connections:
- net labels added: BT-UART-RTS
- wire segments 75 -> 90
- no-connect marks 1 -> 3
Other:
- moved on the sheet: AE1, C75, C77, C78, L5, R74, R75, R76

Commit message: fixed axp bug, fixed schematics, fixed eeprom
Connections:
- net GND: no longer X1.1 (EN)
- no-connect marks 3 -> 4
Changed lines of the file:
@@
 	-1   0    0    -1
 $EndComp
-$Comp
-L S3-OLinuXino_Rev_A:GND #PWR?
-U 1 1 5FE4A730
-P 2900 4800
-AR Path="/5D8A1FAC/5FE4A730" Ref="#PWR?"  Part="1"
-AR Path="/5FE4A730" Ref="#PWR?"  Part="1"
-AR Path="/602ACDF9/5FE4A730" Ref="#PWR?"  Part="1"
-AR Path="/6191F40B/5FE4A730" Ref="#PWR0221"  Part="1"
-F 0 "#PWR0221" H 2900 4550 50  0001 C CNN
-F 1 "GND" H 2905 4627 50  0000 C CNN
-F 2 "" H 2900 4800 60  0000 C CNN
-F 3 "" H 2900 4800 60  0000 C CNN
-	1    2900 4800
-	-1   0    0    -1
-$EndComp
-Wire Wire Line
-	2950 4750 2900 4750
-Wire Wire Line
-	2900 4750 2900 4800
 Wire Wire Line
 	3550 4750 4250 4750
 Wire Wire Line
 	4250 4550 4250 4750
+NoConn ~ 2950 4750
 $EndSCHEMATC
