File: WifiBT.sch (KiCad schematic (older format))
At the start: 28 parts, among them U7 AP6236, X1 26Mhz TCXO

Commit message: beautify kicad project
Parts:
- L5: value 2.2uH -> 2.2nH
Connections:
- net labels added: +3V3, AP_CK32KO, AP_WAKE_BT, BT_DIS_N, BT_PCM_CLK, BT_PCM_DIN, BT_PCM_DOUT, BT_PCM_SYNC, BT_UART_CTS, BT_UART_RTS, BT_UART_RX, BT_UART_TX, BT_WAKE_AP, WL_PMU_EN, WL_SDIO_CLK, WL_SDIO_CMD, WL_SDIO_D0, WL_SDIO_D1, WL_SDIO_D2, WL_SDIO_D3, WL_WAKE_AP
- net labels removed: +3.3V, AP-CK32KO, AP-WAKE-BT, BT-DIS-N, BT-PCM-CLK, BT-PCM-DIN, BT-PCM-DOUT, BT-PCM-SYNC, BT-UART-CTS, BT-UART-RTS, BT-UART-RX, BT-UART-TX, BT-WAKE-AP, WL-PMU-EN, WL-SDIO-CLK, WL-SDIO-CMD, WL-SDIO-D0, WL-SDIO-D1, WL-SDIO-D2, WL-SDIO-D3, WL-WAKE-AP
