File: OtterCastAudioV2.kicad_sch (KiCad schematic)
At the start: 21 parts

Commit message: updated kicad files
Parts:
- C1, C4: value (none) -> 10u; footprint (none) -> otter:C_0603
- D1, D2: value (none) -> LED; footprint (none) -> otter:LED_0603_1608Metric
- D5: value (none) -> ESD5302F; footprint (none) -> Package_TO_SOT_SMD:SOT-23
- FB1: value (none) -> FERRET; footprint (none) -> otter:R_0805
- J1: value (none) -> UART; footprint (none) -> otter:PinHeader_1x04_P2.00mm_Vertical_nosilk_center
- J2: value (none) -> SD; footprint (none) -> Connector_Card:microSD_HC_Hirose_DM3D-SF
- R1, R33: value (none) -> 100; footprint (none) -> otter:R_0402
- R10, R11, R12, R13, R7, R8, R9: value (none) -> 47k; footprint (none) -> otter:R_0402
- R2: value (none) -> 22; footprint (none) -> otter:R_0402
- R3, R4: value (none) -> 5k1; footprint (none) -> otter:R_0402
- U1: value (none) -> AllWinner-S3(FBGA-234); footprint (none) -> otter:FBGA-234(Pitch-0.65mm_Pad-0.3mm_11x11x1.08mm)
