File: Audio.kicad_sch (KiCad schematic)
At the start: 53 parts

Commit message: updated kicad files to v2.1.1, updated license
Parts:
- C46, C50, C53, C70, C71: renamed from C?; value (none) -> 220p; footprint (none) -> otter:C_0402
- C47: renamed from C?; value (none) -> 1n; footprint (none) -> otter:C_0402
- C51, C52: renamed from C?; value (none) -> 18p; footprint (none) -> otter:C_0402
- C54, C55, C56, C57, C60, C62, C63, C64, C69: value (none) -> 10u; footprint (none) -> otter:CP_EIA-3216-10
- C58, C59, C61, C65, C66: renamed from C?; value (none) -> 100n; footprint (none) -> otter:C_0402
- C67, C68: value (none) -> 100u; footprint (none) -> otter:CP_EIA-3528-12
- FB2, FB3: renamed from FB?; value (none) -> FERRET; footprint (none) -> otter:R_0805
- J5, J6, J7: value (none) -> PJ-3270; footprint (none) -> otter:PJ-3270
- MK1: value (none) -> Mic; footprint (none) -> otter:B4013AM422-42
- R27: renamed from R?; value (none) -> 0R; footprint (none) -> otter:R_0805
- R40: renamed from R?; value (none) -> 200k; footprint (none) -> otter:R_0402
- R41, R48, R49, R50, R51: renamed from R?; value (none) -> 2k2; footprint (none) -> otter:R_0402
- R42, R58, R59, R60, R63: renamed from R?; value (none) -> 47k; footprint (none) -> otter:R_0402
- R43: renamed from R?; value (none) -> 680; footprint (none) -> otter:R_0402
- R44, R45, R46: renamed from R?; value (none) -> 0; footprint (none) -> otter:R_0402
- R47, R52: renamed from R?; value (none) -> DNP; footprint (none) -> otter:R_0402
- R54: renamed from R?; value (none) -> 22; footprint (none) -> otter:R_0402
- R61, R62: renamed from R?; value (none) -> 100; footprint (none) -> otter:R_0402
- U6: value (none) -> SSM2603; footprint (none) -> otter:LFCSP-28-5x5mm-0.5mm-EP3.14x3.14mm
- Y1: renamed from Y?; value (none) -> 12.288Mhz; footprint (none) -> otter:Oscillator_3225
