File: MIPI.kicad_sch (KiCad schematic)
At the start: 40 parts

Commit message: updated kicad files to v2.1.1, updated license
Parts:
- C100, C101, C102, C103, C3, C82, C83, C85, C88, C89, C98, C99: renamed from C?; value (none) -> 100n; footprint (none) -> otter:C_0402
- C104: renamed from C?; value (none) -> 1n; footprint (none) -> otter:C_0805
- C79, C90, C92, C95: renamed from C?; value (none) -> 10u; footprint (none) -> otter:C_0603
- C93, C94, C96, C97: renamed from C?; value (none) -> 18p; footprint (none) -> otter:C_0402
- J8: value (none) -> 49F-1201GYD2NL; footprint (none) -> otter:49F-1201GYDXNL
- R78: renamed from R?; value (none) -> 200k; footprint (none) -> otter:R_0402
- R79, R80, R87, R88: renamed from R?; value (none) -> 2k2; footprint (none) -> otter:R_0402
- R81: renamed from R?; value (none) -> 22; footprint (none) -> otter:R_0402
- R82, R83: renamed from R?; value (none) -> 240; footprint (none) -> otter:R_0402
- R84: renamed from R?; value (none) -> 10M; footprint (none) -> otter:R_0402
- R86: renamed from R?; value (none) -> 5k1; footprint (none) -> otter:R_0402
- R89: renamed from R?; value (none) -> 6k04; footprint (none) -> otter:R_0402
- R90, R91, R92, R93: renamed from R?; value (none) -> 51; footprint (none) -> otter:R_0402
- U1: renamed from U?; value (none) -> AllWinner-S3(FBGA-234); footprint (none) -> otter:FBGA-234(Pitch-0.65mm_Pad-0.3mm_11x11x1.08mm)
- Y2: value (none) -> 32.768kHz; footprint (none) -> otter:Crystal_SMD_3215-2Pin_3.2x1.5mm
- Y3: value (none) -> 24MHz; footprint (none) -> otter:Oscillator_3225
