File: Power.kicad_sch (KiCad schematic)
At the start: 78 parts

Commit message: updated kicad files to v2.1.1, updated license
Parts:
- C10, C11, C42, C43, C45, C5: renamed from C?; value (none) -> 47u; footprint (none) -> otter:C_0805
- C12: renamed from C?; value (none) -> 1n; footprint (none) -> otter:C_0402
- C13: renamed from C?; value (none) -> 1n; footprint (none) -> otter:C_0805
- C14, C16, C17, C19, C20, C22, C23, C24, C25, C26, C27, C28, C29, C30, C31, C39, C41, C6: renamed from C?; value (none) -> 10u; footprint (none) -> otter:C_0603
- C15, C18, C21, C32, C33, C34, C35, C36, C37, C38, C44, C7, C8: renamed from C?; value (none) -> 100n; footprint (none) -> otter:C_0402
- C2: renamed from C?; value (none) -> 470n; footprint (none) -> otter:C_0402
- C9: renamed from C?; value (none) -> 2.2u; footprint (none) -> otter:C_0603
- D3: renamed from D?; value (none) -> LED; footprint (none) -> LED_SMD:LED_0603_1608Metric_Castellated
- D4: value (none) -> P6SMB6.8CA; footprint (none) -> Diode_SMD:D_SMB
- D6: value (none) -> ESD5302F; footprint (none) -> Package_TO_SOT_SMD:SOT-23
- J3: value (none) -> USB; footprint (none) -> otter:USB-C 16Pin
- J4: renamed from J?; value (none) -> OTG; footprint (none) -> otter:PinHeader_1x04_P2.00mm_Vertical_nosilk_center
- L1, L2, L3: value (none) -> 2.2uH; footprint (none) -> Inductor_SMD:L_Taiyo-Yuden_MD-3030
- Q1: value (none) -> DTA114YKA; footprint (none) -> Package_TO_SOT_SMD:SOT-23
- R14, R24, R25, R30, R35, R36, R39: renamed from R?; value (none) -> 5k1; footprint (none) -> otter:R_0402
- R15, R34: renamed from R?; value (none) -> 22; footprint (none) -> otter:R_0402
- R16, R21: renamed from R?; value (none) -> 200k; footprint (none) -> otter:R_0402
- R17, R28, R37: renamed from R?; value (none) -> 2k2; footprint (none) -> otter:R_0402
- R18, R26: renamed from R?; value (none) -> 47k; footprint (none) -> otter:R_0402
- R22, R23, R29, R6: renamed from R?; value (none) -> DNP; footprint (none) -> otter:R_0402
- R31: renamed from R?; value (none) -> 3k3; footprint (none) -> otter:R_0402
- R32: renamed from R?; value (none) -> 100; footprint (none) -> otter:R_0402
- R38: renamed from R?; value (none) -> 3k9; footprint (none) -> otter:R_0402
- SW3: value (none) -> RST; footprint (none) -> otter:SW_SPST_PTS810
- U1: renamed from U?; value (none) -> AllWinner-S3(FBGA-234); footprint (none) -> otter:FBGA-234(Pitch-0.65mm_Pad-0.3mm_11x11x1.08mm)
- U3: value (none) -> AXP209(QFN-48); footprint (none) -> otter:QFN-48-1EP_6x6mm_P0.4mm_EP4.05x4.05mm
- U4: renamed from U?; value (none) -> SY8089AAAC; footprint (none) -> Package_TO_SOT_SMD:SOT-23-5
- U5: renamed from U?; value (none) -> SY6280AAC; footprint (none) -> Package_TO_SOT_SMD:SOT-23-5
