File: WifiBT.kicad_sch (KiCad schematic)
At the start: 28 parts

Commit message: updated kicad files to v2.1.1, updated license
Parts:
- AE1: value (none) -> KH-5220-A56_U.FL; footprint (none) -> otter:KH-5220-A56
- C48, C72, C74: renamed from C?; value (none) -> 10u; footprint (none) -> otter:C_0603
- C49: renamed from C?; value (none) -> DNP; footprint (none) -> otter:C_0402
- C73, C76: renamed from C?; value (none) -> 100n; footprint (none) -> otter:C_0402
- C75, C77: renamed from C?; value (none) -> 1p; footprint (none) -> otter:C_0402
- C78: renamed from C?; value (none) -> 10p; footprint (none) -> otter:C_0402
- L4: renamed from L?; value (none) -> 2.2uH; footprint (none) -> Inductor_SMD:L_Taiyo-Yuden_MD-3030
- L5: renamed from L?; value (none) -> 2.2nH; footprint (none) -> otter:L_0402
- R64, R65, R70, R71, R72, R73, R74, R75: renamed from R?; value (none) -> 47k; footprint (none) -> otter:R_0402
- R66, R67, R68, R69: renamed from R?; value (none) -> DNP; footprint (none) -> otter:R_0402
- R76, R77: renamed from R?; value (none) -> 22; footprint (none) -> otter:R_0402
- U7: value (none) -> AP6236; footprint (none) -> otter:LGA_44_12x12mm_0.9mm
- X1: value (none) -> 26Mhz TCXO; footprint (none) -> otter:2016_SMD_CRYSTAL
