File: Edgerails/Edgerails.kicad_pcb (KiCad board)
At the start: 4 copper layers, 4 x 50 mm, 1 part

Commit message: added i2c to axp209, fixed tvs diodes
Other:
- board text added: "OtterCastAudioV2 v2.1"
- board text removed: "OtterCastAudioV2 v2.0"
Changed lines of the file:
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@@
     (effects (font (size 0.6 0.6) (thickness 0.1)))
   )
-  (gr_text "OtterCastAudioV2 v2.0" (at 52 75 270) (layer F.SilkS)
+  (gr_text "OtterCastAudioV2 v2.1\n" (at 52 75 270) (layer F.SilkS)
     (effects (font (size 1.5 1.5) (thickness 0.15)))
   )

Commit message: updated edgerails
Other:
- net class Default removed
- board text added: "OtterCastAudioV2 v2.1.1"
- board text removed: "OtterCastAudioV2 v2.1"
